File: Circuit/Power_dist/component-alignment.kicad_pcb (KiCad board)
At the start: 2 copper layers, 150.2 x 108.9 mm, 97 parts, among them CON1 Conn-PCIE-x16, J1 Thruster_Off_Switch, P1 XT60, P11 XT60, P15 USB_B, P16 XT60, P17 XT60, P2 XT30, P3 XT30, P4 XT30, P5 XT30, Q1 IPD90P03P4L, Q2 IPD90P03P4L, Q3 IPD90P03P4L, Q5 IPD90P03P4L, Q6 AUIRFS8409-7P, Q7 AUIRFS8409-7P, U1 93LC56BT-I/OT, U2 FT232H, U3 ACPL-247-500E, U4 ACPL-247-500E, U5 LTC4357, U6 LTC4357, U7 UWE-12/6-Q12P, U8 TEN_20-2411WIN, Y1 12MHz

Commit message: route pcb except gnd
Parts:
- moved C13 1.55 mm to (95.2, 158.2)
- moved C14 1.55 mm to (89.1, 155.2)
- moved C15 1.55 mm to (94.9, 155.2)
- moved C17 1.55 mm to (101.1, 155.2)
- moved C5 1.55 mm to (83.9, 162.8)
- moved C7 1.55 mm to (89.1, 152.1)
- moved C8 1.55 mm to (78.5, 162.8)
- moved D7 1.55 mm to (69.8, 159.0)
- moved L2 1.55 mm to (95.0, 152.1)
- moved P15 1.55 mm to (53.6, 168.4)
- moved R10 1.55 mm to (65.1, 159.0)
- moved R17 1.55 mm to (68.5, 148.1)
- moved R18 1.55 mm to (59.6, 159.0)
- moved R19 1.55 mm to (63.8, 148.1)
- moved R22 1.55 mm to (78.4, 173.7)
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Routing:
- net +12V: track 0.00 -> 168.8 mm
- net Net-(JP1-Pad2): track 0.00 -> 53.3 mm
- net +5V: track 0.00 -> 30.1 mm
- net +BATT: track 0.00 -> 10.1 mm
- net Net-(D12-Pad2): track 0.00 -> 3.64 mm
- net Net-(D11-Pad2): track 0.00 -> 3.56 mm
- net VBUS: track 70.4 -> 71.6 mm
Other:
- outline, holes or cut-outs redrawn
