File: Circuit/Power_dist/Power-Volt-Converter.sch (KiCad schematic (older format))
At the start: 25 parts, among them P18 XT60, P19 XT60, P20 XT60, P21 XT60, P22 XT60, P23 XT60, P24 XT60, P25 XT60, Q8 BC817-40, U10 I6A24014A033V, U7 UWE-12/6-Q12P, U8 TEN_20-2411WIN, U9 TEN_20-2411WIN

Commit message: Merge commit '3eda1dba5ca6e598d51cb20764784284330d387d'
Parts:
- removed C19: 100uF, Capacitors_SMD:CP_Elec_8x10.5, symbol C
- removed D13, D14: Led_Small, LEDs:LED_0603, symbol LED_Small
- removed P18, P19, P20, P21, P22, P23, P24, P25: XT60, Zeabus:XT60, symbol XT60
- removed Q8: BC817-40, TO_SOT_Packages_SMD:SOT-23, symbol BC817-40
- removed R29: 10k, Resistors_SMD:R_0603, symbol R
- removed R32, R33: 1k, Resistors_SMD:R_0603, symbol R
- removed R34: 2.2k, Resistors_SMD:R_0603, symbol R
- removed U10: I6A24014A033V, Zeabus:I6A24014A033V, symbol I6A24014A033V
- removed U9: TEN_20-2411WIN, Zeabus:TEN_20WIN, symbol TEN_20-2411WIN
- added P4, P5: XT30, zeabus:XT30, symbol XT30
- D11, D12: footprint LEDs:LED_0603 -> LEDs:LED_0603_HandSoldering
- R30, R31: footprint Resistors_SMD:R_0603 -> Resistors_SMD:R_0603_HandSoldering
- U7: footprint Zeabus:UWE-xxxx -> zeabus:UWE-xxxx
- U8: footprint Zeabus:TEN_20WIN -> zeabus:TEN_20WIN
Connections:
- net at JP1.2: now also U7.2 (On/~Off), U8.6 (On/Off)
- net GNDREF: now reaches D11.1 (K), U7.4 (-Vout)
- net GNDREF: now also D12.1 (K), U8.5 (-Vout), P4.2 (P2), P5.2 (P2)
- net +12V: now reaches R30.2, U7.8 (+Vout)
- net +12V: now also P4.1 (P1)
- net +5V: now reaches R31.2, U8.3 (+Vout)
- net +5V: now also P5.1 (P1)
- no-connect marks 4 -> 3
Other:
- note removed: "DSP"
- note removed: "DSP Supply"
- note removed: "Eth Switch"
- note removed: "Lamp1"
- note removed: "Lamp2"
- note removed: "NUC1"
- note removed: "NUC2"
- note removed: "Solenoid"
- note removed: "USB Hub"
- moved on the sheet: D12, JP1, R31, U8
