File: Circuit/Power_dist/Power-Volt-Converter.sch (KiCad schematic (older format))
At the start: 9 parts, among them P4 XT30, P5 XT30, U7 UWE-12/6-Q12P, U8 TEN_20-2411WIN

Commit message: added filter to dc-dc converters in Power_dist
Parts:
- added C? (x4): 1000pF, symbol C_Small
- added C? (x2): 6.8uF, symbol C_Small
- added L?: 3.3uF, symbol L
- D11: value Led_Small -> +12V_LED
- D12: value Led_Small -> +5V_LED
- JP1: value Main Switch (N.O.) -> Main_Switch_(N.O.)
- P4: value XT30 -> +12V
- P5: value XT30 -> +5V
Connections:
- wire segments 29 -> 52
- no-connect marks 3 -> 1
Other:
- note removed: "Main 5V Supply"
- note removed: "Master Supply"
- moved on the sheet: D11, D12, JP1, P4, P5, R30, R31, U7, U8

Commit message: added +5v voltage regulator on battery side of Power_dist
Changed lines of the file:
@@
 	1    0    0    -1
 $EndComp
-Text HLabel 3875 2375 0    60   Input ~ 0
+Text HLabel 3875 2375 0    60   UnSpc ~ 0
 +VBatt
 $Comp
@@
 	6675 5075 7400 5075
 Wire Wire Line
-	6550 4525 7400 4525
+	6550 4525 8100 4525
 Wire Wire Line
 	6550 4675 6675 4675
@@
 Connection ~ 7050 2375
 Wire Wire Line
-	6550 2375 7400 2375
+	6550 2375 8100 2375
 Wire Wire Line
 	6550 2975 7400 2975
@@
 Wire Wire Line
 	4100 2200 4100 2375
+Text HLabel 8100 2375 2    60   UnSpc ~ 0
++12V
+Text HLabel 8100 4525 2    60   UnSpc ~ 0
++5V
 $EndSCHEMATC

Commit message: refactor Power_dist
Parts:
- C? (x4): footprint (none) -> Capacitors_SMD:C_1206_HandSoldering
- C? (x2): footprint (none) -> Capacitors_SMD:C_1812_HandSoldering
Connections:
- net labels added: GNDPWR
- net labels removed: GND
Changed lines of the file:
@@
 $EndDescr
-$Comp
-L GND #PWR037
-U 1 1 58C8506B
-P 5250 2825
-F 0 "#PWR037" H 5250 2575 60  0001 C CNN
-F 1 "GND" H 5250 2675 60  0000 C CNN
-F 2 "" H 5250 2825 60  0000 C CNN
-F 3 "" H 5250 2825 60  0000 C CNN
-	1    5250 2825
-	1    0    0    -1
-$EndComp
 $Comp
 L R R30
@@
 $EndComp
 $Comp
-L GND #PWR038
-U 1 1 58C8524E
-P 5250 4825
-F 0 "#PWR038" H 5250 4575 60  0001 C CNN
-F 1 "GND" H 5250 4675 60  0000 C CNN
-F 2 "" H 5250 4825 60  0000 C CNN
-F 3 "" H 5250 4825 60  0000 C CNN
-	1    5250 4825
-	1    0    0    -1
-$EndComp
-$Comp
 L TEN_20-2411WIN U8
 U 1 1 58C8526A
@@
 $EndComp
 $Comp
-L GND #PWR040
-U 1 1 58C8B273
-P 4225 5375
-F 0 "#PWR040" H 4225 5125 60  0001 C CNN
-F 1 "GND" H 4225 5225 60  0000 C CNN
-F 2 "" H 4225 5375 60  0000 C CNN
-F 3 "" H 4225 5375 60  0000 C CNN
-	1    4225 5375
-	1    0    0    -1
-$EndComp
-$Comp
 L +BATT #PWR041
 U 1 1 58C8C536
-P 5250 4350
-F 0 "#PWR041" H 5250 4200 50  0001 C CNN
-F 1 "+BATT" H 5250 4490 50  0000 C CNN
-F 2 "" H 5250 4350 50  0000 C CNN
-F 3 "" H 5250 4350 50  0000 C CNN
-	1    5250 4350
+P 5225 4350
+F 0 "#PWR041" H 5225 4200 50  0001 C CNN
+F 1 "+BATT" H 5225 4490 50  0000 C CNN
+F 2 "" H 5225 4350 50  0000 C CNN
+F 3 "" H 5225 4350 50  0000 C CNN
+	1    5225 4350
 	1    0    0    -1
 $EndComp
@@
 	6550 4675 6675 4675
 Wire Wire Line
-	5250 4675 5450 4675
-Wire Wire Line
-	5250 4525 5450 4525
+	5225 4675 5450 4675
+Wire Wire Line
+	5225 4525 5450 4525
 Wire Wire Line
 	4325 5175 4225 5175
@@
 F 0 "C?" V 5900 3825 50  0000 L CNN
 F 1 "1000pF" V 6100 3900 50  0000 L CNN
-F 2 "" H 6000 3900 50  0001 C CNN
+F 2 "Capacitors_SMD:C_1206_HandSoldering" H 6000 3900 50  0001 C CNN
 F 3 "" H 6000 3900 50  0001 C CNN
 	1    6000 3900
 	0    1    1    0
 $EndComp
-Wire Wire Line
-	5250 4350 5250 4525
-Wire Wire Line
-	5250 4825 5250 4675
 Wire Wire Line
 	5450 4825 5375 4825
@@
 F 0 "C?" V 5900 5250 50  0000 L CNN
 F 1 "1000pF" V 6100 5325 50  0000 L CNN
-F 2 "" H 6000 5325 50  0001 C CNN
+F 2 "Capacitors_SMD:C_1206_HandSoldering" H 6000 5325 50  0001 C CNN
 F 3 "" H 6000 5325 50  0001 C CNN
 	1    6000 5325
@@
 F 0 "C?" V 5900 3325 50  0000 L CNN
 F 1 "1000pF" V 6100 3400 50  0000 L CNN
-F 2 "" H 6000 3400 50  0001 C CNN
+F 2 "Capacitors_SMD:C_1206_HandSoldering" H 6000 3400 50  0001 C CNN
 F 3 "" H 6000 3400 50  0001 C CNN
 	1    6000 3400
@@
 F 0 "C?" V 5900 1850 50  0000 L CNN
 F 1 "1000pF" V 6100 1925 50  0000 L CNN
-F 2 "" H 6000 1925 50  0001 C CNN
+F 2 "Capacitors_SMD:C_1206_HandSoldering" H 6000 1925 50  0001 C CNN
 F 3 "" H 6000 1925 50  0001 C CNN
 	1    6000 1925
@@
 F 0 "C?" H 4335 2670 50  0000 L CNN
 F 1 "6.8uF" H 4335 2520 50  0000 L CNN
-F 2 "" H 4325 2600 50  0001 C CNN
+F 2 "Capacitors_SMD:C_1812_HandSoldering" H 4325 2600 50  0001 C CNN
 F 3 "" H 4325 2600 50  0001 C CNN
 	1    4325 2600
-	1    0    0    -1
-$EndComp
-$Comp
-L GND #PWR?
-U 1 1 5B576777
-P 4325 2775
-F 0 "#PWR?" H 4325 2525 60  0001 C CNN
-F 1 "GND" H 4325 2625 60  0000 C CNN
-F 2 "" H 4325 2775 60  0000 C CNN
-F 3 "" H 4325 2775 60  0000 C CNN
-	1    4325 2775
 	1    0    0    -1
 $EndComp
@@
 F 0 "C?" H 4835 2670 50  0000 L CNN
 F 1 "6.8uF" H 4835 2520 50  0000 L CNN
-F 2 "" H 4825 2600 50  0001 C CNN
+F 2 "Capacitors_SMD:C_1812_HandSoldering" H 4825 2600 50  0001 C CNN
 F 3 "" H 4825 2600 50  0001 C CNN
 	1    4825 2600
@@
 	4825 2375 4825 2500
 Connection ~ 4825 2375
-$Comp
-L GND #PWR?
-U 1 1 5B577B5F
-P 4825 2775
-F 0 "#PWR?" H 4825 2525 60  0001 C CNN
-F 1 "GND" H 4825 2625 60  0000 C CNN
-F 2 "" H 4825 2775 60  0000 C CNN
-F 3 "" H 4825 2775 60  0000 C CNN
-	1    4825 2775
-	1    0    0    -1
-$EndComp
 Wire Wire Line
 	4825 2775 4825 2700
-Wire Wire Line
-	5250 2525 5450 2525
-Wire Wire Line
-	5250 2525 5250 2825
 Wire Wire Line
 	5900 3400 5375 3400
@@
 Text HLabel 8100 4525 2    60   UnSpc ~ 0
 +5V
+$Comp
+L GNDPWR #PWR?
+U 1 1 5B5D1EF8
+P 4325 2775
+F 0 "#PWR?" H 4325 2575 50  0001 C CNN
+F 1 "GNDPWR" H 4325 2645 50  0000 C CNN
+F 2 "" H 4325 2725 50  0001 C CNN
+F 3 "" H 4325 2725 50  0001 C CNN
+	1    4325 2775
+	1    0    0    -1
+$EndComp
+$Comp
+L GNDPWR #PWR?
+U 1 1 5B5D205A
+P 4825 2775
+F 0 "#PWR?" H 4825 2575 50  0001 C CNN
+F 1 "GNDPWR" H 4825 2645 50  0000 C CNN
+F 2 "" H 4825 2725 50  0001 C CNN
+F 3 "" H 4825 2725 50  0001 C CNN
+	1    4825 2775
+	1    0    0    -1
+$EndComp
+$Comp
+L GNDPWR #PWR?
+U 1 1 5B5D2095
+P 5200 2850
+F 0 "#PWR?" H 5200 2650 50  0001 C CNN
+F 1 "GNDPWR" H 5200 2720 50  0000 C CNN
+F 2 "" H 5200 2800 50  0001 C CNN
+F 3 "" H 5200 2800 50  0001 C CNN
+	1    5200 2850
+	1    0    0    -1
+$EndComp
+Wire Wire Line
+	5200 2850 5200 2525
+Wire Wire Line
+	5200 2525 5450 2525
+$Comp
+L GNDPWR #PWR?
+U 1 1 5B5D3A17
+P 5225 4825
+F 0 "#PWR?" H 5225 4625 50  0001 C CNN
+F 1 "GNDPWR" H 5225 4695 50  0000 C CNN
+F 2 "" H 5225 4775 50  0001 C CNN
+F 3 "" H 5225 4775 50  0001 C CNN
+	1    5225 4825
+	1    0    0    -1
+$EndComp
+Wire Wire Line
+	5225 4675 5225 4825
+Wire Wire Line
+	5225 4350 5225 4525
+$Comp
+L GNDPWR #PWR?
+U 1 1 5B5D410B
+P 4225 5375
+F 0 "#PWR?" H 4225 5175 50  0001 C CNN
+F 1 "GNDPWR" H 4225 5245 50  0000 C CNN
+F 2 "" H 4225 5325 50  0001 C CNN
+F 3 "" H 4225 5325 50  0001 C CNN
+	1    4225 5375
+	1    0    0    -1
+$EndComp
 $EndSCHEMATC

Commit message: Thruster_SW3 could be controlled
Connections:
- net labels added: +PWR
- net labels removed: +VBatt
Changed lines of the file:
@@
 $Descr A4 11693 8268
 encoding utf-8
-Sheet 6 11
+Sheet 4 11
 Title "Power Voltage Convertor"
 Date "2017-04-06"
@@
 $EndComp
 Text HLabel 3875 2375 0    60   UnSpc ~ 0
-+VBatt
++PWR
 $Comp
 L +BATT #PWR039

Commit message: Power_dist could be monitor battery voltage and system current
Parts:
- L1: renamed from L?; footprint (none) -> Inductors_SMD:L_Vishay_IHLP-2525
- gave numbers to parts that had none: 6
- renumbered D11 to D13, JP1 to JP2, P4 to P5, P5 to P6, R31 to R23, R30 to R24, U7 to U3, U8 to U4
Changed lines of the file:
@@
 $EndDescr
 $Comp
-L R R30
+L R R24
 U 1 1 58C85083
 P 7050 2575
-F 0 "R30" V 7130 2575 40  0000 C CNN
+F 0 "R24" V 7130 2575 40  0000 C CNN
 F 1 "1k" V 7057 2576 40  0000 C CNN
 F 2 "Resistors_SMD:R_0603_HandSoldering" V 6980 2575 30  0001 C CNN
@@
 $EndComp
 $Comp
-L LED_Small D11
+L LED_Small D13
 U 1 1 58C85089
 P 7050 2825
-F 0 "D11" H 7000 2950 50  0000 L CNN
+F 0 "D13" H 7000 2950 50  0000 L CNN
 F 1 "+12V_LED" H 6875 2725 50  0000 L CNN
 F 2 "LEDs:LED_0603_HandSoldering" V 7050 2825 60  0001 C CNN
@@
 $EndComp
 $Comp
-L R R31
+L R R23
 U 1 1 58C85236
 P 7025 4700
-F 0 "R31" V 7105 4700 40  0000 C CNN
+F 0 "R23" V 7105 4700 40  0000 C CNN
 F 1 "1k" V 7032 4701 40  0000 C CNN
 F 2 "Resistors_SMD:R_0603_HandSoldering" V 6955 4700 30  0001 C CNN
@@
 $EndComp
 $Comp
-L TEN_20-2411WIN U8
+L TEN_20-2411WIN U4
 U 1 1 58C8526A
 P 6000 4675
-F 0 "U8" H 6000 5112 60  0000 C CNN
+F 0 "U4" H 6000 5112 60  0000 C CNN
 F 1 "TEN_20-2411WIN" H 6000 5006 60  0000 C CNN
 F 2 "zeabus:TEN_20WIN" H 6050 4575 60  0001 C CNN
@@
 +PWR
 $Comp
-L +BATT #PWR039
+L +BATT #PWR48
 U 1 1 58C81568
 P 4100 2200
-F 0 "#PWR039" H 4100 2050 50  0001 C CNN
+F 0 "#PWR48" H 4100 2050 50  0001 C CNN
 F 1 "+BATT" H 4100 2340 50  0000 C CNN
 F 2 "" H 4100 2200 50  0000 C CNN
@@
 $EndComp
 $Comp
-L Jumper JP1
+L Jumper JP2
 U 1 1 58C8A24F
 P 4625 5175
-F 0 "JP1" H 4625 5325 50  0000 C CNN
+F 0 "JP2" H 4625 5325 50  0000 C CNN
 F 1 "Main_Switch_(N.O.)" H 4625 5095 50  0000 C CNN
 F 2 "Pin_Headers:Pin_Header_Straight_1x02_Pitch2.54mm" H 4625 5175 60  0001 C CNN
@@
 $EndComp
 $Comp
-L +BATT #PWR041
+L +BATT #PWR53
 U 1 1 58C8C536
 P 5225 4350
-F 0 "#PWR041" H 5225 4200 50  0001 C CNN
+F 0 "#PWR53" H 5225 4200 50  0001 C CNN
 F 1 "+BATT" H 5225 4490 50  0000 C CNN
 F 2 "" H 5225 4350 50  0000 C CNN
@@
 	7400 2725 7400 3075
 $Comp
-L +12V #PWR042
+L +12V #PWR55
 U 1 1 5A370E35
 P 7400 2200
-F 0 "#PWR042" H 7400 2050 50  0001 C CNN
+F 0 "#PWR55" H 7400 2050 50  0001 C CNN
 F 1 "+12V" H 7400 2340 50  0000 C CNN
 F 2 "" H 7400 2200 50  0001 C CNN
@@
 $EndComp
 $Comp
-L +5V #PWR043
+L +5V #PWR57
 U 1 1 5A370FF9
 P 7400 4350
-F 0 "#PWR043" H 7400 4200 50  0001 C CNN
+F 0 "#PWR57" H 7400 4200 50  0001 C CNN
 F 1 "+5V" H 7400 4490 50  0000 C CNN
 F 2 "" H 7400 4350 50  0001 C CNN
@@
 	7400 4875 7400 5125
 $Comp
-L GNDREF #PWR044
+L GNDREF #PWR56
 U 1 1 5A373347
 P 7400 3075
-F 0 "#PWR044" H 7400 2825 50  0001 C CNN
+F 0 "#PWR56" H 7400 2825 50  0001 C CNN
 F 1 "GNDREF" H 7400 2925 50  0000 C CNN
 F 2 "" H 7400 3075 50  0001 C CNN
@@
 $EndComp
 $Comp
-L GNDREF #PWR045
+L GNDREF #PWR58
 U 1 1 5A37353E
 P 7400 5125
-F 0 "#PWR045" H 7400 4875 50  0001 C CNN
+F 0 "#PWR58" H 7400 4875 50  0001 C CNN
 F 1 "GNDREF" H 7400 4975 50  0000 C CNN
 F 2 "" H 7400 5125 50  0001 C CNN
@@
 $EndComp
 $Comp
-L XT30 P4
+L XT30 P5
 U 1 1 5A3A2D2C
 P 7600 2675
-F 0 "P4" H 7600 2825 50  0000 C CNN
+F 0 "P5" H 7600 2825 50  0000 C CNN
 F 1 "+12V" H 7600 2525 50  0000 C CNN
 F 2 "zeabus:XT30" H 7600 2675 60  0001 C CNN
@@
 Connection ~ 7400 2975
 $Comp
-L XT30 P5
+L XT30 P6
 U 1 1 5A3A2E02
 P 7600 4825
-F 0 "P5" H 7600 4975 50  0000 C CNN
+F 0 "P6" H 7600 4975 50  0000 C CNN
 F 1 "+5V" H 7600 4675 50  0000 C CNN
 F 2 "zeabus:XT30" H 7600 4825 60  0001 C CNN
@@
 Connection ~ 7400 5075
 $Comp
-L UWE-12/6-Q12P U7
+L UWE-12/6-Q12P U3
 U 1 1 58C85071
 P 6000 2675
-F 0 "U7" H 5700 3075 60  0000 C CNN
+F 0 "U3" H 5700 3075 60  0000 C CNN
 F 1 "UWE-12/6-Q12P" H 6000 2275 60  0000 C CNN
 F 2 "zeabus:UWE-xxxx" H 6050 2375 60  0001 C CNN
@@
 Connection ~ 7025 5075
 $Comp
-L C_Small C?
+L C_Small C12
 U 1 1 5B56CC57
 P 6000 3900
-F 0 "C?" V 5900 3825 50  0000 L CNN
+F 0 "C12" V 5900 3825 50  0000 L CNN
 F 1 "1000pF" V 6100 3900 50  0000 L CNN
 F 2 "Capacitors_SMD:C_1206_HandSoldering" H 6000 3900 50  0001 C CNN
@@
 Connection ~ 6600 4525
 $Comp
-L C_Small C?
+L C_Small C13
 U 1 1 5B56F67E
 P 6000 5325
-F 0 "C?" V 5900 5250 50  0000 L CNN
+F 0 "C13" V 5900 5250 50  0000 L CNN
 F 1 "1000pF" V 6100 5325 50  0000 L CNN
 F 2 "Capacitors_SMD:C_1206_HandSoldering" H 6000 5325 50  0001 C CNN
@@
 $EndComp
 $Comp
-L C_Small C?
+L C_Small C11
 U 1 1 5B5708E4
 P 6000 3400
-F 0 "C?" V 5900 3325 50  0000 L CNN
+F 0 "C11" V 5900 3325 50  0000 L CNN
 F 1 "1000pF" V 6100 3400 50  0000 L CNN
 F 2 "Capacitors_SMD:C_1206_HandSoldering" H 6000 3400 50  0001 C CNN
@@
 $EndComp
 $Comp
-L C_Small C?
+L C_Small C10
 U 1 1 5B570CAE
 P 6000 1925
-F 0 "C?" V 5900 1850 50  0000 L CNN
+F 0 "C10" V 5900 1850 50  0000 L CNN
 F 1 "1000pF" V 6100 1925 50  0000 L CNN
 F 2 "Capacitors_SMD:C_1206_HandSoldering" H 6000 1925 50  0001 C CNN
@@
 Connection ~ 4100 2375
 $Comp
-L C_Small C?
+L C_Small C8
 U 1 1 5B575A61
 P 4325 2600
-F 0 "C?" H 4335 2670 50  0000 L CNN
+F 0 "C8" H 4335 2670 50  0000 L CNN
 F 1 "6.8uF" H 4335 2520 50  0000 L CNN
 F 2 "Capacitors_SMD:C_1812_HandSoldering" H 4325 2600 50  0001 C CNN
@@
 Connection ~ 4325 2375
 $Comp
-L C_Small C?
+L C_Small C9
 U 1 1 5B5777FB
 P 4825 2600
-F 0 "C?" H 4835 2670 50  0000 L CNN
+F 0 "C9" H 4835 2670 50  0000 L CNN
 F 1 "6.8uF" H 4835 2520 50  0000 L CNN
 F 2 "Capacitors_SMD:C_1812_HandSoldering" H 4825 2600 50  0001 C CNN
@@
 Connection ~ 5375 2375
 $Comp
-L L L?
+L L L1
 U 1 1 5B57BC45
 P 4575 2375
-F 0 "L?" V 4675 2375 50  0000 C CNN
+F 0 "L1" V 4675 2375 50  0000 C CNN
 F 1 "3.3uF" V 4500 2375 50  0000 C CNN
-F 2 "" H 4575 2375 50  0001 C CNN
+F 2 "Inductors_SMD:L_Vishay_IHLP-2525" H 4575 2375 50  0001 C CNN
 F 3 "" H 4575 2375 50  0001 C CNN
 	1    4575 2375
@@
 +5V
 $Comp
-L GNDPWR #PWR?
+L GNDPWR #PWR50
 U 1 1 5B5D1EF8
 P 4325 2775
-F 0 "#PWR?" H 4325 2575 50  0001 C CNN
+F 0 "#PWR50" H 4325 2575 50  0001 C CNN
 F 1 "GNDPWR" H 4325 2645 50  0000 C CNN
 F 2 "" H 4325 2725 50  0001 C CNN
@@
 $EndComp
 $Comp
-L GNDPWR #PWR?
+L GNDPWR #PWR51
 U 1 1 5B5D205A
 P 4825 2775
-F 0 "#PWR?" H 4825 2575 50  0001 C CNN
+F 0 "#PWR51" H 4825 2575 50  0001 C CNN
 F 1 "GNDPWR" H 4825 2645 50  0000 C CNN
 F 2 "" H 4825 2725 50  0001 C CNN
@@
 $EndComp
 $Comp
-L GNDPWR #PWR?
+L GNDPWR #PWR52
 U 1 1 5B5D2095
 P 5200 2850
-F 0 "#PWR?" H 5200 2650 50  0001 C CNN
+F 0 "#PWR52" H 5200 2650 50  0001 C CNN
 F 1 "GNDPWR" H 5200 2720 50  0000 C CNN
 F 2 "" H 5200 2800 50  0001 C CNN
@@
 	5200 2525 5450 2525
 $Comp
-L GNDPWR #PWR?
+L GNDPWR #PWR54
 U 1 1 5B5D3A17
 P 5225 4825
-F 0 "#PWR?" H 5225 4625 50  0001 C CNN
+F 0 "#PWR54" H 5225 4625 50  0001 C CNN
 F 1 "GNDPWR" H 5225 4695 50  0000 C CNN
 F 2 "" H 5225 4775 50  0001 C CNN
@@
 	5225 4350 5225 4525
 $Comp
-L GNDPWR #PWR?
+L GNDPWR #PWR49
 U 1 1 5B5D410B
 P 4225 5375
-F 0 "#PWR?" H 4225 5175 50  0001 C CNN
+F 0 "#PWR49" H 4225 5175 50  0001 C CNN
 F 1 "GNDPWR" H 4225 5245 50  0000 C CNN
 F 2 "" H 4225 5325 50  0001 C CNN
