File: Circuit/Power_dist/Power_Distributor.sch (KiCad schematic (older format))
At the start: 1 part, among them J1 Thruster_Off_Switch

Commit message: Merge commit '3eda1dba5ca6e598d51cb20764784284330d387d'
Parts:
- added CON1: Conn-PCIE-x16, zeabus:pcie-x16-edge, symbol Conn-PCIE-x16
- added D7: LED_Small, LEDs:LED_0603_HandSoldering, symbol LED_Small
- added R10: 1k, Resistors_SMD:R_0603_HandSoldering, symbol R
- J1: footprint Socket_Strips:Socket_Strip_Straight_1x02_Pitch2.54mm -> Pin_Headers:Pin_Header_Straight_1x02_Pitch2.54mm; symbol CONN_01X02 -> Conn_01x02
Connections:
- net +BATT: now also CON1.A3 (V12)
- net GND: now also CON1.B7 (GND)
- new net: D7.1 (K), R10.1
- new net +12V: CON1.A2 (V12), CON1.B1 (V12), CON1.B2 (V12), CON1.B3 (V12)
- new net +5V: CON1.A10 (VCC3), CON1.A9 (VCC3), CON1.B8 (VCC3)
- new net D+: CON1.B14 (HSO0+)
- new net D-: CON1.B15 (HSO0-)
- new net GNDD: CON1.B16 (GND), R10.2
- new net GNDREF: CON1.A12 (GND), CON1.A15 (GND), CON1.A18 (GND), CON1.A4 (GND), CON1.B13 (GND), CON1.B18 (GND), CON1.B4 (GND)
- new net VBUS: CON1.B10 (3VSB), D7.2 (A)
- no-connect marks 2 -> 0
