File: Circuit/Power_dist/Power_Distributor.sch (KiCad schematic (older format))
At the start: 18 parts, among them CON1 Conn-PCIE-x16, P16 BATT1, P17 BATT2

Commit message: Thruster_SW3 could be controlled
Connections:
- wire segments 103 -> 108
Changed lines of the file:
@@
 $EndDescr
 $Sheet
-S 4550 3650 900  400
+S 4550 4175 900  400
 U 58E52973
 F0 "Thruster_SW2" 60
 F1 "Thruster_Switch.sch" 60
-F2 "+PWR" U R 5450 3750 60
-F3 "Software_SW" U R 5450 3850 60
+F2 "+PWR" U R 5450 4275 60
+F3 "Software_SW" U R 5450 4375 60
 $EndSheet
 $Comp
@@
 $EndComp
 $Sheet
-S 4550 2950 900  400
+S 4550 3475 900  400
 U 58E0048C
 F0 "Thruster_SW1" 60
 F1 "Thruster_Switch.sch" 60
-F2 "+PWR" U R 5450 3050 60
-F3 "Software_SW" U R 5450 3150 60
+F2 "+PWR" U R 5450 3575 60
+F3 "Software_SW" U R 5450 3675 60
 $EndSheet
 $Comp
 L +BATT #PWR03
 U 1 1 58EB597A
-P 5750 2950
-F 0 "#PWR03" H 5750 2800 50  0001 C CNN
-F 1 "+BATT" H 5750 3090 50  0000 C CNN
-F 2 "" H 5750 2950 50  0001 C CNN
-F 3 "" H 5750 2950 50  0001 C CNN
-	1    5750 2950
+P 5750 3475
+F 0 "#PWR03" H 5750 3325 50  0001 C CNN
+F 1 "+BATT" H 5750 3615 50  0000 C CNN
+F 2 "" H 5750 3475 50  0001 C CNN
+F 3 "" H 5750 3475 50  0001 C CNN
+	1    5750 3475
 	1    0    0    -1
 $EndComp
@@
 L +BATT #PWR04
 U 1 1 58EB69B2
-P 5750 3650
-F 0 "#PWR04" H 5750 3500 50  0001 C CNN
-F 1 "+BATT" H 5750 3790 50  0000 C CNN
-F 2 "" H 5750 3650 50  0001 C CNN
-F 3 "" H 5750 3650 50  0001 C CNN
-	1    5750 3650
+P 5750 4175
+F 0 "#PWR04" H 5750 4025 50  0001 C CNN
+F 1 "+BATT" H 5750 4315 50  0000 C CNN
+F 2 "" H 5750 4175 50  0001 C CNN
+F 3 "" H 5750 4175 50  0001 C CNN
+	1    5750 4175
 	1    0    0    -1
 $EndComp
@@
 F0 "DC-DC Converter" 60
 F1 "Power-Volt-Converter.sch" 60
-F2 "+VBatt" U L 9150 5075 60
-F3 "+12V" U L 9150 5550 60
-F4 "+5V" U L 9150 5700 60
+F2 "+12V" U L 9150 5550 60
+F3 "+5V" U L 9150 5700 60
+F4 "+PWR" U L 9150 5075 60
 $EndSheet
 $Comp
@@
 Text GLabel 1525 5450 0    60   Input ~ 0
 D-
-$Sheet
-S 6450 2950 1000 3200
-U 58E54EC3
-F0 "Power_Controller" 60
-F1 "Power-Controller.sch" 60
-F2 "SW1_C" I L 6450 3150 60
-F3 "SW2_C" I L 6450 3850 60
-F4 "SW3_C" I L 6450 4550 60
-F5 "SW4_C" I L 6450 5250 60
-F6 "SW1_E" O L 6450 3250 60
-F7 "SW2_E" O L 6450 3950 60
-F8 "SW3_E" O L 6450 4650 60
-F9 "SW4_E" O L 6450 5350 60
-$EndSheet
 $Sheet
 S 5050 800  1250 750
@@
 L GNDPWR #PWR?
 U 1 1 5B5CB6FC
-P 6250 5450
-F 0 "#PWR?" H 6250 5250 50  0001 C CNN
-F 1 "GNDPWR" H 6250 5320 50  0000 C CNN
-F 2 "" H 6250 5400 50  0001 C CNN
-F 3 "" H 6250 5400 50  0001 C CNN
-	1    6250 5450
+P 6250 5975
+F 0 "#PWR?" H 6250 5775 50  0001 C CNN
+F 1 "GNDPWR" H 6250 5845 50  0000 C CNN
+F 2 "" H 6250 5925 50  0001 C CNN
+F 3 "" H 6250 5925 50  0001 C CNN
+	1    6250 5975
 	1    0    0    -1
 $EndComp
@@
 Text GLabel 9725 2100 0    60   Input ~ 0
 KILL_SWITCH
-Text GLabel 6325 3250 0    60   Input ~ 0
+Text GLabel 6325 3775 0    60   Input ~ 0
 KILL_SWITCH
-Text GLabel 6325 3950 0    60   Input ~ 0
+Text GLabel 6325 4475 0    60   Input ~ 0
 KILL_SWITCH
 $Comp
 L +BATT #PWR?
 U 1 1 5B536166
-P 5750 5050
-F 0 "#PWR?" H 5750 4900 50  0001 C CNN
-F 1 "+BATT" H 5750 5190 50  0000 C CNN
-F 2 "" H 5750 5050 50  0001 C CNN
-F 3 "" H 5750 5050 50  0001 C CNN
-	1    5750 5050
+P 5750 5575
+F 0 "#PWR?" H 5750 5425 50  0001 C CNN
+F 1 "+BATT" H 5750 5715 50  0000 C CNN
+F 2 "" H 5750 5575 50  0001 C CNN
+F 3 "" H 5750 5575 50  0001 C CNN
+	1    5750 5575
 	-1   0    0    -1
 $EndComp
 $Sheet
-S 4550 4350 900  400
+S 4550 4875 900  400
 U 5B53D7CB
 F0 "Thruster_SW3" 60
 F1 "Thruster_Switch.sch" 60
-F2 "+PWR" U R 5450 4450 60
-F3 "Software_SW" U R 5450 4550 60
+F2 "+PWR" U R 5450 4975 60
+F3 "Software_SW" U R 5450 5075 60
 $EndSheet
 $Comp
 L +BATT #PWR?
 U 1 1 5B54246D
-P 5750 4350
-F 0 "#PWR?" H 5750 4200 50  0001 C CNN
-F 1 "+BATT" H 5750 4490 50  0000 C CNN
-F 2 "" H 5750 4350 50  0001 C CNN
-F 3 "" H 5750 4350 50  0001 C CNN
-	1    5750 4350
-	1    0    0    -1
-$EndComp
-Text GLabel 6325 4650 0    60   Input ~ 0
+P 5750 4875
+F 0 "#PWR?" H 5750 4725 50  0001 C CNN
+F 1 "+BATT" H 5750 5015 50  0000 C CNN
+F 2 "" H 5750 4875 50  0001 C CNN
+F 3 "" H 5750 4875 50  0001 C CNN
+	1    5750 4875
+	1    0    0    -1
+$EndComp
+Text GLabel 6325 5175 0    60   Input ~ 0
 KILL_SWITCH
 Wire Wire Line
-	5450 3750 5750 3750
-Wire Wire Line
-	5450 3850 6450 3850
-Wire Wire Line
-	6450 3150 5450 3150
+	5450 4275 5750 4275
+Wire Wire Line
+	5450 4375 6450 4375
+Wire Wire Line
+	6450 3675 5450 3675
 Wire Wire Line
 	2025 5450 1525 5450
@@
 	8350 1825 8350 1725
 Wire Wire Line
-	6250 5450 6250 5350
+	6250 5975 6250 5875
 Wire Wire Line
 	1875 3825 1875 4150
@@
 	10600 2100 10600 2325
 Wire Wire Line
-	6325 3250 6450 3250
-Wire Wire Line
-	6325 3950 6450 3950
-Wire Wire Line
-	5450 4450 5750 4450
-Wire Wire Line
-	6450 4550 5450 4550
-Wire Wire Line
-	6325 4650 6450 4650
-Wire Wire Line
-	5750 3750 5750 3650
-Wire Wire Line
-	5750 3050 5450 3050
-Wire Wire Line
-	5750 3050 5750 2950
-Wire Wire Line
-	5750 4450 5750 4350
+	6325 3775 6450 3775
+Wire Wire Line
+	6325 4475 6450 4475
+Wire Wire Line
+	5450 4975 5750 4975
+Wire Wire Line
+	6450 5075 5450 5075
+Wire Wire Line
+	6325 5175 6450 5175
+Wire Wire Line
+	5750 4275 5750 4175
+Wire Wire Line
+	5750 3575 5450 3575
+Wire Wire Line
+	5750 3575 5750 3475
+Wire Wire Line
+	5750 4975 5750 4875
 $Sheet
-S 4550 5050 900  400
+S 4550 5575 900  400
 U 58E51F99
 F0 "DVL_SW" 60
 F1 "Power_Switch_VBatt.sch" 60
-F2 "+PWR" U R 5450 5150 60
-F3 "Software_SW" U R 5450 5250 60
+F2 "+PWR" U R 5450 5675 60
+F3 "Software_SW" U R 5450 5775 60
 $EndSheet
 Wire Wire Line
-	5450 5250 6450 5250
-Wire Wire Line
-	5450 5150 5750 5150
-Wire Wire Line
-	5750 5150 5750 5050
-Wire Wire Line
-	6250 5350 6450 5350
+	5450 5775 6450 5775
+Wire Wire Line
+	5450 5675 5750 5675
+Wire Wire Line
+	5750 5675 5750 5575
+Wire Wire Line
+	6250 5875 6450 5875
 $Sheet
-S 8450 2950 900  400
+S 8450 3475 900  400
 U 5B530A41
 F0 "Imaging_Sonar" 60
 F1 "Power_Switch_VBatt.sch" 60
-F2 "+PWR" U L 8450 3050 60
-F3 "Software_SW" U L 8450 3150 60
+F2 "+PWR" U L 8450 3575 60
+F3 "Software_SW" U L 8450 3675 60
 $EndSheet
 Wire Wire Line
-	8450 3050 8150 3050
+	8450 3575 8150 3575
 $Comp
 L +BATT #PWR?
 U 1 1 5B53EA2A
-P 8150 2950
-F 0 "#PWR?" H 8150 2800 50  0001 C CNN
-F 1 "+BATT" H 8150 3090 50  0000 C CNN
-F 2 "" H 8150 2950 50  0001 C CNN
-F 3 "" H 8150 2950 50  0001 C CNN
-	1    8150 2950
-	1    0    0    -1
-$EndComp
-Wire Wire Line
-	8150 3050 8150 2950
+P 8150 3475
+F 0 "#PWR?" H 8150 3325 50  0001 C CNN
+F 1 "+BATT" H 8150 3615 50  0000 C CNN
+F 2 "" H 8150 3475 50  0001 C CNN
+F 3 "" H 8150 3475 50  0001 C CNN
+	1    8150 3475
+	1    0    0    -1
+$EndComp
+Wire Wire Line
+	8150 3575 8150 3475
+Wire Wire Line
+	8450 3675 7450 3675
+$Comp
+L GNDPWR #PWR?
+U 1 1 5B5F781B
+P 7675 3875
+F 0 "#PWR?" H 7675 3675 50  0001 C CNN
+F 1 "GNDPWR" H 7675 3745 50  0000 C CNN
+F 2 "" H 7675 3825 50  0001 C CNN
+F 3 "" H 7675 3825 50  0001 C CNN
+	1    7675 3875
+	-1   0    0    -1
+$EndComp
+Wire Wire Line
+	7675 3875 7675 3775
+Wire Wire Line
+	7675 3775 7450 3775
+$Sheet
+S 6450 2950 1000 3200
+U 58E54EC3
+F0 "Power_Controller" 60
+F1 "Power-Controller.sch" 60
+F2 "+PWR" U L 6450 3150 60
+F3 "SW5_C" U R 7450 3675 60
+F4 "SW5_E" U R 7450 3775 60
+F5 "SW1_C" U L 6450 3675 60
+F6 "SW2_C" U L 6450 4375 60
+F7 "SW3_C" U L 6450 5075 60
+F8 "SW4_C" U L 6450 5775 60
+F9 "SW1_E" U L 6450 3775 60
+F10 "SW2_E" U L 6450 4475 60
+F11 "SW3_E" U L 6450 5175 60
+F12 "SW4_E" U L 6450 5875 60
+$EndSheet
+Wire Wire Line
+	6450 3150 6150 3150
+$Comp
+L +BATT #PWR?
+U 1 1 5B61FF32
+P 6150 3050
+F 0 "#PWR?" H 6150 2900 50  0001 C CNN
+F 1 "+BATT" H 6150 3190 50  0000 C CNN
+F 2 "" H 6150 3050 50  0001 C CNN
+F 3 "" H 6150 3050 50  0001 C CNN
+	1    6150 3050
+	1    0    0    -1
+$EndComp
+Wire Wire Line
+	6150 3150 6150 3050
 $EndSCHEMATC

Commit message: changed +5V voltage regulator on battery side of Power_dist to L78
Parts:
- removed U?: L78L05_SOT89, TO_SOT_Packages_SMD:SOT89-3_Housing, symbol L78L05_SOT89
- added U?: L7805, TO_SOT_Packages_SMD:TO-263-2, symbol L7805
Changed lines of the file:
@@
-$EndComp
-$Comp
-L L78L05_SOT89 U?
-U 1 1 5B4F178E
-P 10150 1000
-F 0 "U?" H 10000 1125 50  0000 C CNN
-F 1 "L78L05_SOT89" H 10150 1125 50  0000 L CNN
-F 2 "TO_SOT_Packages_SMD:SOT89-3_Housing" H 10150 1200 50  0001 C CIN
-F 3 "" H 10150 950 50  0001 C CNN
-	1    10150 1000
-	1    0    0    -1
 $EndComp
 $Comp
@@
 Wire Wire Line
 	6150 3150 6150 3050
+$Comp
+L L7805 U?
+U 1 1 5B5077FE
+P 10150 1000
+F 0 "U?" H 10000 1125 50  0000 C CNN
+F 1 "L7805" H 10150 1125 50  0000 L CNN
+F 2 "TO_SOT_Packages_SMD:TO-263-2" H 10175 850 50  0001 L CIN
+F 3 "" H 10150 950 50  0001 C CNN
+	1    10150 1000
+	1    0    0    -1
+$EndComp
 $EndSCHEMATC

Commit message: power line and data line source of Power_Controller on Power_dist could be manual selected
Parts:
- added C?: 0.1uF, Capacitors_SMD:C_0603_HandSoldering, symbol C_Small
- added D?: +5V_USB_LED, LEDs:LED_0603_HandSoldering, symbol LED_Small
- added J?: USB_B, Connectors:USB_Mini-B, symbol USB_OTG
- added J?: PWR_CTRL_PWR_SRC_SEL, Pin_Headers:Pin_Header_Straight_1x03_Pitch2.54mm, symbol Conn_01x03_Selection_Source
- added J?: PWR_CTRL_DATA_SRC_SEL, Pin_Headers:Pin_Header_Straight_1x03_Pitch2.54mm, symbol Conn_01x03_Selection_Source
- added R?: 1k, Resistors_SMD:R_0603_HandSoldering, symbol R
- added R?: 50, Resistors_SMD:R_0603_HandSoldering, symbol R
- added R?: 100, Resistors_SMD:R_0603_HandSoldering, symbol R
- added U?: FSUSB30, Housings_SSOP:MSOP-10_3x3mm_Pitch0.5mm, symbol FSUSB30
- D7: value VBUS_LED -> +5V_PCIE_LED
- R29, R?: footprint (none) -> Resistors_SMD:R_0603_HandSoldering
Connections:
- net labels added: +3V3_CTRL, +5V_CTRL, +5V_PCIE, +5V_USB, D+_CTRL, D+_PCIE, D+_USB, D-_CTRL, D-_PCIE, D-_USB
- net labels removed: D+, D-, VBUS
- wire segments 108 -> 147
- no-connect marks 0 -> 44
Other:
- moved on the sheet: CON1A, D7, P16, P17, R10, R11, R12, R29, R?
