File: Circuit/Power_dist/Power_Switch_VBatt.sch (KiCad schematic (older format))
At the start: 8 parts, among them P5 XT60, Q2 IPD90P03P4L

Commit message: Merge commit '3eda1dba5ca6e598d51cb20764784284330d387d'
Parts:
- removed P5: XT60, zeabus:XT60, symbol XT60
- added P2: XT30, zeabus:XT30, symbol XT30
- D4: footprint LEDs:LED_0603 -> LEDs:LED_0603_HandSoldering
- F2: footprint Zeabus:FUSE_AUTO -> zeabus:FUSE_AUTO
- Q2: footprint TO_SOT_Packages_SMD:TO-252-2Lead -> TO_SOT_Packages_SMD:TO-252-2
Connections:
- net GND: now also P2.2 (P2)
- net at F2.2, R6.2: now also P2.1 (P1)
Changed lines of the file:
@@
 EESchema Schematic File Version 2
+LIBS:Power_Distributor-rescue
 LIBS:power
 LIBS:device
@@
 LIBS:zeabus
 LIBS:ftdi
+LIBS:Power_Distributor-cache
 EELAYER 25 0
 EELAYER END
 $Descr A4 11693 8268
 encoding utf-8
-Sheet 3 9
+Sheet 3 8
 Title "DVL and Sonar Switch"
 Date "2017-04-06"
@@
 AR Path="/58E51F99/58E52089" Ref="Q2"  Part="1"
 AR Path="/58E527AF/58E52089" Ref="Q3"  Part="1"
-F 0 "Q3" H 6550 3350 50  0000 L CNN
+F 0 "Q2" H 6550 3350 50  0000 L CNN
 F 1 "IPD90P03P4L" H 6550 3250 50  0000 L CNN
-F 2 "TO_SOT_Packages_SMD:TO-252-2Lead" H 6550 3400 50  0001 C CNN
+F 2 "TO_SOT_Packages_SMD:TO-252-2" H 6550 3400 50  0001 C CNN
 F 3 "" H 6350 3300 50  0001 C CNN
 	1    6350 3300
@@
 AR Path="/58E51F99/58E5219E" Ref="R5"  Part="1"
 AR Path="/58E527AF/58E5219E" Ref="R8"  Part="1"
-F 0 "R8" V 5930 3300 50  0000 C CNN
+F 0 "R5" V 5930 3300 50  0000 C CNN
 F 1 "2.2k" V 5850 3300 50  0000 C CNN
 F 2 "Resistors_SMD:R_0603" V 5780 3300 50  0001 C CNN
@@
 $EndComp
 $Comp
-L XT60 P5
-U 1 1 58E521F9
-P 7050 4250
-AR Path="/58E51F99/58E521F9" Ref="P5"  Part="1"
-AR Path="/58E527AF/58E521F9" Ref="P6"  Part="1"
-F 0 "P6" H 7050 4400 50  0000 C CNN
-F 1 "XT60" H 7050 4100 50  0000 C CNN
-F 2 "zeabus:XT60" H 7150 4000 60  0001 C CNN
-F 3 "" H 7050 4250 60  0000 C CNN
-	1    7050 4250
-	1    0    0    -1
-$EndComp
-$Comp
 L LED_Small D4
 U 1 1 58E52234
@@
 AR Path="/58E51F99/58E52234" Ref="D4"  Part="1"
 AR Path="/58E527AF/58E52234" Ref="D6"  Part="1"
-F 0 "D6" H 6400 4675 50  0000 L CNN
+F 0 "D4" H 6400 4675 50  0000 L CNN
 F 1 "LED_Small" H 6275 4450 50  0000 L CNN
-F 2 "LEDs:LED_0603" V 6450 4550 50  0001 C CNN
+F 2 "LEDs:LED_0603_HandSoldering" V 6450 4550 50  0001 C CNN
 F 3 "" V 6450 4550 50  0001 C CNN
 	1    6450 4550
@@
 AR Path="/58E51F99/58E5234D" Ref="R4"  Part="1"
 AR Path="/58E527AF/58E5234D" Ref="R7"  Part="1"
-F 0 "R7" V 5930 2700 50  0000 C CNN
+F 0 "R4" V 5930 2700 50  0000 C CNN
 F 1 "10k" V 5850 2700 50  0000 C CNN
 F 2 "Resistors_SMD:R_0603" V 5780 2700 50  0001 C CNN
@@
 AR Path="/58E51F99/58E52389" Ref="R6"  Part="1"
 AR Path="/58E527AF/58E52389" Ref="R9"  Part="1"
-F 0 "R9" V 6530 4150 50  0000 C CNN
+F 0 "R6" V 6530 4150 50  0000 C CNN
 F 1 "10k" V 6450 4150 50  0000 C CNN
 F 2 "Resistors_SMD:R_0603" V 6380 4150 50  0001 C CNN
@@
 $EndComp
 $Comp
-L GND #PWR012
+L GND #PWR027
 U 1 1 58E527F8
 P 6450 4950
-AR Path="/58E51F99/58E527F8" Ref="#PWR012"  Part="1"
-AR Path="/58E527AF/58E527F8" Ref="#PWR013"  Part="1"
-F 0 "#PWR013" H 6450 4700 50  0001 C CNN
+AR Path="/58E51F99/58E527F8" Ref="#PWR027"  Part="1"
+AR Path="/58E527AF/58E527F8" Ref="#PWR028"  Part="1"
+F 0 "#PWR027" H 6450 4700 50  0001 C CNN
 F 1 "GND" H 6450 4800 50  0000 C CNN
 F 2 "" H 6450 4950 50  0001 C CNN
@@
 AR Path="/58E51F99/58E648CE" Ref="D3"  Part="1"
 AR Path="/58E527AF/58E648CE" Ref="D5"  Part="1"
-F 0 "D5" H 6100 3100 50  0000 C CNN
+F 0 "D3" H 6100 3100 50  0000 C CNN
 F 1 "BZX585-C12" H 6100 2900 50  0000 C CNN
 F 2 "Diodes_SMD:D_SOD-523" H 6100 3000 50  0001 C CNN
@@
 AR Path="/58E51F99/58E651FD" Ref="F2"  Part="1"
 AR Path="/58E527AF/58E651FD" Ref="F3"  Part="1"
-F 0 "F3" V 6530 3750 50  0000 C CNN
+F 0 "F2" V 6530 3750 50  0000 C CNN
 F 1 "Fuse" V 6375 3750 50  0000 C CNN
-F 2 "Zeabus:FUSE_AUTO" V 6380 3750 50  0001 C CNN
+F 2 "zeabus:FUSE_AUTO" V 6380 3750 50  0001 C CNN
 F 3 "" H 6450 3750 50  0001 C CNN
 	1    6450 3750
@@
 Wire Wire Line
 	6850 4850 6450 4850
+$Comp
+L XT30 P2
+U 1 1 5A39572B
+P 7050 4250
+AR Path="/58E51F99/5A39572B" Ref="P2"  Part="1"
+AR Path="/58E527AF/5A39572B" Ref="P3"  Part="1"
+F 0 "P2" H 7050 4400 50  0000 C CNN
+F 1 "XT30" H 7050 4100 50  0000 C CNN
+F 2 "zeabus:XT30" H 7050 4250 60  0000 C CNN
+F 3 "" H 7050 4250 60  0000 C CNN
+	1    7050 4250
+	1    0    0    -1
+$EndComp
 $EndSCHEMATC
