File: Circuit/Power_dist/Power_Switch_VBatt.sch (KiCad schematic (older format))
At the start: 8 parts, among them P2 XT30, Q2 IPD90P03P4L

Commit message: refactor Power_dist
Connections:
- net labels added: GNDPWR
- net labels removed: GND
Other:
- moved on the sheet: P2
Changed lines of the file:
@@
 	-1   0    0    1
-$EndComp
-$Comp
-L GND #PWR027
-U 1 1 58E527F8
-P 6450 4950
-AR Path="/58E51F99/58E527F8" Ref="#PWR027"  Part="1"
-AR Path="/58E527AF/58E527F8" Ref="#PWR028"  Part="1"
-F 0 "#PWR027" H 6450 4700 50  0001 C CNN
-F 1 "GND" H 6450 4800 50  0000 C CNN
-F 2 "" H 6450 4950 50  0001 C CNN
-F 3 "" H 6450 4950 50  0001 C CNN
-	1    6450 4950
-	1    0    0    -1
 $EndComp
 Text HLabel 3650 2450 0    60   Input ~ 0
@@
 Wire Wire Line
 	6450 4650 6450 4950
-Wire Wire Line
-	6850 4850 6850 4300
 Connection ~ 6450 4850
 Wire Wire Line
 	6450 3950 6850 3950
-Wire Wire Line
-	6850 3950 6850 4200
 Connection ~ 6450 3950
 Wire Wire Line
@@
 L XT30 P2
 U 1 1 5A39572B
-P 7050 4250
+P 7050 4375
 AR Path="/58E51F99/5A39572B" Ref="P2"  Part="1"
 AR Path="/58E527AF/5A39572B" Ref="P3"  Part="1"
-F 0 "P2" H 7050 4400 50  0000 C CNN
-F 1 "XT30" H 7050 4100 50  0000 C CNN
-F 2 "zeabus:XT30" H 7050 4250 60  0000 C CNN
-F 3 "" H 7050 4250 60  0000 C CNN
-	1    7050 4250
+F 0 "P2" H 7050 4525 50  0000 C CNN
+F 1 "XT30" H 7050 4225 50  0000 C CNN
+F 2 "zeabus:XT30" H 7050 4375 60  0001 C CNN
+F 3 "" H 7050 4375 60  0000 C CNN
+	1    7050 4375
 	1    0    0    -1
 $EndComp
+$Comp
+L GNDPWR #PWR?
+U 1 1 5B5DF3EC
+P 6450 4950
+AR Path="/58E51F99/5B5DF3EC" Ref="#PWR?"  Part="1"
+AR Path="/58E527AF/5B5DF3EC" Ref="#PWR?"  Part="1"
+F 0 "#PWR?" H 6450 4750 50  0001 C CNN
+F 1 "GNDPWR" H 6450 4820 50  0000 C CNN
+F 2 "" H 6450 4900 50  0001 C CNN
+F 3 "" H 6450 4900 50  0001 C CNN
+	1    6450 4950
+	1    0    0    -1
+$EndComp
+Wire Wire Line
+	6850 3950 6850 4325
+Wire Wire Line
+	6850 4425 6850 4850
 $EndSCHEMATC

Commit message: changed 12V zener of Power_dist to BZT52c12s
Parts:
- D3: value BZX585-C12 -> BZT52c12s; footprint Diodes_SMD:D_SOD-523 -> Diodes_SMD:D_SOD-323_HandSoldering
Changed lines of the file:
@@
 $Descr A4 11693 8268
 encoding utf-8
-Sheet 3 10
+Sheet 4 10
 Title "DVL and Sonar Switch"
 Date "2017-04-06"
@@
 AR Path="/58E51F99/58E52089" Ref="Q2"  Part="1"
 AR Path="/58E527AF/58E52089" Ref="Q3"  Part="1"
-F 0 "Q2" H 6550 3350 50  0000 L CNN
+F 0 "Q3" H 6550 3350 50  0000 L CNN
 F 1 "IPD90P03P4L" H 6550 3250 50  0000 L CNN
 F 2 "TO_SOT_Packages_SMD:TO-252-2" H 6550 3400 50  0001 C CNN
@@
 AR Path="/58E51F99/58E5219E" Ref="R5"  Part="1"
 AR Path="/58E527AF/58E5219E" Ref="R8"  Part="1"
-F 0 "R5" V 5930 3300 50  0000 C CNN
+F 0 "R8" V 5930 3300 50  0000 C CNN
 F 1 "2.2k" V 5850 3300 50  0000 C CNN
 F 2 "Resistors_SMD:R_0603" V 5780 3300 50  0001 C CNN
@@
 AR Path="/58E51F99/58E52234" Ref="D4"  Part="1"
 AR Path="/58E527AF/58E52234" Ref="D6"  Part="1"
-F 0 "D4" H 6400 4675 50  0000 L CNN
+F 0 "D6" H 6400 4675 50  0000 L CNN
 F 1 "LED_Small" H 6275 4450 50  0000 L CNN
 F 2 "LEDs:LED_0603_HandSoldering" V 6450 4550 50  0001 C CNN
@@
 AR Path="/58E51F99/58E5234D" Ref="R4"  Part="1"
 AR Path="/58E527AF/58E5234D" Ref="R7"  Part="1"
-F 0 "R4" V 5930 2700 50  0000 C CNN
+F 0 "R7" V 5930 2700 50  0000 C CNN
 F 1 "10k" V 5850 2700 50  0000 C CNN
 F 2 "Resistors_SMD:R_0603" V 5780 2700 50  0001 C CNN
@@
 AR Path="/58E51F99/58E52389" Ref="R6"  Part="1"
 AR Path="/58E527AF/58E52389" Ref="R9"  Part="1"
-F 0 "R6" V 6530 4150 50  0000 C CNN
+F 0 "R9" V 6530 4150 50  0000 C CNN
 F 1 "10k" V 6450 4150 50  0000 C CNN
 F 2 "Resistors_SMD:R_0603" V 6380 4150 50  0001 C CNN
@@
 AR Path="/58E51F99/58E648CE" Ref="D3"  Part="1"
 AR Path="/58E527AF/58E648CE" Ref="D5"  Part="1"
-F 0 "D3" H 6100 3100 50  0000 C CNN
-F 1 "BZX585-C12" H 6100 2900 50  0000 C CNN
-F 2 "Diodes_SMD:D_SOD-523" H 6100 3000 50  0001 C CNN
+F 0 "D5" H 6100 3100 50  0000 C CNN
+F 1 "BZT52c12s" H 6100 2900 50  0000 C CNN
+F 2 "Diodes_SMD:D_SOD-323_HandSoldering" H 6100 3000 50  0001 C CNN
 F 3 "" H 6100 3000 50  0001 C CNN
 	1    6100 3000
@@
 AR Path="/58E51F99/58E651FD" Ref="F2"  Part="1"
 AR Path="/58E527AF/58E651FD" Ref="F3"  Part="1"
-F 0 "F2" V 6530 3750 50  0000 C CNN
+F 0 "F3" V 6530 3750 50  0000 C CNN
 F 1 "Fuse" V 6375 3750 50  0000 C CNN
 F 2 "zeabus:FUSE_AUTO" V 6380 3750 50  0001 C CNN
@@
 AR Path="/58E51F99/5A39572B" Ref="P2"  Part="1"
 AR Path="/58E527AF/5A39572B" Ref="P3"  Part="1"
-F 0 "P2" H 7050 4525 50  0000 C CNN
+F 0 "P3" H 7050 4525 50  0000 C CNN
 F 1 "XT30" H 7050 4225 50  0000 C CNN
 F 2 "zeabus:XT30" H 7050 4375 60  0001 C CNN

Commit message: changed pmos in Power_Switch_VBatt of Power_dist to STR2P3LLH6
Parts:
- removed Q2: IPD90P03P4L, TO_SOT_Packages_SMD:TO-252-2, symbol Q_PMOS_GDS
- added Q?: STR2P3LLH6, TO_SOT_Packages_SMD:SOT-23_Handsoldering, symbol Q_PMOS_GSD
- D4: value LED_Small -> PWR_SW_LED
Connections:
- net labels added: +PWR, Software_SW
- net labels removed: +Power, Software_Switch
Changed lines of the file:
@@
 $Descr A4 11693 8268
 encoding utf-8
-Sheet 4 10
+Sheet 10 10
 Title "DVL and Sonar Switch"
 Date "2017-04-06"
@@
 $EndDescr
 $Comp
-L Q_PMOS_GDS Q2
-U 1 1 58E52089
-P 6350 3300
-AR Path="/58E51F99/58E52089" Ref="Q2"  Part="1"
-AR Path="/58E527AF/58E52089" Ref="Q3"  Part="1"
-F 0 "Q3" H 6550 3350 50  0000 L CNN
-F 1 "IPD90P03P4L" H 6550 3250 50  0000 L CNN
-F 2 "TO_SOT_Packages_SMD:TO-252-2" H 6550 3400 50  0001 C CNN
-F 3 "" H 6350 3300 50  0001 C CNN
-	1    6350 3300
-	1    0    0    1
-$EndComp
-$Comp
 L R R5
 U 1 1 58E5219E
@@
 AR Path="/58E51F99/58E5219E" Ref="R5"  Part="1"
 AR Path="/58E527AF/58E5219E" Ref="R8"  Part="1"
-F 0 "R8" V 5930 3300 50  0000 C CNN
+F 0 "R5" V 5930 3300 50  0000 C CNN
 F 1 "2.2k" V 5850 3300 50  0000 C CNN
 F 2 "Resistors_SMD:R_0603" V 5780 3300 50  0001 C CNN
@@
 AR Path="/58E51F99/58E52234" Ref="D4"  Part="1"
 AR Path="/58E527AF/58E52234" Ref="D6"  Part="1"
-F 0 "D6" H 6400 4675 50  0000 L CNN
-F 1 "LED_Small" H 6275 4450 50  0000 L CNN
+F 0 "D4" H 6400 4675 50  0000 L CNN
+F 1 "PWR_SW_LED" H 6275 4450 50  0000 L CNN
 F 2 "LEDs:LED_0603_HandSoldering" V 6450 4550 50  0001 C CNN
 F 3 "" V 6450 4550 50  0001 C CNN
@@
 AR Path="/58E51F99/58E5234D" Ref="R4"  Part="1"
 AR Path="/58E527AF/58E5234D" Ref="R7"  Part="1"
-F 0 "R7" V 5930 2700 50  0000 C CNN
+F 0 "R4" V 5930 2700 50  0000 C CNN
 F 1 "10k" V 5850 2700 50  0000 C CNN
 F 2 "Resistors_SMD:R_0603" V 5780 2700 50  0001 C CNN
@@
 AR Path="/58E51F99/58E52389" Ref="R6"  Part="1"
 AR Path="/58E527AF/58E52389" Ref="R9"  Part="1"
-F 0 "R9" V 6530 4150 50  0000 C CNN
+F 0 "R6" V 6530 4150 50  0000 C CNN
 F 1 "10k" V 6450 4150 50  0000 C CNN
 F 2 "Resistors_SMD:R_0603" V 6380 4150 50  0001 C CNN
@@
 	-1   0    0    1
 $EndComp
-Text HLabel 3650 2450 0    60   Input ~ 0
-+Power
-Text HLabel 3650 3300 0    60   Input ~ 0
-Software_Switch
+Text HLabel 3650 2450 0    60   UnSpc ~ 0
++PWR
+Text HLabel 3650 3300 0    60   UnSpc ~ 0
+Software_SW
 Wire Wire Line
 	6000 3300 6150 3300
@@
 AR Path="/58E51F99/58E648CE" Ref="D3"  Part="1"
 AR Path="/58E527AF/58E648CE" Ref="D5"  Part="1"
-F 0 "D5" H 6100 3100 50  0000 C CNN
+F 0 "D3" H 6100 3100 50  0000 C CNN
 F 1 "BZT52c12s" H 6100 2900 50  0000 C CNN
 F 2 "Diodes_SMD:D_SOD-323_HandSoldering" H 6100 3000 50  0001 C CNN
@@
 	6100 3150 6100 3300
 Connection ~ 6100 3300
-Wire Wire Line
-	3650 2450 6450 2450
 Connection ~ 6450 2700
 $Comp
@@
 AR Path="/58E51F99/58E651FD" Ref="F2"  Part="1"
 AR Path="/58E527AF/58E651FD" Ref="F3"  Part="1"
-F 0 "F3" V 6530 3750 50  0000 C CNN
+F 0 "F2" V 6530 3750 50  0000 C CNN
 F 1 "Fuse" V 6375 3750 50  0000 C CNN
 F 2 "zeabus:FUSE_AUTO" V 6380 3750 50  0001 C CNN
@@
 AR Path="/58E51F99/5A39572B" Ref="P2"  Part="1"
 AR Path="/58E527AF/5A39572B" Ref="P3"  Part="1"
-F 0 "P3" H 7050 4525 50  0000 C CNN
+F 0 "P2" H 7050 4525 50  0000 C CNN
 F 1 "XT30" H 7050 4225 50  0000 C CNN
 F 2 "zeabus:XT30" H 7050 4375 60  0001 C CNN
@@
 Wire Wire Line
 	6850 4425 6850 4850
+$Comp
+L Q_PMOS_GSD Q?
+U 1 1 5B50BB80
+P 6350 3300
+AR Path="/58E51F99/5B50BB80" Ref="Q?"  Part="1"
+AR Path="/58E527AF/5B50BB80" Ref="Q?"  Part="1"
+F 0 "Q?" H 6550 3350 50  0000 L CNN
+F 1 "STR2P3LLH6" H 6550 3250 50  0000 L CNN
+F 2 "TO_SOT_Packages_SMD:SOT-23_Handsoldering" H 6550 3400 50  0001 C CNN
+F 3 "" H 6350 3300 50  0001 C CNN
+	1    6350 3300
+	1    0    0    1
+$EndComp
+Wire Wire Line
+	6450 2450 3650 2450
 $EndSCHEMATC

Commit message: added 47uF capacitor to Power_Switch_VBatt of Power_dist
Parts:
- added C?: 47uF, symbol C_Small
Connections:
- wire segments 17 -> 19
Changed lines of the file:
@@
 $EndComp
 Wire Wire Line
-	6450 2450 3650 2450
+	3650 2450 6750 2450
+Connection ~ 6450 2450
+$Comp
+L C_Small C?
+U 1 1 5B510029
+P 6750 2650
+F 0 "C?" H 6760 2720 50  0000 L CNN
+F 1 "47uF" H 6760 2570 50  0000 L CNN
+F 2 "" H 6750 2650 50  0001 C CNN
+F 3 "" H 6750 2650 50  0001 C CNN
+	1    6750 2650
+	1    0    0    -1
+$EndComp
+$Comp
+L GNDPWR #PWR?
+U 1 1 5B51011B
+P 6750 2800
+F 0 "#PWR?" H 6750 2600 50  0001 C CNN
+F 1 "GNDPWR" H 6750 2670 50  0000 C CNN
+F 2 "" H 6750 2750 50  0001 C CNN
+F 3 "" H 6750 2750 50  0001 C CNN
+	1    6750 2800
+	1    0    0    -1
+$EndComp
+Wire Wire Line
+	6750 2450 6750 2550
+Wire Wire Line
+	6750 2750 6750 2800
 $EndSCHEMATC

Commit message: added 1uF capacitor for LM4014CF in Current_Monitor of Power_dist
Parts:
- removed C?: 47uF, symbol C_Small
- added C?: 47uF, symbol CP_Small
Changed lines of the file:
@@
 $Descr A4 11693 8268
 encoding utf-8
-Sheet 10 11
+Sheet 9 11
 Title "DVL and Sonar Switch"
 Date "2017-04-06"
@@
 Connection ~ 6450 2450
 $Comp
-L C_Small C?
-U 1 1 5B510029
-P 6750 2650
-AR Path="/58E51F99/5B510029" Ref="C?"  Part="1"
-AR Path="/5B530A41/5B510029" Ref="C?"  Part="1"
-F 0 "C?" H 6760 2720 50  0000 L CNN
-F 1 "47uF" H 6760 2570 50  0000 L CNN
-F 2 "" H 6750 2650 50  0001 C CNN
-F 3 "" H 6750 2650 50  0001 C CNN
-	1    6750 2650
-	1    0    0    -1
-$EndComp
-$Comp
 L GNDPWR #PWR?
 U 1 1 5B51011B
@@
 Wire Wire Line
 	6750 2750 6750 2800
+$Comp
+L CP_Small C?
+U 1 1 5B532465
+P 6750 2650
+F 0 "C?" H 6760 2720 50  0000 L CNN
+F 1 "47uF" H 6760 2570 50  0000 L CNN
+F 2 "" H 6750 2650 50  0001 C CNN
+F 3 "" H 6750 2650 50  0001 C CNN
+	1    6750 2650
+	1    0    0    -1
+$EndComp
 $EndSCHEMATC

Commit message: Power_dist could be monitor battery voltage and system current
Parts:
- D19: renamed from D3; symbol D_Zener -> D_Zener_Small
- gave numbers to parts that had none: 2
- renumbered D4 to D20, F2 to F1, P2 to P8, R4 to R41, R5 to R42, R6 to R43
Changed lines of the file:
@@
 $EndDescr
 $Comp
-L R R5
+L R R42
 U 1 1 58E5219E
 P 5850 3300
-AR Path="/58E51F99/58E5219E" Ref="R5"  Part="1"
-AR Path="/58E527AF/58E5219E" Ref="R8"  Part="1"
-AR Path="/5B530A41/58E5219E" Ref="R5"  Part="1"
-F 0 "R5" V 5930 3300 50  0000 C CNN
+AR Path="/58E51F99/58E5219E" Ref="R42"  Part="1"
+AR Path="/5B530A41/58E5219E" Ref="R45"  Part="1"
+F 0 "R45" V 5930 3300 50  0000 C CNN
 F 1 "2.2k" V 5850 3300 50  0000 C CNN
 F 2 "Resistors_SMD:R_0603" V 5780 3300 50  0001 C CNN
@@
 $EndComp
 $Comp
-L LED_Small D4
+L LED_Small D20
 U 1 1 58E52234
 P 6450 4550
-AR Path="/58E51F99/58E52234" Ref="D4"  Part="1"
-AR Path="/58E527AF/58E52234" Ref="D6"  Part="1"
-AR Path="/5B530A41/58E52234" Ref="D4"  Part="1"
-F 0 "D4" H 6400 4675 50  0000 L CNN
+AR Path="/58E51F99/58E52234" Ref="D20"  Part="1"
+AR Path="/5B530A41/58E52234" Ref="D22"  Part="1"
+F 0 "D22" H 6400 4675 50  0000 L CNN
 F 1 "PWR_SW_LED" H 6275 4450 50  0000 L CNN
 F 2 "LEDs:LED_0603_HandSoldering" V 6450 4550 50  0001 C CNN
@@
 $EndComp
 $Comp
-L R R4
+L R R41
 U 1 1 58E5234D
 P 5850 2700
-AR Path="/58E51F99/58E5234D" Ref="R4"  Part="1"
-AR Path="/58E527AF/58E5234D" Ref="R7"  Part="1"
-AR Path="/5B530A41/58E5234D" Ref="R4"  Part="1"
-F 0 "R4" V 5930 2700 50  0000 C CNN
+AR Path="/58E51F99/58E5234D" Ref="R41"  Part="1"
+AR Path="/5B530A41/58E5234D" Ref="R44"  Part="1"
+F 0 "R44" V 5930 2700 50  0000 C CNN
 F 1 "10k" V 5850 2700 50  0000 C CNN
 F 2 "Resistors_SMD:R_0603" V 5780 2700 50  0001 C CNN
@@
 $EndComp
 $Comp
-L R R6
+L R R43
 U 1 1 58E52389
 P 6450 4150
-AR Path="/58E51F99/58E52389" Ref="R6"  Part="1"
-AR Path="/58E527AF/58E52389" Ref="R9"  Part="1"
-AR Path="/5B530A41/58E52389" Ref="R6"  Part="1"
-F 0 "R6" V 6530 4150 50  0000 C CNN
+AR Path="/58E51F99/58E52389" Ref="R43"  Part="1"
+AR Path="/5B530A41/58E52389" Ref="R46"  Part="1"
+F 0 "R46" V 6530 4150 50  0000 C CNN
 F 1 "10k" V 6450 4150 50  0000 C CNN
 F 2 "Resistors_SMD:R_0603" V 6380 4150 50  0001 C CNN
@@
 	6450 2450 6450 3100
 $Comp
-L D_Zener D3
+L D_Zener_Small D19
 U 1 1 58E648CE
 P 6100 3000
-AR Path="/58E51F99/58E648CE" Ref="D3"  Part="1"
-AR Path="/58E527AF/58E648CE" Ref="D5"  Part="1"
-AR Path="/5B530A41/58E648CE" Ref="D3"  Part="1"
-F 0 "D3" H 6100 3100 50  0000 C CNN
+AR Path="/58E51F99/58E648CE" Ref="D19"  Part="1"
+AR Path="/5B530A41/58E648CE" Ref="D21"  Part="1"
+F 0 "D21" H 6100 3100 50  0000 C CNN
 F 1 "BZT52c12s" H 6100 2900 50  0000 C CNN
 F 2 "Diodes_SMD:D_SOD-323_HandSoldering" H 6100 3000 50  0001 C CNN
@@
 	6000 2700 6450 2700
 Wire Wire Line
-	6100 2850 6100 2700
+	6100 2700 6100 2900
 Connection ~ 6100 2700
 Wire Wire Line
-	6100 3150 6100 3300
+	6100 3100 6100 3300
 Connection ~ 6100 3300
 Connection ~ 6450 2700
 $Comp
-L Fuse F2
+L Fuse F1
 U 1 1 58E651FD
 P 6450 3750
-AR Path="/58E51F99/58E651FD" Ref="F2"  Part="1"
-AR Path="/58E527AF/58E651FD" Ref="F3"  Part="1"
+AR Path="/58E51F99/58E651FD" Ref="F1"  Part="1"
 AR Path="/5B530A41/58E651FD" Ref="F2"  Part="1"
 F 0 "F2" V 6530 3750 50  0000 C CNN
@@
 	6850 4850 6450 4850
 $Comp
-L XT30 P2
+L XT30 P8
 U 1 1 5A39572B
 P 7050 4375
-AR Path="/58E51F99/5A39572B" Ref="P2"  Part="1"
-AR Path="/58E527AF/5A39572B" Ref="P3"  Part="1"
-AR Path="/5B530A41/5A39572B" Ref="P2"  Part="1"
-F 0 "P2" H 7050 4525 50  0000 C CNN
+AR Path="/58E51F99/5A39572B" Ref="P8"  Part="1"
+AR Path="/5B530A41/5A39572B" Ref="P9"  Part="1"
+F 0 "P9" H 7050 4525 50  0000 C CNN
 F 1 "XT30" H 7050 4225 50  0000 C CNN
 F 2 "zeabus:XT30" H 7050 4375 60  0001 C CNN
@@
 $EndComp
 $Comp
-L GNDPWR #PWR?
+L GNDPWR #PWR74
 U 1 1 5B5DF3EC
 P 6450 4950
-AR Path="/58E51F99/5B5DF3EC" Ref="#PWR?"  Part="1"
-AR Path="/58E527AF/5B5DF3EC" Ref="#PWR?"  Part="1"
-AR Path="/5B530A41/5B5DF3EC" Ref="#PWR?"  Part="1"
-F 0 "#PWR?" H 6450 4750 50  0001 C CNN
+AR Path="/58E51F99/5B5DF3EC" Ref="#PWR74"  Part="1"
+AR Path="/5B530A41/5B5DF3EC" Ref="#PWR76"  Part="1"
+F 0 "#PWR76" H 6450 4750 50  0001 C CNN
 F 1 "GNDPWR" H 6450 4820 50  0000 C CNN
 F 2 "" H 6450 4900 50  0001 C CNN
@@
 	6850 4425 6850 4850
 $Comp
-L Q_PMOS_GSD Q?
+L Q_PMOS_GSD Q8
 U 1 1 5B50BB80
 P 6350 3300
-AR Path="/58E51F99/5B50BB80" Ref="Q?"  Part="1"
-AR Path="/58E527AF/5B50BB80" Ref="Q?"  Part="1"
-AR Path="/5B530A41/5B50BB80" Ref="Q?"  Part="1"
-F 0 "Q?" H 6550 3350 50  0000 L CNN
+AR Path="/58E51F99/5B50BB80" Ref="Q8"  Part="1"
+AR Path="/5B530A41/5B50BB80" Ref="Q9"  Part="1"
+F 0 "Q9" H 6550 3350 50  0000 L CNN
 F 1 "STR2P3LLH6" H 6550 3250 50  0000 L CNN
 F 2 "TO_SOT_Packages_SMD:SOT-23_Handsoldering" H 6550 3400 50  0001 C CNN
@@
 Connection ~ 6450 2450
 $Comp
-L GNDPWR #PWR?
+L GNDPWR #PWR75
 U 1 1 5B51011B
 P 6750 2800
-AR Path="/58E51F99/5B51011B" Ref="#PWR?"  Part="1"
-AR Path="/5B530A41/5B51011B" Ref="#PWR?"  Part="1"
-F 0 "#PWR?" H 6750 2600 50  0001 C CNN
+AR Path="/58E51F99/5B51011B" Ref="#PWR75"  Part="1"
+AR Path="/5B530A41/5B51011B" Ref="#PWR77"  Part="1"
+F 0 "#PWR77" H 6750 2600 50  0001 C CNN
 F 1 "GNDPWR" H 6750 2670 50  0000 C CNN
 F 2 "" H 6750 2750 50  0001 C CNN
@@
 	6750 2750 6750 2800
 $Comp
-L CP_Small C?
+L CP_Small C23
 U 1 1 5B532465
 P 6750 2650
-F 0 "C?" H 6760 2720 50  0000 L CNN
+AR Path="/58E51F99/5B532465" Ref="C23"  Part="1"
+AR Path="/5B530A41/5B532465" Ref="C24"  Part="1"
+F 0 "C24" H 6760 2720 50  0000 L CNN
 F 1 "47uF" H 6760 2570 50  0000 L CNN
 F 2 "" H 6750 2650 50  0001 C CNN
