File: Circuit/Power_dist/Current_Monitor.sch (KiCad schematic (older format))
At the start: 6 parts

Commit message: refactor Power_dist
Connections:
- net labels added: GNDPWR
- net labels removed: GND
- no-connect marks 0 -> 1
Changed lines of the file:
@@
-	1    0    0    -1
-$EndComp
-$Comp
-L GND #PWR?
-U 1 1 5B4C3925
-P 5500 4350
-F 0 "#PWR?" H 5500 4100 50  0001 C CNN
-F 1 "GND" H 5500 4200 50  0000 C CNN
-F 2 "" H 5500 4350 50  0001 C CNN
-F 3 "" H 5500 4350 50  0001 C CNN
-	1    5500 4350
 	1    0    0    -1
 $EndComp
@@
 Text HLabel 7275 3875 2    60   Output ~ 0
 OUT
-$Comp
-L GND #PWR?
-U 1 1 5B4CDA84
-P 7050 4875
-F 0 "#PWR?" H 7050 4625 50  0001 C CNN
-F 1 "GND" H 7050 4725 50  0000 C CNN
-F 2 "" H 7050 4875 50  0001 C CNN
-F 3 "" H 7050 4875 50  0001 C CNN
-	1    7050 4875
-	1    0    0    -1
-$EndComp
 Wire Wire Line
 	7000 4700 7050 4700
@@
 	1    0    0    -1
 $EndComp
-$Comp
-L GND #PWR?
-U 1 1 5B4D19FF
-P 5125 3500
-F 0 "#PWR?" H 5125 3250 50  0001 C CNN
-F 1 "GND" H 5125 3350 50  0000 C CNN
-F 2 "" H 5125 3500 50  0001 C CNN
-F 3 "" H 5125 3500 50  0001 C CNN
-	1    5125 3500
-	1    0    0    -1
-$EndComp
 Wire Wire Line
 	5125 3500 5125 3425
@@
 Text HLabel 4025 3125 0    60   UnSpc ~ 0
 +5V_PWR
+NoConn ~ 5150 3900
+$Comp
+L GNDPWR #PWR?
+U 1 1 5B599606
+P 5125 3500
+F 0 "#PWR?" H 5125 3300 50  0001 C CNN
+F 1 "GNDPWR" H 5125 3370 50  0000 C CNN
+F 2 "" H 5125 3450 50  0001 C CNN
+F 3 "" H 5125 3450 50  0001 C CNN
+	1    5125 3500
+	1    0    0    -1
+$EndComp
+$Comp
+L GNDPWR #PWR?
+U 1 1 5B59962A
+P 5500 4350
+F 0 "#PWR?" H 5500 4150 50  0001 C CNN
+F 1 "GNDPWR" H 5500 4220 50  0000 C CNN
+F 2 "" H 5500 4300 50  0001 C CNN
+F 3 "" H 5500 4300 50  0001 C CNN
+	1    5500 4350
+	1    0    0    -1
+$EndComp
+$Comp
+L GNDPWR #PWR?
+U 1 1 5B599647
+P 7050 4875
+F 0 "#PWR?" H 7050 4675 50  0001 C CNN
+F 1 "GNDPWR" H 7050 4745 50  0000 C CNN
+F 2 "" H 7050 4825 50  0001 C CNN
+F 3 "" H 7050 4825 50  0001 C CNN
+	1    7050 4875
+	1    0    0    -1
+$EndComp
 $EndSCHEMATC

Commit message: added 1uF capacitor for LM4014CF in Current_Monitor of Power_dist
Parts:
- added C?: 1uF, symbol CP_Small
Connections:
- wire segments 28 -> 29
Changed lines of the file:
@@
 $Descr A4 11693 8268
 encoding utf-8
-Sheet 7 11
+Sheet 5 11
 Title ""
 Date ""
@@
 	5600 4275 6000 4275
 Wire Wire Line
-	6000 3450 6000 4700
-Wire Wire Line
 	5850 4700 6150 4700
 Connection ~ 6000 4700
@@
 	1    0    0    -1
 $EndComp
+$Comp
+L CP_Small C?
+U 1 1 5B5067FF
+P 6000 5000
+F 0 "C?" H 6010 5070 50  0000 L CNN
+F 1 "1uF" H 6010 4920 50  0000 L CNN
+F 2 "" H 6000 5000 50  0001 C CNN
+F 3 "" H 6000 5000 50  0001 C CNN
+	1    6000 5000
+	1    0    0    -1
+$EndComp
+$Comp
+L GNDPWR #PWR?
+U 1 1 5B50689B
+P 6000 5175
+F 0 "#PWR?" H 6000 4975 50  0001 C CNN
+F 1 "GNDPWR" H 6000 5045 50  0000 C CNN
+F 2 "" H 6000 5125 50  0001 C CNN
+F 3 "" H 6000 5125 50  0001 C CNN
+	1    6000 5175
+	1    0    0    -1
+$EndComp
+Wire Wire Line
+	6000 3450 6000 4900
+Wire Wire Line
+	6000 5175 6000 5100
 $EndSCHEMATC

Commit message: power line and data line source of Power_Controller on Power_dist could be manual selected
Parts:
- R?: footprint Resistors_SMD:R_0805_HandSoldering -> Resistors_SMD:R_0603_HandSoldering
Changed lines of the file:
@@
 F 0 "R?" V 5780 4700 50  0000 C CNN
 F 1 "1.5k" V 5700 4700 50  0000 C CNN
-F 2 "Resistors_SMD:R_0805_HandSoldering" V 5630 4700 50  0001 C CNN
+F 2 "Resistors_SMD:R_0603_HandSoldering" V 5630 4700 50  0001 C CNN
 F 3 "" H 5700 4700 50  0001 C CNN
 	1    5700 4700

Commit message: Power_dist could be monitor battery voltage and system current
Parts:
- C15: renamed from C?; footprint (none) -> Capacitors_SMD:C_1206_HandSoldering
- gave numbers to parts that had none: 6
Connections:
- no-connect marks 1 -> 0
Changed lines of the file:
@@
 $EndDescr
 $Comp
-L R R?
+L R R26
 U 1 1 5B4C1590
 P 4700 2825
-F 0 "R?" V 4780 2825 50  0000 C CNN
+F 0 "R26" V 4780 2825 50  0000 C CNN
 F 1 "2m" V 4700 2825 50  0000 C CNN
 F 2 "Resistors_SMD:R_2512_HandSoldering" V 4630 2825 50  0001 C CNN
@@
 	4850 2825 4950 2825
 $Comp
-L INA240 U?
+L INA240 U5
 U 1 1 5B4C345B
 P 5500 3875
-F 0 "U?" H 5650 4000 50  0000 L CNN
+F 0 "U5" H 5650 4000 50  0000 L CNN
 F 1 "INA240" H 5650 3750 50  0000 L CNN
 F 2 "Housings_SOIC:SOIC-8_3.9x4.9mm_Pitch1.27mm" H 5500 4275 50  0001 C CNN
@@
 Connection ~ 5500 4275
 $Comp
-L LM4041CF U?
+L LM4041CF U6
 U 1 1 5B4C7EB6
 P 6575 4700
-F 0 "U?" H 6300 4900 50  0000 C CNN
+F 0 "U6" H 6300 4900 50  0000 C CNN
 F 1 "LM4041CF" H 6550 4900 50  0000 L CNN
 F 2 "TO_SOT_Packages_SMD:SOT-23_Handsoldering" H 6575 5000 50  0001 C CIN
@@
 $EndComp
 $Comp
-L R R?
+L R R25
 U 1 1 5B4C8001
 P 4700 2525
-F 0 "R?" V 4780 2525 50  0000 C CNN
+F 0 "R25" V 4780 2525 50  0000 C CNN
 F 1 "2m" V 4700 2525 50  0000 C CNN
 F 2 "Resistors_SMD:R_2512_HandSoldering" V 4630 2525 50  0001 C CNN
@@
 $EndComp
 $Comp
-L R R?
+L R R27
 U 1 1 5B4C80AE
 P 5700 4700
-F 0 "R?" V 5780 4700 50  0000 C CNN
+F 0 "R27" V 5780 4700 50  0000 C CNN
 F 1 "1.5k" V 5700 4700 50  0000 C CNN
 F 2 "Resistors_SMD:R_0603_HandSoldering" V 5630 4700 50  0001 C CNN
@@
 	7050 4700 7050 4875
 $Comp
-L C_Small C?
+L C_Small C14
 U 1 1 5B4D120C
 P 5125 3325
-F 0 "C?" H 5135 3395 50  0000 L CNN
+F 0 "C14" H 5135 3395 50  0000 L CNN
 F 1 "0.1uF" H 5135 3245 50  0000 L CNN
 F 2 "Capacitors_SMD:C_0603_HandSoldering" H 5125 3325 50  0001 C CNN
@@
 Text HLabel 4025 3125 0    60   UnSpc ~ 0
 +5V_PWR
-NoConn ~ 5150 3900
 $Comp
-L GNDPWR #PWR?
+L GNDPWR #PWR59
 U 1 1 5B599606
 P 5125 3500
-F 0 "#PWR?" H 5125 3300 50  0001 C CNN
+F 0 "#PWR59" H 5125 3300 50  0001 C CNN
 F 1 "GNDPWR" H 5125 3370 50  0000 C CNN
 F 2 "" H 5125 3450 50  0001 C CNN
@@
 $EndComp
 $Comp
-L GNDPWR #PWR?
+L GNDPWR #PWR60
 U 1 1 5B59962A
 P 5500 4350
-F 0 "#PWR?" H 5500 4150 50  0001 C CNN
+F 0 "#PWR60" H 5500 4150 50  0001 C CNN
 F 1 "GNDPWR" H 5500 4220 50  0000 C CNN
 F 2 "" H 5500 4300 50  0001 C CNN
@@
 $EndComp
 $Comp
-L GNDPWR #PWR?
+L GNDPWR #PWR62
 U 1 1 5B599647
 P 7050 4875
-F 0 "#PWR?" H 7050 4675 50  0001 C CNN
+F 0 "#PWR62" H 7050 4675 50  0001 C CNN
 F 1 "GNDPWR" H 7050 4745 50  0000 C CNN
 F 2 "" H 7050 4825 50  0001 C CNN
@@
 $EndComp
 $Comp
-L CP_Small C?
+L CP_Small C15
 U 1 1 5B5067FF
 P 6000 5000
-F 0 "C?" H 6010 5070 50  0000 L CNN
+F 0 "C15" H 6010 5070 50  0000 L CNN
 F 1 "1uF" H 6010 4920 50  0000 L CNN
-F 2 "" H 6000 5000 50  0001 C CNN
+F 2 "Capacitors_SMD:C_1206_HandSoldering" H 6000 5000 50  0001 C CNN
 F 3 "" H 6000 5000 50  0001 C CNN
 	1    6000 5000
@@
 $EndComp
 $Comp
-L GNDPWR #PWR?
+L GNDPWR #PWR61
 U 1 1 5B50689B
 P 6000 5175
-F 0 "#PWR?" H 6000 4975 50  0001 C CNN
+F 0 "#PWR61" H 6000 4975 50  0001 C CNN
 F 1 "GNDPWR" H 6000 5045 50  0000 C CNN
 F 2 "" H 6000 5125 50  0001 C CNN
