File: Circuit/Power_dist/Power_Aggregator.sch (KiCad schematic (older format))
At the start: 19 parts, among them P16 XT60, P17 XT60, Q6 AUIRFS8409-7P, Q7 AUIRFS8409-7P, U5 LTC4357, U6 LTC4357

Commit message: added filter to dc-dc converters in Power_dist
Parts:
- P16: value XT60 -> BATT1
- P17: value XT60 -> BATT2
Changed lines of the file:
@@
 $Descr A4 11693 8268
 encoding utf-8
-Sheet 6 10
+Sheet 10 10
 Title "Power Aggregator"
 Date "2017-04-06"
@@
 P 3450 4450
 F 0 "P17" H 3450 4600 50  0000 C CNN
-F 1 "XT60" H 3450 4300 50  0000 C CNN
+F 1 "BATT2" H 3450 4300 50  0000 C CNN
 F 2 "zeabus:XT60" H 3450 4450 60  0001 C CNN
 F 3 "" H 3450 4450 60  0000 C CNN
@@
 P 3450 2550
 F 0 "P16" H 3450 2700 50  0000 C CNN
-F 1 "XT60" H 3450 2400 50  0000 C CNN
+F 1 "BATT1" H 3450 2400 50  0000 C CNN
 F 2 "zeabus:XT60" H 3450 2550 60  0001 C CNN
 F 3 "" H 3450 2550 60  0000 C CNN

Commit message: refactor Power_dist
Parts:
- removed D13: BATT2_LED, LEDs:LED_0603_HandSoldering, symbol LED_Small
- removed D14: BATT_LED, LEDs:LED_0603_HandSoldering, symbol LED_Small
- removed D8: BATT1_LED, LEDs:LED_0603_HandSoldering, symbol LED_Small
- removed P16: BATT1, zeabus:XT60, symbol XT60
- removed P17: BATT2, zeabus:XT60, symbol XT60
- removed R11, R12, R29: 10k, Resistors_SMD:R_0603_HandSoldering, symbol R
Connections:
- net labels added: +BATT1, +BATT2, GNDPWR
- net labels removed: GND
- wire segments 66 -> 55

Commit message: added 1uF capacitor for LM4014CF in Current_Monitor of Power_dist
Parts:
- removed C?: 47uF, Capacitors_SMD:CP_Elec_6.3x5.8, symbol C_Small
- added C?: 47uF, symbol CP_Small
Changed lines of the file:
@@
 $Descr A4 11693 8268
 encoding utf-8
-Sheet 9 11
+Sheet 7 11
 Title "Power Aggregator"
 Date "2017-04-06"
@@
 	1    0    0    -1
 $EndComp
-$Comp
-L C_Small C?
-U 1 1 5B4C70EB
-P 7650 2200
-F 0 "C?" H 7660 2270 50  0000 L CNN
-F 1 "47uF" H 7660 2120 50  0000 L CNN
-F 2 "Capacitors_SMD:CP_Elec_6.3x5.8" H 7650 2200 50  0001 C CNN
-F 3 "" H 7650 2200 50  0001 C CNN
-	1    7650 2200
-	1    0    0    -1
-$EndComp
 Text HLabel 4125 2100 0    60   UnSpc ~ 0
 +BATT1
@@
 	7000 3450 6700 3450
 Connection ~ 6700 3450
+$Comp
+L CP_Small C?
+U 1 1 5B53302F
+P 7650 2200
+F 0 "C?" H 7660 2270 50  0000 L CNN
+F 1 "47uF" H 7660 2120 50  0000 L CNN
+F 2 "" H 7650 2200 50  0001 C CNN
+F 3 "" H 7650 2200 50  0001 C CNN
+	1    7650 2200
+	1    0    0    -1
+$EndComp
 $EndSCHEMATC

Commit message: power line and data line source of Power_Controller on Power_dist could be manual selected
Parts:
- C?: footprint (none) -> Capacitors_SMD:CP_Elec_6.3x5.8
Changed lines of the file:
@@
 F 1 "AUIRFS8409-7P" H 5450 3650 50  0000 L CNN
 F 2 "TO_SOT_Packages_SMD:TO-263-6" H 5650 3550 50  0001 C CIN
-F 3 "${KIPJTMOD}" H 5450 4300 50  0001 L CNN
+F 3 "" H 5450 4300 50  0001 L CNN
 	1    5650 4000
 	-1   0    0    -1
@@
 F 0 "C?" H 7660 2270 50  0000 L CNN
 F 1 "47uF" H 7660 2120 50  0000 L CNN
-F 2 "" H 7650 2200 50  0001 C CNN
+F 2 "Capacitors_SMD:CP_Elec_6.3x5.8" H 7650 2200 50  0001 C CNN
 F 3 "" H 7650 2200 50  0001 C CNN
 	1    7650 2200

Commit message: Power_dist could be monitor battery voltage and system current
Parts:
- removed D? (x2): B340AE, Diodes_SMD:D_SMA_Handsoldering, symbol D
- added D15, D16: B340AE, Diodes_SMD:D_SMA_Handsoldering, symbol D_Small
- gave numbers to parts that had none: 5
- renumbered Q6 to Q5, Q7 to Q6, U5 to U8, U6 to U9
Changed lines of the file:
@@
 $EndDescr
 $Comp
-L LTC4357 U6
+L LTC4357 U9
 U 1 1 5626F549
 P 6150 5050
-F 0 "U6" H 5900 5350 60  0000 C CNN
+F 0 "U9" H 5900 5350 60  0000 C CNN
 F 1 "LTC4357" H 6050 4750 60  0000 C CNN
 F 2 "Housings_SSOP:MSOP-8_3x3mm_Pitch0.65mm" H 5850 4900 60  0001 C CNN
@@
 $EndComp
 $Comp
-L LTC4357 U5
+L LTC4357 U8
 U 1 1 5626F94D
 P 6150 3150
-F 0 "U5" H 5900 3450 60  0000 C CNN
+F 0 "U8" H 5900 3450 60  0000 C CNN
 F 1 "LTC4357" H 6050 2850 60  0000 C CNN
 F 2 "Housings_SSOP:MSOP-8_3x3mm_Pitch0.65mm" H 5850 3000 60  0001 C CNN
@@
 Text HLabel 8100 2000 2    60   UnSpc ~ 0
 +VBatt
-NoConn ~ 6600 5100
-NoConn ~ 5700 5000
-NoConn ~ 5700 5100
-NoConn ~ 5700 3100
-NoConn ~ 5700 3200
-NoConn ~ 6600 3200
-$Comp
-L AUIRFS8409-7P Q7
+$Comp
+L AUIRFS8409-7P Q6
 U 1 1 5B464942
 P 5650 4000
-F 0 "Q7" H 5450 4300 50  0000 L CNN
+F 0 "Q6" H 5450 4300 50  0000 L CNN
 F 1 "AUIRFS8409-7P" H 5450 3650 50  0000 L CNN
 F 2 "TO_SOT_Packages_SMD:TO-263-6" H 5650 3550 50  0001 C CIN
@@
 $EndComp
 $Comp
-L AUIRFS8409-7P Q6
+L AUIRFS8409-7P Q5
 U 1 1 5B465336
 P 5650 2100
-F 0 "Q6" H 5450 2400 50  0000 L CNN
+F 0 "Q5" H 5450 2400 50  0000 L CNN
 F 1 "AUIRFS8409-7P" H 5450 1750 50  0000 L CNN
 F 2 "TO_SOT_Packages_SMD:TO-263-6" H 5650 1650 50  0001 C CIN
@@
 $EndComp
 $Comp
-L D D?
-U 1 1 5B4A7AEB
-P 4650 2350
-F 0 "D?" H 4650 2450 50  0000 C CNN
-F 1 "B340AE" H 4650 2250 50  0000 C CNN
-F 2 "Diodes_SMD:D_SMA_Handsoldering" H 4650 2350 50  0001 C CNN
-F 3 "" H 4650 2350 50  0001 C CNN
-	1    4650 2350
-	0    1    1    0
-$EndComp
-$Comp
-L D D?
-U 1 1 5B4A9ECD
-P 4650 4250
-F 0 "D?" H 4650 4350 50  0000 C CNN
-F 1 "B340AE" H 4650 4150 50  0000 C CNN
-F 2 "Diodes_SMD:D_SMA_Handsoldering" H 4650 4250 50  0001 C CNN
-F 3 "" H 4650 4250 50  0001 C CNN
-	1    4650 4250
-	0    1    1    0
-$EndComp
-$Comp
-L C_Small C?
+L C_Small C18
 U 1 1 5B4B4A1C
 P 7000 3300
-F 0 "C?" H 7010 3370 50  0000 L CNN
+F 0 "C18" H 7010 3370 50  0000 L CNN
 F 1 "1uF" H 7010 3220 50  0000 L CNN
 F 2 "Capacitors_SMD:C_0603_HandSoldering" H 7000 3300 50  0001 C CNN
@@
 $EndComp
 $Comp
-L R R?
+L R R36
 U 1 1 5B4B4A87
 P 7000 2850
-F 0 "R?" V 7080 2850 50  0000 C CNN
+F 0 "R36" V 7080 2850 50  0000 C CNN
 F 1 "100" V 7000 2850 50  0000 C CNN
 F 2 "Resistors_SMD:R_0603_HandSoldering" V 6930 2850 50  0001 C CNN
@@
 $EndComp
 $Comp
-L C_Small C?
+L C_Small C19
 U 1 1 5B4BDB43
 P 7000 5200
-F 0 "C?" H 7010 5270 50  0000 L CNN
+F 0 "C19" H 7010 5270 50  0000 L CNN
 F 1 "1uF" H 7010 5120 50  0000 L CNN
 F 2 "Capacitors_SMD:C_0603_HandSoldering" H 7000 5200 50  0001 C CNN
@@
 $EndComp
 $Comp
-L R R?
+L R R37
 U 1 1 5B4BDB49
 P 7000 4750
-F 0 "R?" V 7080 4750 50  0000 C CNN
+F 0 "R37" V 7080 4750 50  0000 C CNN
 F 1 "100" V 7000 4750 50  0000 C CNN
 F 2 "Resistors_SMD:R_0603_HandSoldering" V 6930 4750 50  0001 C CNN
@@
 	5600 5200 5700 5200
 Wire Wire Line
-	4650 2650 4650 2500
-Wire Wire Line
-	4650 4400 4650 4500
+	4650 2550 4650 2400
+Wire Wire Line
+	4650 4300 4650 4400
 Wire Wire Line
 	4650 2100 4650 2200
@@
 	4125 4000 5350 4000
 $Comp
-L GNDPWR #PWR?
+L GNDPWR #PWR67
 U 1 1 5B5869D6
-P 4650 2650
-F 0 "#PWR?" H 4650 2450 50  0001 C CNN
-F 1 "GNDPWR" H 4650 2520 50  0000 C CNN
-F 2 "" H 4650 2600 50  0001 C CNN
-F 3 "" H 4650 2600 50  0001 C CNN
-	1    4650 2650
-	1    0    0    -1
-$EndComp
-$Comp
-L GNDPWR #PWR?
+P 4650 2550
+F 0 "#PWR67" H 4650 2350 50  0001 C CNN
+F 1 "GNDPWR" H 4650 2420 50  0000 C CNN
+F 2 "" H 4650 2500 50  0001 C CNN
+F 3 "" H 4650 2500 50  0001 C CNN
+	1    4650 2550
+	1    0    0    -1
+$EndComp
+$Comp
+L GNDPWR #PWR68
 U 1 1 5B586D7F
-P 4650 4500
-F 0 "#PWR?" H 4650 4300 50  0001 C CNN
-F 1 "GNDPWR" H 4650 4370 50  0000 C CNN
-F 2 "" H 4650 4450 50  0001 C CNN
-F 3 "" H 4650 4450 50  0001 C CNN
-	1    4650 4500
-	1    0    0    -1
-$EndComp
-$Comp
-L GNDPWR #PWR?
+P 4650 4400
+F 0 "#PWR68" H 4650 4200 50  0001 C CNN
+F 1 "GNDPWR" H 4650 4270 50  0000 C CNN
+F 2 "" H 4650 4350 50  0001 C CNN
+F 3 "" H 4650 4350 50  0001 C CNN
+	1    4650 4400
+	1    0    0    -1
+$EndComp
+$Comp
+L GNDPWR #PWR71
 U 1 1 5B586DAB
 P 7650 2400
-F 0 "#PWR?" H 7650 2200 50  0001 C CNN
+F 0 "#PWR71" H 7650 2200 50  0001 C CNN
 F 1 "GNDPWR" H 7650 2270 50  0000 C CNN
 F 2 "" H 7650 2350 50  0001 C CNN
@@
 $EndComp
 $Comp
-L GNDPWR #PWR?
+L GNDPWR #PWR69
 U 1 1 5B586E03
 P 6700 3500
-F 0 "#PWR?" H 6700 3300 50  0001 C CNN
+F 0 "#PWR69" H 6700 3300 50  0001 C CNN
 F 1 "GNDPWR" H 6700 3370 50  0000 C CNN
 F 2 "" H 6700 3450 50  0001 C CNN
@@
 $EndComp
 $Comp
-L GNDPWR #PWR?
+L GNDPWR #PWR70
 U 1 1 5B586E3A
 P 6700 5400
-F 0 "#PWR?" H 6700 5200 50  0001 C CNN
+F 0 "#PWR70" H 6700 5200 50  0001 C CNN
 F 1 "GNDPWR" H 6700 5270 50  0000 C CNN
 F 2 "" H 6700 5350 50  0001 C CNN
@@
 Connection ~ 6700 3450
 $Comp
-L CP_Small C?
+L CP_Small C20
 U 1 1 5B53302F
 P 7650 2200
-F 0 "C?" H 7660 2270 50  0000 L CNN
+F 0 "C20" H 7660 2270 50  0000 L CNN
 F 1 "47uF" H 7660 2120 50  0000 L CNN
 F 2 "Capacitors_SMD:CP_Elec_6.3x5.8" H 7650 2200 50  0001 C CNN
@@
 	1    0    0    -1
 $EndComp
+$Comp
+L D_Small D15
+U 1 1 5B6B4986
+P 4650 2300
+F 0 "D15" H 4600 2380 50  0000 L CNN
+F 1 "B340AE" H 4500 2220 50  0000 L CNN
+F 2 "Diodes_SMD:D_SMA_Handsoldering" V 4650 2300 50  0001 C CNN
+F 3 "" V 4650 2300 50  0001 C CNN
+	1    4650 2300
+	0    1    1    0
+$EndComp
+$Comp
+L D_Small D16
+U 1 1 5B6B5D89
+P 4650 4200
+F 0 "D16" H 4600 4280 50  0000 L CNN
+F 1 "B340AE" H 4500 4120 50  0000 L CNN
+F 2 "Diodes_SMD:D_SMA_Handsoldering" V 4650 4200 50  0001 C CNN
+F 3 "" V 4650 4200 50  0001 C CNN
+	1    4650 4200
+	0    1    1    0
+$EndComp
+NoConn ~ 5700 5100
+NoConn ~ 5700 5000
+NoConn ~ 6600 5100
+NoConn ~ 6600 3200
+NoConn ~ 5700 3200
+NoConn ~ 5700 3100
 $EndSCHEMATC
