File: Circuit/Power_dist/Soft_Start_Circuit.sch (KiCad schematic (older format))
At the start: 14 parts

Commit message: added filter to dc-dc converters in Power_dist
Connections:
- wire segments 48 -> 49
Other:
- moved on the sheet: R?
Changed lines of the file:
@@
 $Descr A4 11693 8268
 encoding utf-8
-Sheet 10 10
+Sheet 9 10
 Title ""
 Date ""
@@
 L R R?
 U 1 1 5B4C6A59
-P 4700 2250
-F 0 "R?" V 4780 2250 50  0000 C CNN
-F 1 "5" V 4700 2250 50  0000 C CNN
-F 2 "zeabus:THK45" V 4630 2250 50  0001 C CNN
-F 3 "" H 4700 2250 50  0001 C CNN
-	1    4700 2250
+P 6450 2250
+F 0 "R?" V 6530 2250 50  0000 C CNN
+F 1 "5" V 6450 2250 50  0000 C CNN
+F 2 "zeabus:THK45" V 6380 2250 50  0001 C CNN
+F 3 "" H 6450 2250 50  0001 C CNN
+	1    6450 2250
 	0    1    1    0
 $EndComp
@@
 L R R?
 U 1 1 5B4C6AA7
-P 4700 2600
-F 0 "R?" V 4780 2600 50  0000 C CNN
-F 1 "5" V 4700 2600 50  0000 C CNN
-F 2 "zeabus:THK45" V 4630 2600 50  0001 C CNN
-F 3 "" H 4700 2600 50  0001 C CNN
-	1    4700 2600
+P 6450 2600
+F 0 "R?" V 6530 2600 50  0000 C CNN
+F 1 "5" V 6450 2600 50  0000 C CNN
+F 2 "zeabus:THK45" V 6380 2600 50  0001 C CNN
+F 3 "" H 6450 2600 50  0001 C CNN
+	1    6450 2600
 	0    1    1    0
 $EndComp
@@
 $EndComp
 Wire Wire Line
-	3700 2425 4400 2425
-Wire Wire Line
-	4400 2250 4550 2250
-Connection ~ 4400 2425
-Wire Wire Line
-	4850 2250 5000 2250
-Wire Wire Line
-	5000 2425 7775 2425
-Connection ~ 5000 2425
-Wire Wire Line
-	4400 2600 4550 2600
-Wire Wire Line
-	5000 2250 5000 2600
-Wire Wire Line
-	5000 2600 4850 2600
+	6150 2250 6300 2250
+Connection ~ 6150 2425
+Wire Wire Line
+	6600 2250 6750 2250
+Connection ~ 6750 2425
+Wire Wire Line
+	6150 2600 6300 2600
+Wire Wire Line
+	6750 2250 6750 2600
+Wire Wire Line
+	6750 2600 6600 2600
 Wire Wire Line
 	4025 3000 6150 3000
-Connection ~ 4400 2600
 Wire Wire Line
 	6150 3875 5825 3875
@@
 	6075 4275 6150 4275
 Connection ~ 6075 4175
-Wire Wire Line
-	4400 2250 4400 3725
 Wire Wire Line
 	5825 3000 5825 4700
@@
 	4025 4775 4025 3000
 Wire Wire Line
-	4950 3900 4950 3000
+	4950 2425 4950 3900
 Connection ~ 4950 3000
 Wire Wire Line
@@
 Wire Wire Line
 	4025 5725 4025 5600
+Wire Wire Line
+	6750 2425 7775 2425
+Wire Wire Line
+	6150 2425 3700 2425
+Wire Wire Line
+	4400 3725 4400 3000
+Wire Wire Line
+	6150 2250 6150 2600
+Connection ~ 4950 2425
 $EndSCHEMATC

Commit message: refactor Power_dist
Connections:
- net labels added: GNDPWR
- net labels removed: GND
Changed lines of the file:
@@
-$EndComp
-$Comp
-L GND #PWR?
-U 1 1 5B4CC69C
-P 4950 5550
-F 0 "#PWR?" H 4950 5300 50  0001 C CNN
-F 1 "GND" H 4950 5400 50  0000 C CNN
-F 2 "" H 4950 5550 50  0001 C CNN
-F 3 "" H 4950 5550 50  0001 C CNN
-	1    4950 5550
-	1    0    0    -1
 $EndComp
 $Comp
@@
 	1    0    0    -1
 $EndComp
-$Comp
-L GND #PWR?
-U 1 1 5B4D2FF4
-P 4400 4725
-F 0 "#PWR?" H 4400 4475 50  0001 C CNN
-F 1 "GND" H 4400 4575 50  0000 C CNN
-F 2 "" H 4400 4725 50  0001 C CNN
-F 3 "" H 4400 4725 50  0001 C CNN
-	1    4400 4725
-	1    0    0    -1
-$EndComp
-$Comp
-L GND #PWR?
-U 1 1 5B4D302C
-P 5175 4725
-F 0 "#PWR?" H 5175 4475 50  0001 C CNN
-F 1 "GND" H 5175 4575 50  0000 C CNN
-F 2 "" H 5175 4725 50  0001 C CNN
-F 3 "" H 5175 4725 50  0001 C CNN
-	1    5175 4725
-	1    0    0    -1
-$EndComp
-$Comp
-L GND #PWR?
-U 1 1 5B4D532A
-P 4025 5725
-F 0 "#PWR?" H 4025 5475 50  0001 C CNN
-F 1 "GND" H 4025 5575 50  0000 C CNN
-F 2 "" H 4025 5725 50  0001 C CNN
-F 3 "" H 4025 5725 50  0001 C CNN
-	1    4025 5725
-	1    0    0    -1
-$EndComp
 Wire Wire Line
 	6150 2250 6300 2250
@@
 	6150 2250 6150 2600
 Connection ~ 4950 2425
+$Comp
+L GNDPWR #PWR?
+U 1 1 5B59FA75
+P 4400 4725
+F 0 "#PWR?" H 4400 4525 50  0001 C CNN
+F 1 "GNDPWR" H 4400 4595 50  0000 C CNN
+F 2 "" H 4400 4675 50  0001 C CNN
+F 3 "" H 4400 4675 50  0001 C CNN
+	1    4400 4725
+	1    0    0    -1
+$EndComp
+$Comp
+L GNDPWR #PWR?
+U 1 1 5B59FADB
+P 5175 4725
+F 0 "#PWR?" H 5175 4525 50  0001 C CNN
+F 1 "GNDPWR" H 5175 4595 50  0000 C CNN
+F 2 "" H 5175 4675 50  0001 C CNN
+F 3 "" H 5175 4675 50  0001 C CNN
+	1    5175 4725
+	1    0    0    -1
+$EndComp
+$Comp
+L GNDPWR #PWR?
+U 1 1 5B59FB10
+P 4950 5550
+F 0 "#PWR?" H 4950 5350 50  0001 C CNN
+F 1 "GNDPWR" H 4950 5420 50  0000 C CNN
+F 2 "" H 4950 5500 50  0001 C CNN
+F 3 "" H 4950 5500 50  0001 C CNN
+	1    4950 5550
+	1    0    0    -1
+$EndComp
+$Comp
+L GNDPWR #PWR?
+U 1 1 5B59FB99
+P 4025 5725
+F 0 "#PWR?" H 4025 5525 50  0001 C CNN
+F 1 "GNDPWR" H 4025 5595 50  0000 C CNN
+F 2 "" H 4025 5675 50  0001 C CNN
+F 3 "" H 4025 5675 50  0001 C CNN
+	1    4025 5725
+	1    0    0    -1
+$EndComp
 $EndSCHEMATC

Commit message: Power_dist could be monitor battery voltage and system current
Parts:
- removed C?: 0.47uF, Capacitors_SMD:C_0603_HandSoldering, symbol C_Small
- removed D?: BZT52c12s, Diodes_SMD:D_SOD-323_HandSoldering, symbol D_Zener
- added C16: 0.47uF, Capacitors_SMD:C_1206_HandSoldering, symbol CP_Small
- added D14: BZT52c12s, Diodes_SMD:D_SOD-323_HandSoldering, symbol D_Zener_Small
- R29: renamed from R?; value 200k -> 2.2k
- R30: renamed from R?; value 1.8M -> 18k
- gave numbers to parts that had none: 10
Changed lines of the file:
@@
 Current_OUT
 $Comp
-L R R?
+L R R33
 U 1 1 5B4C6A59
 P 6450 2250
-F 0 "R?" V 6530 2250 50  0000 C CNN
+F 0 "R33" V 6530 2250 50  0000 C CNN
 F 1 "5" V 6450 2250 50  0000 C CNN
 F 2 "zeabus:THK45" V 6380 2250 50  0001 C CNN
@@
 $EndComp
 $Comp
-L R R?
+L R R34
 U 1 1 5B4C6AA7
 P 6450 2600
-F 0 "R?" V 6530 2600 50  0000 C CNN
+F 0 "R34" V 6530 2600 50  0000 C CNN
 F 1 "5" V 6450 2600 50  0000 C CNN
 F 2 "zeabus:THK45" V 6380 2600 50  0001 C CNN
@@
 $EndComp
 $Comp
-L TL331 U?
+L TL331 U7
 U 1 1 5B4C9184
 P 5050 5175
-F 0 "U?" H 5200 5325 50  0000 C CNN
+F 0 "U7" H 5200 5325 50  0000 C CNN
 F 1 "TL331" H 5200 5025 50  0000 C CNN
 F 2 "TO_SOT_Packages_SMD:SOT-23-5" H 5050 5175 50  0001 C CNN
@@
 $EndComp
 $Comp
-L IPB180P04P4-03 Q?
+L IPB180P04P4-03 Q3
 U 1 1 5B4C8D9C
 P 6450 3200
-F 0 "Q?" H 6250 3500 50  0000 L CNN
+F 0 "Q3" H 6250 3500 50  0000 L CNN
 F 1 "IPB180P04P4-03" H 6250 2850 50  0000 L CNN
 F 2 "TO_SOT_Packages_SMD:TO-263-6" H 6450 2750 50  0001 C CIN
@@
 $EndComp
 $Comp
-L IPB180P04P4-03 Q?
+L IPB180P04P4-03 Q4
 U 1 1 5B4C99CC
 P 6450 4075
-F 0 "Q?" H 6250 4375 50  0000 L CNN
+F 0 "Q4" H 6250 4375 50  0000 L CNN
 F 1 "IPB180P04P4-03" H 6250 3725 50  0000 L CNN
 F 2 "TO_SOT_Packages_SMD:TO-263-6" H 6450 3625 50  0001 C CIN
@@
 $EndComp
 $Comp
-L R R?
+L R R29
 U 1 1 5B4CB67A
 P 4400 3875
-F 0 "R?" V 4480 3875 50  0000 C CNN
-F 1 "200k" V 4400 3875 50  0000 C CNN
+F 0 "R29" V 4480 3875 50  0000 C CNN
+F 1 "2.2k" V 4400 3875 50  0000 C CNN
 F 2 "Resistors_SMD:R_0603_HandSoldering" V 4330 3875 50  0001 C CNN
 F 3 "" H 4400 3875 50  0001 C CNN
@@
 $EndComp
 $Comp
-L R R?
+L R R30
 U 1 1 5B4CB6EB
 P 4400 4475
-F 0 "R?" V 4480 4475 50  0000 C CNN
-F 1 "1.8M" V 4400 4475 50  0000 C CNN
+F 0 "R30" V 4480 4475 50  0000 C CNN
+F 1 "18k" V 4400 4475 50  0000 C CNN
 F 2 "Resistors_SMD:R_0603_HandSoldering" V 4330 4475 50  0001 C CNN
 F 3 "" H 4400 4475 50  0001 C CNN
@@
 $EndComp
 $Comp
-L R R?
+L R R28
 U 1 1 5B4CB8CC
 P 4025 4925
-F 0 "R?" V 4105 4925 50  0000 C CNN
+F 0 "R28" V 4105 4925 50  0000 C CNN
 F 1 "1M" V 4025 4925 50  0000 C CNN
 F 2 "Resistors_SMD:R_0603_HandSoldering" V 3955 4925 50  0001 C CNN
@@
 $EndComp
 $Comp
-L C_Small C?
-U 1 1 5B4CB996
-P 4025 5500
-F 0 "C?" H 4035 5570 50  0000 L CNN
-F 1 "0.47uF" H 4035 5420 50  0000 L CNN
-F 2 "Capacitors_SMD:C_0603_HandSoldering" H 4025 5500 50  0001 C CNN
-F 3 "" H 4025 5500 50  0001 C CNN
-	1    4025 5500
-	1    0    0    -1
-$EndComp
-$Comp
-L R R?
+L R R32
 U 1 1 5B4CC1F1
 P 5600 4950
-F 0 "R?" V 5680 4950 50  0000 C CNN
+F 0 "R32" V 5680 4950 50  0000 C CNN
 F 1 "10k" V 5600 4950 50  0000 C CNN
 F 2 "Resistors_SMD:R_0603_HandSoldering" V 5530 4950 50  0001 C CNN
@@
 $EndComp
 $Comp
-L C_Small C?
+L C_Small C17
 U 1 1 5B4CCD3A
 P 5175 4525
-F 0 "C?" H 5185 4595 50  0000 L CNN
+F 0 "C17" H 5185 4595 50  0000 L CNN
 F 1 "0.1uF" H 5185 4445 50  0000 L CNN
 F 2 "Capacitors_SMD:C_0603_HandSoldering" H 5175 4525 50  0001 C CNN
@@
 $EndComp
 $Comp
-L D_Zener D?
-U 1 1 5B4CD68B
-P 6450 4700
-F 0 "D?" H 6450 4800 50  0000 C CNN
-F 1 "BZT52c12s" H 6450 4600 50  0000 C CNN
-F 2 "Diodes_SMD:D_SOD-323_HandSoldering" H 6450 4700 50  0001 C CNN
-F 3 "" H 6450 4700 50  0001 C CNN
-	1    6450 4700
-	1    0    0    -1
-$EndComp
-$Comp
-L R R?
+L R R35
 U 1 1 5B4CEB07
 P 6900 4950
-F 0 "R?" V 6980 4950 50  0000 C CNN
+F 0 "R35" V 6980 4950 50  0000 C CNN
 F 1 "2.2k" V 6900 4950 50  0000 C CNN
 F 2 "Resistors_SMD:R_0603_HandSoldering" V 6830 4950 50  0001 C CNN
@@
 $EndComp
 $Comp
-L R R?
+L R R31
 U 1 1 5B4D20C2
 P 4950 4050
-F 0 "R?" V 5030 4050 50  0000 C CNN
+F 0 "R31" V 5030 4050 50  0000 C CNN
 F 1 "10" V 4950 4050 50  0000 C CNN
 F 2 "Resistors_SMD:R_0603_HandSoldering" V 4880 4050 50  0001 C CNN
@@
 	4950 5550 4950 5475
 Wire Wire Line
-	5825 4700 6300 4700
+	5825 4700 6350 4700
 Connection ~ 5825 3875
 Wire Wire Line
@@
 Connection ~ 6900 4175
 Wire Wire Line
-	6600 4700 6900 4700
+	6550 4700 6900 4700
 Connection ~ 6900 4700
 Wire Wire Line
@@
 Connection ~ 4950 2425
 $Comp
-L GNDPWR #PWR?
+L GNDPWR #PWR64
 U 1 1 5B59FA75
 P 4400 4725
-F 0 "#PWR?" H 4400 4525 50  0001 C CNN
+F 0 "#PWR64" H 4400 4525 50  0001 C CNN
 F 1 "GNDPWR" H 4400 4595 50  0000 C CNN
 F 2 "" H 4400 4675 50  0001 C CNN
@@
 $EndComp
 $Comp
-L GNDPWR #PWR?
+L GNDPWR #PWR66
 U 1 1 5B59FADB
 P 5175 4725
-F 0 "#PWR?" H 5175 4525 50  0001 C CNN
+F 0 "#PWR66" H 5175 4525 50  0001 C CNN
 F 1 "GNDPWR" H 5175 4595 50  0000 C CNN
 F 2 "" H 5175 4675 50  0001 C CNN
@@
 $EndComp
 $Comp
-L GNDPWR #PWR?
+L GNDPWR #PWR65
 U 1 1 5B59FB10
 P 4950 5550
-F 0 "#PWR?" H 4950 5350 50  0001 C CNN
+F 0 "#PWR65" H 4950 5350 50  0001 C CNN
 F 1 "GNDPWR" H 4950 5420 50  0000 C CNN
 F 2 "" H 4950 5500 50  0001 C CNN
@@
 $EndComp
 $Comp
-L GNDPWR #PWR?
+L GNDPWR #PWR63
 U 1 1 5B59FB99
 P 4025 5725
-F 0 "#PWR?" H 4025 5525 50  0001 C CNN
+F 0 "#PWR63" H 4025 5525 50  0001 C CNN
 F 1 "GNDPWR" H 4025 5595 50  0000 C CNN
 F 2 "" H 4025 5675 50  0001 C CNN
@@
 	1    0    0    -1
 $EndComp
+$Comp
+L D_Zener_Small D14
+U 1 1 5B6BF01A
+P 6450 4700
+F 0 "D14" H 6450 4790 50  0000 C CNN
+F 1 "BZT52c12s" H 6450 4610 50  0000 C CNN
+F 2 "Diodes_SMD:D_SOD-323_HandSoldering" V 6450 4700 50  0001 C CNN
+F 3 "" V 6450 4700 50  0001 C CNN
+	1    6450 4700
+	1    0    0    -1
+$EndComp
+$Comp
+L CP_Small C16
+U 1 1 5B5B6DCE
+P 4025 5500
+F 0 "C16" H 4035 5570 50  0000 L CNN
+F 1 "0.47uF" H 4035 5420 50  0000 L CNN
+F 2 "Capacitors_SMD:C_1206_HandSoldering" H 4025 5500 50  0001 C CNN
+F 3 "" H 4025 5500 50  0001 C CNN
+	1    4025 5500
+	1    0    0    -1
+$EndComp
