File: Circuit/Power_dist/Power-Controller.sch (KiCad schematic (older format))
At the start: 48 parts, among them P15 USB_B, U1 93LC56BT-I/OT, U2 FT232H, U3 ACPL-247-500E, U4 ACPL-247-500E, Y1 12MHz

Commit message: power line and data line source of Power_Controller on Power_dist could be manual selected
Parts:
- removed P15: USB_B, Connectors:USB_Mini-B, symbol USB_OTG
- U? (x2): footprint (none) -> zeabus:SO16_4.4x10.3mm_Pitch1.27mm
- Y1: footprint Crystals:Crystal_SMD_Abracon_ABM3-2pin_5.0x3.2mm -> Crystals:Crystal_SMD_Abracon_ABM3-2pin_5.0x3.2mm_HandSoldering
Connections:
- net labels added: +3V3_CTRL, +5V_CTRL
- net labels removed: VBUS
- wire segments 177 -> 173
- no-connect marks 14 -> 13
Other:
- moved on the sheet: C1, R16, R17, R18, R19, U1

Commit message: Power_dist could be monitor battery voltage and system current
Parts:
- added C43, C44, C45, C46, C48, C49: 0.1uF, Capacitors_SMD:C_0603_HandSoldering, symbol C_Small
- added C47: 1uF, Capacitors_SMD:C_1206_HandSoldering, symbol CP_Small
- added L5: 600R 500mA, Capacitors_SMD:C_0603_HandSoldering, symbol L_Core_Iron
- added Q10: BSS138, TO_SOT_Packages_SMD:SOT-23, symbol BSS138
- added R59: 1k, Resistors_SMD:R_0603_HandSoldering, symbol R
- added R60: 1M, Resistors_SMD:R_0603_HandSoldering, symbol R
- added R61, R62: 150, Resistors_SMD:R_0603_HandSoldering, symbol R
- added R63, R64: 10k, Resistors_SMD:R_0603_HandSoldering, symbol R
- added unit 2 of U13
- added unit 3 of U13
- added U14: Si8660BA-B-IS1, Housings_SOIC:SOIC-16_3.9x9.9mm_Pitch1.27mm, symbol Si8660BA-B-IS1
- added U15: TS5A23159, Housings_SSOP:MSOP-10_3x3mm_Pitch0.5mm, symbol TS5A23159
- added U16, U17: ADC101S021, TO_SOT_Packages_SMD:SOT-23-6_Handsoldering, symbol ADC101S021
- gave numbers to parts that had none: 5
- renumbered C1 to C25, C2 to C26, C3 to C27, C4 to C28, C5 to C29, C6 to C30, C7 to C31, C8 to C32, C9 to C33, C10 to C34, C11 to C35, C12 to C36, C13 to C37, C14 to C38, C15 to C39, C16 to C40, C17 to C41, C18 to C42, JP2 to JP3, L1 to L2, L2 to L3, L3 to L4, R22 to R47, R16 to R48, R17 to R49, R18 to R50, R23 to R51, R24 to R52, R19 to R53, R20 to R56, R21 to R57, R25 to R65, R26 to R66, R27 to R67, R28 to R68, U1 to U10, U3 to U11, U2 to U12, U4 to U13, U4 to U18
Connections:
- net labels added: +5P, +5VD, +5V_PWR, ADC1, ADC1_Vin, ADC2, ADC2_Vin, CS_ADC1, CS_ADC2, Current_Sense_OUT, D_VBatt1, D_VBatt2, D_VPWR, GPIO_SW, MCLK, MISO, SCLK, SW1, SW2, SW3, SW4, SW5, ~PWRREN
- net labels removed: +3.3V
- wire segments 173 -> 259
- no-connect marks 13 -> 14
Other:
- moved on the sheet: C25, C26, C27, C28, C29, C30, C31, C32, C33, C34, C35, C36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

Commit message: organzied datasheets of Power_dist
Parts:
- removed U11, U13, U18: ACPL-247-500E, zeabus:SO16_4.4x10.3mm_Pitch1.27mm, symbol ACPL-247-500E
- added U11, U13, U18: ACPL-247-560E, zeabus:SO16_4.4x10.3mm_Pitch1.27mm, symbol ACPL-247-560E
Changed lines of the file:
@@
-$EndComp
-$Comp
-L ACPL-247-500E U13
-U 1 1 58C66F21
-P 5025 7250
-F 0 "U13" H 4825 7450 50  0000 L CNN
-F 1 "ACPL-247-500E" H 4725 7050 50  0000 L CNN
-F 2 "zeabus:SO16_4.4x10.3mm_Pitch1.27mm" H 5025 7250 50  0001 L CNN
-F 3 "" H 5025 7250 50  0000 L CNN
-	1    5025 7250
-	1    0    0    -1
 $EndComp
 $Comp
@@
 $EndComp
 $Comp
-L ACPL-247-500E U13
-U 4 1 58C67F4F
-P 10500 950
-F 0 "U13" H 10300 1150 50  0000 L CNN
-F 1 "ACPL-247-500E" H 10200 750 50  0000 L CNN
-F 2 "zeabus:SO16_4.4x10.3mm_Pitch1.27mm" H 10500 950 50  0001 L CNN
-F 3 "" H 10500 950 50  0000 L CNN
-	4    10500 950
-	1    0    0    -1
-$EndComp
-$Comp
 L R R66
 U 1 1 58C67F55
@@
 $EndComp
 $Comp
-L ACPL-247-500E U18
-U 1 1 58C68069
-P 10500 1625
-F 0 "U18" H 10300 1825 50  0000 L CNN
-F 1 "ACPL-247-500E" H 10200 1425 50  0000 L CNN
-F 2 "zeabus:SO16_4.4x10.3mm_Pitch1.27mm" H 10500 1625 50  0001 L CNN
-F 3 "" H 10500 1625 50  0000 L CNN
-	1    10500 1625
-	1    0    0    -1
-$EndComp
-$Comp
 L R R67
 U 1 1 58C6806F
@@
 $EndComp
 $Comp
-L ACPL-247-500E U18
-U 2 1 58C6807E
-P 10500 2300
-F 0 "U18" H 10300 2500 50  0000 L CNN
-F 1 "ACPL-247-500E" H 10200 2100 50  0000 L CNN
-F 2 "zeabus:SO16_4.4x10.3mm_Pitch1.27mm" H 10500 2300 50  0001 L CNN
-F 3 "" H 10500 2300 50  0000 L CNN
-	2    10500 2300
-	1    0    0    -1
-$EndComp
-$Comp
 L R R68
 U 1 1 58C68084
@@
 $EndComp
 $Comp
-L ACPL-247-500E U11
-U 1 1 58C68C6D
-P 1575 6575
-F 0 "U11" H 1375 6775 50  0000 L CNN
-F 1 "ACPL-247-500E" H 1275 6375 50  0000 L CNN
-F 2 "zeabus:SO16_4.4x10.3mm_Pitch1.27mm" H 1575 6575 50  0001 L CNN
-F 3 "" H 1575 6575 50  0000 L CNN
-	1    1575 6575
-	1    0    0    -1
-$EndComp
-$Comp
 L R R47
 U 1 1 58C68C73
@@
 $EndComp
 $Comp
-L ACPL-247-500E U11
-U 3 1 58C68C82
-P 3300 6575
-F 0 "U11" H 3100 6775 50  0000 L CNN
-F 1 "ACPL-247-500E" H 3000 6375 50  0000 L CNN
-F 2 "zeabus:SO16_4.4x10.3mm_Pitch1.27mm" H 3300 6575 50  0001 L CNN
-F 3 "" H 3300 6575 50  0000 L CNN
-	3    3300 6575
-	1    0    0    -1
-$EndComp
-$Comp
 L R R51
 U 1 1 58C68C88
@@
 $EndComp
 $Comp
-L ACPL-247-500E U11
-U 2 1 58C68C97
-P 1575 7250
-F 0 "U11" H 1375 7450 50  0000 L CNN
-F 1 "ACPL-247-500E" H 1275 7050 50  0000 L CNN
-F 2 "zeabus:SO16_4.4x10.3mm_Pitch1.27mm" H 1575 7250 50  0001 L CNN
-F 3 "" H 1575 7250 50  0000 L CNN
-	2    1575 7250
-	1    0    0    -1
-$EndComp
-$Comp
 L R R9'1
 U 1 1 58C68C9D
@@
 	1    1075 7150
 	0    -1   -1   0
-$EndComp
-$Comp
-L ACPL-247-500E U11
-U 4 1 58C68CAC
-P 3300 7250
-F 0 "U11" H 3100 7450 50  0000 L CNN
-F 1 "ACPL-247-500E" H 3000 7050 50  0000 L CNN
-F 2 "zeabus:SO16_4.4x10.3mm_Pitch1.27mm" H 3300 7250 50  0001 L CNN
-F 3 "" H 3300 7250 50  0000 L CNN
-	4    3300 7250
-	1    0    0    -1
 $EndComp
 $Comp
@@
 Text HLabel 1275 850  0    60   UnSpc ~ 0
 +PWR
-$Comp
-L ACPL-247-500E U18
-U 3 1 5B53470F
-P 10500 2975
-F 0 "U18" H 10300 3175 50  0000 L CNN
-F 1 "ACPL-247-500E" H 10200 2775 50  0000 L CNN
-F 2 "zeabus:SO16_4.4x10.3mm_Pitch1.27mm" H 10500 2975 50  0001 L CNN
-F 3 "" H 10500 2975 50  0000 L CNN
-	3    10500 2975
-	1    0    0    -1
-$EndComp
-$Comp
-L ACPL-247-500E U18
-U 4 1 5B534AC9
-P 10500 3675
-F 0 "U18" H 10300 3875 50  0000 L CNN
-F 1 "ACPL-247-500E" H 10200 3475 50  0000 L CNN
-F 2 "zeabus:SO16_4.4x10.3mm_Pitch1.27mm" H 10500 3675 50  0001 L CNN
-F 3 "" H 10500 3675 50  0000 L CNN
-	4    10500 3675
-	1    0    0    -1
-$EndComp
 $Comp
 L R R58
@@
 	6975 5825 7750 5825
 $Comp
-L ACPL-247-500E U13
-U 2 1 5B6491A2
-P 7575 2950
-F 0 "U13" H 7375 3150 50  0000 L CNN
-F 1 "ACPL-247-500E" H 7275 2750 50  0000 L CNN
-F 2 "zeabus:SO16_4.4x10.3mm_Pitch1.27mm" H 7575 2950 50  0001 L CNN
-F 3 "" H 7575 2950 50  0000 L CNN
-	2    7575 2950
-	1    0    0    -1
-$EndComp
-$Comp
-L ACPL-247-500E U13
-U 3 1 5B64924D
-P 7575 4200
-F 0 "U13" H 7375 4400 50  0000 L CNN
-F 1 "ACPL-247-500E" H 7275 4000 50  0000 L CNN
-F 2 "zeabus:SO16_4.4x10.3mm_Pitch1.27mm" H 7575 4200 50  0001 L CNN
-F 3 "" H 7575 4200 50  0000 L CNN
-	3    7575 4200
-	1    0    0    -1
-$EndComp
-$Comp
 L +5VD #PWR80
 U 1 1 5B53F88E
@@
 Wire Wire Line
 	3025 3400 3125 3400
+$Comp
+L ACPL-247-560E U11
+U 1 1 5B540179
+P 1575 6575
+F 0 "U11" H 1375 6775 50  0000 L CNN
+F 1 "ACPL-247-560E" H 1275 6375 50  0000 L CNN
+F 2 "zeabus:SO16_4.4x10.3mm_Pitch1.27mm" H 1575 6575 50  0001 L CNN
+F 3 "" H 1575 6575 50  0000 L CNN
+	1    1575 6575
+	1    0    0    -1
+$EndComp
+$Comp
+L ACPL-247-560E U11
+U 2 1 5B54039B
+P 1575 7250
+F 0 "U11" H 1375 7450 50  0000 L CNN
+F 1 "ACPL-247-560E" H 1275 7050 50  0000 L CNN
+F 2 "zeabus:SO16_4.4x10.3mm_Pitch1.27mm" H 1575 7250 50  0001 L CNN
+F 3 "" H 1575 7250 50  0000 L CNN
+	2    1575 7250
+	1    0    0    -1
+$EndComp
+$Comp
+L ACPL-247-560E U11
+U 3 1 5B54047E
+P 3300 6575
+F 0 "U11" H 3100 6775 50  0000 L CNN
+F 1 "ACPL-247-560E" H 3000 6375 50  0000 L CNN
+F 2 "zeabus:SO16_4.4x10.3mm_Pitch1.27mm" H 3300 6575 50  0001 L CNN
+F 3 "" H 3300 6575 50  0000 L CNN
+	3    3300 6575
+	1    0    0    -1
+$EndComp
+$Comp
+L ACPL-247-560E U11
+U 4 1 5B540551
+P 3300 7250
+F 0 "U11" H 3100 7450 50  0000 L CNN
+F 1 "ACPL-247-560E" H 3000 7050 50  0000 L CNN
+F 2 "zeabus:SO16_4.4x10.3mm_Pitch1.27mm" H 3300 7250 50  0001 L CNN
+F 3 "" H 3300 7250 50  0000 L CNN
+	4    3300 7250
+	1    0    0    -1
+$EndComp
+$Comp
+L ACPL-247-560E U13
+U 1 1 5B544CC9
+P 5025 7250
+F 0 "U13" H 4825 7450 50  0000 L CNN
+F 1 "ACPL-247-560E" H 4725 7050 50  0000 L CNN
+F 2 "zeabus:SO16_4.4x10.3mm_Pitch1.27mm" H 5025 7250 50  0001 L CNN
+F 3 "" H 5025 7250 50  0000 L CNN
+	1    5025 7250
+	1    0    0    -1
+$EndComp
+$Comp
+L ACPL-247-560E U13
+U 2 1 5B545F23
+P 7575 2950
+F 0 "U13" H 7375 3150 50  0000 L CNN
+F 1 "ACPL-247-560E" H 7275 2750 50  0000 L CNN
+F 2 "zeabus:SO16_4.4x10.3mm_Pitch1.27mm" H 7275 3050 50  0001 L CNN
+F 3 "" H 7575 2950 50  0000 L CNN
+	2    7575 2950
+	1    0    0    -1
+$EndComp
+$Comp
+L ACPL-247-560E U13
+U 3 1 5B546181
+P 7575 4200
+F 0 "U13" H 7375 4400 50  0000 L CNN
+F 1 "ACPL-247-560E" H 7275 4000 50  0000 L CNN
+F 2 "zeabus:SO16_4.4x10.3mm_Pitch1.27mm" H 7275 4300 50  0001 L CNN
+F 3 "" H 7575 4200 50  0000 L CNN
+	3    7575 4200
+	1    0    0    -1
+$EndComp
+$Comp
+L ACPL-247-560E U13
+U 4 1 5B5477C3
+P 10500 950
+F 0 "U13" H 10300 1150 50  0000 L CNN
+F 1 "ACPL-247-560E" H 10200 750 50  0000 L CNN
+F 2 "zeabus:SO16_4.4x10.3mm_Pitch1.27mm" H 10200 1050 50  0001 L CNN
+F 3 "" H 10500 950 50  0000 L CNN
+	4    10500 950
+	1    0    0    -1
+$EndComp
+$Comp
+L ACPL-247-560E U18
+U 1 1 5B5482CA
+P 10500 1625
+F 0 "U18" H 10300 1825 50  0000 L CNN
+F 1 "ACPL-247-560E" H 10200 1425 50  0000 L CNN
+F 2 "zeabus:SO16_4.4x10.3mm_Pitch1.27mm" H 10200 1725 50  0001 L CNN
+F 3 "" H 10500 1625 50  0000 L CNN
+	1    10500 1625
+	1    0    0    -1
+$EndComp
+$Comp
+L ACPL-247-560E U18
+U 2 1 5B54B3B1
+P 10500 2300
+F 0 "U18" H 10300 2500 50  0000 L CNN
+F 1 "ACPL-247-560E" H 10200 2100 50  0000 L CNN
+F 2 "zeabus:SO16_4.4x10.3mm_Pitch1.27mm" H 10200 2400 50  0001 L CNN
+F 3 "" H 10500 2300 50  0000 L CNN
+	2    10500 2300
+	1    0    0    -1
+$EndComp
+$Comp
+L ACPL-247-560E U18
+U 3 1 5B54B4B4
+P 10500 2975
+F 0 "U18" H 10300 3175 50  0000 L CNN
+F 1 "ACPL-247-560E" H 10200 2775 50  0000 L CNN
+F 2 "zeabus:SO16_4.4x10.3mm_Pitch1.27mm" H 10200 3075 50  0001 L CNN
+F 3 "" H 10500 2975 50  0000 L CNN
+	3    10500 2975
+	1    0    0    -1
+$EndComp
+$Comp
+L ACPL-247-560E U18
+U 4 1 5B54B5B5
+P 10500 3675
+F 0 "U18" H 10300 3875 50  0000 L CNN
+F 1 "ACPL-247-560E" H 10200 3475 50  0000 L CNN
+F 2 "zeabus:SO16_4.4x10.3mm_Pitch1.27mm" H 10200 3775 50  0001 L CNN
+F 3 "" H 10500 3675 50  0000 L CNN
+	4    10500 3675
+	1    0    0    -1
+$EndComp
 $EndSCHEMATC
