File: Circuit/board-drive/board-drive.kicad_pcb (KiCad board)
At the start: 2 copper layers, 19 parts, among them P1 XT30, P2 XT30, P3 XT30, P4 XT30, P5 XT30, P6 XT30, P7 XT30, P8 XT30, U1 Pololu_Maestro12, U10 Pololu_SimpleMotorController2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, U11 Pololu_SimpleMotorController2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, U2 Si8660BA-B-IS1, U3 Si8660BA-B-IS1, U4 Pololu_SimpleMotorController2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, U5 Pololu_SimpleMotorController2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, U6 Pololu_SimpleMotorController2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, U7 Pololu_SimpleMotorController2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, U8 Pololu_SimpleMotorController2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, U9 Pololu_SimpleMotorController2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

Commit message: PCB routed prototype1
Parts:
- added P10: XT60, zeabus:XT60, F.Cu at (63.2, 104.4)
- added P9: XT60, zeabus:XT60, F.Cu at (63.2, 95.0)
- added U12: Pololu_SimpleMotorController24v23_withnoPowerDist, zeabus:pololu_motorcontroller24v23, B.Cu at (83.1, 118.4)
- added U13: Pololu_SimpleMotorController24v23_withnoPowerDist, zeabus:pololu_motorcontroller24v23, B.Cu at (141.5, 119.1)
- added U14: Pololu_SimpleMotorController24v23_withnoPowerDist, zeabus:pololu_motorcontroller24v23, B.Cu at (143.3, 118.4)
- added U15: Pololu_SimpleMotorController24v23_withnoPowerDist, zeabus:pololu_motorcontroller24v23, B.Cu at (201.7, 119.1)
- added U16: PowerDist_WiretoBoard, zeabus:PowerDist_WiretoBoard, B.Cu at (93.4, 66.7)
- added U17: PowerDist_WiretoBoard, zeabus:PowerDist_WiretoBoard, B.Cu at (134.2, 66.7)
- added U18: PowerDist_WiretoBoard, zeabus:PowerDist_WiretoBoard, B.Cu at (175.1, 66.7)
- added U19: PowerDist_WiretoBoard, zeabus:PowerDist_WiretoBoard, B.Cu at (216.5, 66.4)
- U10, U11, U8, U9: value Pololu_SimpleMotorController24v23 -> PowerDist_WiretoBoard; footprint zeabus:pololu_motorcontroller24v23 -> zeabus:PowerDist_WiretoBoard
- U2, U3: moved to B.Cu
- U4, U5, U6, U7: value Pololu_SimpleMotorController24v23 -> Pololu_SimpleMotorController24v23_withnoPowerDist
- moved U7 150.6 mm to (143.3, 119.1)
- moved U10 98.5 mm to (129.6, 66.7)
- moved U6 94.0 mm to (201.7, 118.4), turned to 180 degrees
- moved U5 93.9 mm to (83.1, 119.1)
- moved U4 93.6 mm to (141.5, 118.4), turned to 180 degrees
- moved P2 88.8 mm to (81.0, 61.0), turned to 270 degrees
- moved P3 88.8 mm to (93.8, 61.0), turned to 270 degrees
- moved P4 87.6 mm to (106.4, 61.0), turned to 270 degrees
- moved P1 86.2 mm to (68.4, 61.0), turned to 270 degrees
- moved U1 76.1 mm to (79.6, 148.1), turned to 180 degrees
- moved U2 68.7 mm to (68.3, 135.8), turned to 90 degrees
- moved U8 52.8 mm to (48.1, 66.6)
- moved U11 51.1 mm to (170.9, 66.6)
- moved U9 47.6 mm to (88.8, 66.7)
- moved P5 34.8 mm to (154.7, 60.7), turned to 270 degrees
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Connections:
- U2 pad 2: Net-(U1-Pad~) -> Net-(U1-Pad11)
- U2 pad 3: Net-(U1-Pad~) -> Net-(U1-Pad12)
- U2 pad 4: Net-(U1-Pad~) -> Net-(U1-Pad13)
- U2 pad 5: Net-(U1-Pad~) -> Net-(U1-Pad14)
- U2 pad 6: Net-(U1-Pad~) -> Net-(U1-Pad15)
- U2 pad 7: Net-(U1-Pad~) -> Net-(U1-Pad16)
- U3 pad 15: /signl6 -> /signal6
- U3 pad 2: Net-(U1-Pad~) -> Net-(U1-Pad17)
- U3 pad 3: Net-(U1-Pad~) -> Net-(U1-Pad18)
- U3 pad 4: Net-(U1-Pad~) -> Net-(U1-Pad19)
- U3 pad 5: Net-(U1-Pad~) -> Net-(U1-Pad20)
- U3 pad 6: Net-(U1-Pad~) -> Net-(U1-Pad21)
- U3 pad 7: Net-(U1-Pad~) -> Net-(U1-Pad22)
Routing:
- net /BATTIN_1: track 0.00 -> 234.3 mm
- net /BATTIN_0: track 0.00 -> 182.7 mm
- net /signal9: track 0.00 -> 159.2 mm, vias 0 -> 1
- net /signal2: track 0.00 -> 154.0 mm, vias 0 -> 1
- net /signal0: track 0.00 -> 94.7 mm, vias 0 -> 1
- net /signal8: track 0.00 -> 93.5 mm, vias 0 -> 1
- net /signal3: track 0.00 -> 87.4 mm, vias 0 -> 1
- net /signal7: track 0.00 -> 79.9 mm, vias 0 -> 1
- net GNDA: track 0.00 -> 79.6 mm, vias 0 -> 1
- net +5V: track 0.00 -> 28.8 mm
- net /OUTA_5: track 0.00 -> 26.9 mm
- net /OUTA_7: track 0.00 -> 26.8 mm
- net /OUTB_2: track 0.00 -> 24.6 mm
- net /signal6: track 0.00 -> 24.0 mm, vias 0 -> 1
- net /OUTA_2: track 0.00 -> 24.0 mm
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- added copper zone on B.Cu, net /BATTGND
- added copper zone on F.Cu, net GNDA
- added copper zone on B.Cu, net GNDD
Other:
- board outline added: 164.4 x 93.2 mm
- net class Default: clearance 0.2 -> 0.1524; trace_width 0.25 -> 0.1524; via_drill 0.4 -> 0.381
- rule trace_clearance: 0.2 -> 0.1524
- rule trace_min: 0.2 -> 0.1524

Commit message: fix bug
Parts:
- added REF**: MountingHole_3.2mm_M3, Mounting_Holes:MountingHole_3.2mm_M3, F.Cu at (55.2, 62.1)
- added REF**: MountingHole_3.2mm_M3, Mounting_Holes:MountingHole_3.2mm_M3, F.Cu at (209.6, 62.2)
- added REF**: MountingHole_3.2mm_M3, Mounting_Holes:MountingHole_3.2mm_M3, F.Cu at (209.6, 146.1)
Routing:
- net GNDA: track 79.6 -> 22.0 mm, vias 1 -> 2
- net Net-(U2-Pad16): track 20.0 -> 40.9 mm, vias 0 -> 2
- net /signal2: track 154.0 -> 173.1 mm
- net GNDD: track 0.00 -> 16.8 mm
- net /signal8: track 93.5 -> 88.8 mm
- net +5V: track 28.8 -> 26.3 mm, vias 0 -> 2
- net /signal1: track 23.9 -> 26.3 mm
- net /signal0: track 94.7 -> 92.6 mm
- net /signal7: track 79.9 -> 81.4 mm
- net /signal9: track 159.2 -> 158.2 mm
