File: Circuit/Backplane/Backplane.sch (KiCad schematic (older format))
At the start: 65 parts

Commit message: relocatedGeneral
Parts:
- J?: value General_Power_Source -> general_power_source
- P?: value General -> general
Connections:
- net genPow: now reaches J?.2 (Pin_2), P?.1 (P1)
Other:
- moved on the sheet: P?
Changed lines of the file:
@@
 L GND #PWR?
 U 1 1 5A65DB26
-P 1850 6650
-F 0 "#PWR?" H 1850 6400 50  0001 C CNN
-F 1 "GND" H 1850 6500 50  0000 C CNN
-F 2 "" H 1850 6650 50  0001 C CNN
-F 3 "" H 1850 6650 50  0001 C CNN
-	1    1850 6650
+P 5500 7500
+F 0 "#PWR?" H 5500 7250 50  0001 C CNN
+F 1 "GND" H 5500 7350 50  0000 C CNN
+F 2 "" H 5500 7500 50  0001 C CNN
+F 3 "" H 5500 7500 50  0001 C CNN
+	1    5500 7500
 	1    0    0    -1
 $EndComp
@@
 L XT30 P?
 U 1 1 5A65DB20
-P 2150 6550
-F 0 "P?" H 2150 6700 50  0000 C CNN
-F 1 "General" H 2150 6400 50  0000 C CNN
-F 2 "" H 2150 6550 60  0000 C CNN
-F 3 "" H 2150 6550 60  0000 C CNN
-	1    2150 6550
+P 5800 7400
+F 0 "P?" H 5800 7550 50  0000 C CNN
+F 1 "general" H 5800 7250 50  0000 C CNN
+F 2 "" H 5800 7400 60  0000 C CNN
+F 3 "" H 5800 7400 60  0000 C CNN
+	1    5800 7400
 	1    0    0    -1
 $EndComp
@@
 P 1050 6500
 F 0 "J?" H 1050 6700 50  0000 C CNN
-F 1 "General_Power_Source" H 1050 6300 50  0000 C CNN
+F 1 "general_power_source" H 1050 6300 50  0000 C CNN
 F 2 "" H 1100 6500 50  0001 C CNN
 F 3 "" H 1100 6500 50  0001 C CNN
@@
 	850  6400 650  6400
 Wire Wire Line
-	1250 6500 1950 6500
-Wire Wire Line
-	1950 6600 1850 6600
-Wire Wire Line
-	1850 6600 1850 6650
+	5600 7450 5500 7450
+Wire Wire Line
+	5500 7450 5500 7500
 Wire Wire Line
 	6800 5700 7300 5700
@@
 Text GLabel 850  6600 0    60   Input ~ 0
 VPCIE
+Wire Wire Line
+	1250 6500 1450 6500
+Wire Wire Line
+	5600 7350 5400 7350
+Text GLabel 1450 6500 2    60   Input ~ 0
+genPow
+Text GLabel 5400 7350 0    60   Input ~ 0
+genPow
 $EndSCHEMATC

Commit message: assigned some footprint
Parts:
- removed R? (x3): 4.7k, symbol R
- added R? (x3): 4.7k, Resistors_SMD:R_0603_HandSoldering, symbol R
- C? (x26): footprint (none) -> Capacitors_SMD:C_0603_HandSoldering
- J?: footprint (none) -> Connectors:USB_Mini-B
- R? (x13): footprint (none) -> Resistors_SMD:R_0603_HandSoldering
- Y?: footprint (none) -> Crystals:Crystal_SMD_Abracon_ABM3-2pin_5.0x3.2mm_HandSoldering
Connections:
- net GND: now also R?.1, R?.1, R?.1
- net at U?.1 (PWRCTL3/BATEN3): now also R?.2
- net at U?.3 (PWRCTL2/BATEN2): now also R?.2
- net at U?.4 (PWRCTL1/BATEN1): now also R?.2

Commit message: wow
Parts:
- CON? (x2): footprint (none) -> Zeabus:pcie-x16-conn
- D? (x2): footprint (none) -> LEDs:LED_0603_HandSoldering
- P? (x6): footprint (none) -> Zeabus:XT30
Changed lines of the file:
@@
 F 0 "CON?" H 7650 4250 60  0000 C CNN
 F 1 "peripheral_bridge" H 7900 2100 60  0000 C CNN
-F 2 "" H 7500 4200 60  0001 C CNN
+F 2 "Zeabus:pcie-x16-conn" H 7500 4200 60  0001 C CNN
 F 3 "" H 7500 4200 60  0001 C CNN
 	1    7500 4200
@@
 F 0 "P?" H 4600 7550 50  0000 C CNN
 F 1 "ethernet_switch" H 4600 7250 50  0000 C CNN
-F 2 "" H 4600 7400 60  0000 C CNN
+F 2 "Zeabus:XT30" H 4600 7400 60  0000 C CNN
 F 3 "" H 4600 7400 60  0000 C CNN
 	1    4600 7400
@@
 F 0 "P?" H 2150 7550 50  0000 C CNN
 F 1 "DVL" H 2150 7250 50  0000 C CNN
-F 2 "" H 2150 7400 60  0000 C CNN
+F 2 "Zeabus:XT30" H 2150 7400 60  0000 C CNN
 F 3 "" H 2150 7400 60  0000 C CNN
 	1    2150 7400
@@
 F 0 "P?" H 2950 7550 50  0000 C CNN
 F 1 "computer1" H 2950 7250 50  0000 C CNN
-F 2 "" H 2950 7400 60  0000 C CNN
+F 2 "Zeabus:XT30" H 2950 7400 60  0000 C CNN
 F 3 "" H 2950 7400 60  0000 C CNN
 	1    2950 7400
@@
 F 0 "P?" H 3800 7550 50  0000 C CNN
 F 1 "computer2" H 3800 7250 50  0000 C CNN
-F 2 "" H 3800 7400 60  0000 C CNN
+F 2 "Zeabus:XT30" H 3800 7400 60  0000 C CNN
 F 3 "" H 3800 7400 60  0000 C CNN
 	1    3800 7400
@@
 F 0 "P?" H 1300 7550 50  0000 C CNN
 F 1 "imaging_sonar" H 1300 7250 50  0000 C CNN
-F 2 "" H 1300 7400 60  0000 C CNN
+F 2 "Zeabus:XT30" H 1300 7400 60  0000 C CNN
 F 3 "" H 1300 7400 60  0000 C CNN
 	1    1300 7400
@@
 F 0 "CON?" H 10200 800 60  0000 C CNN
 F 1 "power_distributor" H 10400 700 60  0000 C CNN
-F 2 "" H 10050 650 60  0001 C CNN
+F 2 "Zeabus:pcie-x16-conn" H 10050 650 60  0001 C CNN
 F 3 "" H 10050 650 60  0001 C CNN
 	1    10050 650
@@
 F 0 "D?" H 8200 750 50  0000 C CNN
 F 1 "LED_VPCIe" H 8200 550 50  0000 C CNN
-F 2 "" H 8200 650 50  0001 C CNN
+F 2 "LEDs:LED_0603_HandSoldering" H 8200 650 50  0001 C CNN
 F 3 "" H 8200 650 50  0001 C CNN
 	1    8200 650
@@
 F 0 "D?" H 7150 750 50  0000 C CNN
 F 1 "LED_VBUS" H 7150 550 50  0000 C CNN
-F 2 "" H 7150 650 50  0001 C CNN
+F 2 "LEDs:LED_0603_HandSoldering" H 7150 650 50  0001 C CNN
 F 3 "" H 7150 650 50  0001 C CNN
 	1    7150 650
@@
 F 0 "P?" H 5800 7550 50  0000 C CNN
 F 1 "general" H 5800 7250 50  0000 C CNN
-F 2 "" H 5800 7400 60  0000 C CNN
+F 2 "Zeabus:XT30" H 5800 7400 60  0000 C CNN
 F 3 "" H 5800 7400 60  0000 C CNN
 	1    5800 7400
