File: Circuit/Backplane/noname.kicad_pcb1.kicad_pcb (KiCad board)
At the start: 2 copper layers, 94 x 307.3 mm, 89 parts, among them CON1 peripheral_bridge, CON2 power_distributor, J1 USB_OTG, J2 power_source_mode, J3 general_power_source, J4 pneumatic, J5 pressure_sensor, J6 RS232_DVL, P1 imaging_sonar, P2 DVL, P3 computer1, P4 computer2, P5 ethernet_switch, P6 general, U1 LM1117-3.3, U2 TUSB4041I, U3 TLV73311PDBVT, Y1 24MHz

Commit message: retracking in pcb
Parts:
- moved R11 8.63 mm to (142.3, 231.1), turned to 180 degrees
- moved R5 0.36 mm to (143.7, 246.6)
Routing:
- net +12V: track 447.4 -> 615.3 mm, vias 22 -> 2
- net VPCIE: track 283.1 -> 390.8 mm, vias 2 -> 3
- net Net-(C11-Pad1): track 393.7 -> 446.3 mm, vias 20 -> 11
- net Net-(CON1-PadA13): track 154.6 -> 117.2 mm, vias 0 -> 1
- net VBUS: track 407.0 -> 372.6 mm, vias 18 -> 6
- net +BATT: track 168.7 -> 199.3 mm, vias 10 -> 8
- net Net-(R1-Pad1): track 6.39 -> 28.4 mm
- net Net-(CON1-PadA14): track 153.0 -> 132.8 mm, vias 0 -> 1
- net Net-(CON1-PadA15): track 162.3 -> 142.8 mm
- net Net-(CON1-PadA16): track 159.4 -> 141.1 mm
- net Net-(CON1-PadA18): track 166.6 -> 148.3 mm, vias 2 -> 1
- net Net-(C5-Pad1): track 26.8 -> 44.8 mm
- net Net-(CON1-PadA17): track 169.6 -> 152.4 mm, vias 2 -> 1
- net Net-(CON1-PadA7): track 133.7 -> 121.6 mm, vias 6 -> 3
- net Net-(CON1-PadB15): track 90.9 -> 99.9 mm
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