File: Circuit/Backplane/Backplane.kicad_pcb (KiCad board)
At the start: 2 copper layers, 90.2 x 288.5 mm, 86 parts, among them CON1 peripheral_bridge, CON2 power_distributor, J1 USB_OTG, J2 power_source_mode, J3 general_power_source, J4 pneumatic, J5 pressure_sensor, J6 RS232_DVL, P1 imaging_sonar, P2 DVL, P3 computer1, P4 computer2, P5 ethernet_switch, P6 general, Q1 Q_NPN_BCE, U1 LM1117-3.3, U2 TUSB4041I, U3 TLV73311PDBVT, Y1 24MHz

Commit message: reassigned transistor footprint SOT-323 to SOT-23 for BC817-40 and rounted pcb
Parts:
- Q1: footprint TO_SOT_Packages_SMD:SOT-323_SC-70_Handsoldering -> TO_SOT_Packages_SMD:SOT-23
- R22: value 500 -> 40
Routing:
- net GND: track 38.5 -> 51.9 mm, vias 15 -> 16
Changed lines of the file:
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@@
   (general
     (links 258)
-    (no_connects 68)
+    (no_connects 67)
     (area 76.124999 -26.745001 166.445001 261.949001)
     (thickness 1.6)
     (drawings 32)
-    (tracks 1492)
+    (tracks 1505)
     (zones 0)
     (modules 86)
@@
   )
   (setup
-    (last_trace_width 0.381)
+    (last_trace_width 0.254)
     (user_trace_width 0.381)
     (user_trace_width 0.762)
@@
     )
   )
-  (module TO_SOT_Packages_SMD:SOT-323_SC-70_Handsoldering (layer F.Cu)
-    (at 128.464 -21.53 180)
-    (descr "SOT-323, SC-70 Handsoldering")
-    (tags "SOT-323 SC-70 Handsoldering")
-    (attr smd)
-    (fp_text reference Q1 (at 0 -2 180) (layer F.SilkS)
-      (effects (font (size 1 1) (thickness 0.15)))
-    )
-    (fp_text value Q_NPN_BCE (at 0 2.05 180) (layer F.Fab)
-      (effects (font (size 1 1) (thickness 0.15)))
-    )
-    (fp_text user %R (at 0 0 270) (layer F.Fab)
-      (effects (font (size 0.5 0.5) (thickness 0.075)))
-    )
-    (fp_line (start 0.735 0.5) (end 0.735 1.16) (layer F.SilkS) (width 0.12))
-    (fp_line (start 0.735 -1.17) (end 0.735 -0.5) (layer F.SilkS) (width 0.12))
-    (fp_line (start 2.4 1.3) (end -2.4 1.3) (layer F.CrtYd) (width 0.05))
-    (fp_line (start 2.4 -1.3) (end 2.4 1.3) (layer F.CrtYd) (width 0.05))
-    (fp_line (start -2.4 -1.3) (end 2.4 -1.3) (layer F.CrtYd) (width 0.05))
-    (fp_line (start -2.4 1.3) (end -2.4 -1.3) (layer F.CrtYd) (width 0.05))
-    (fp_line (start 0.735 -1.16) (end -2 -1.16) (layer F.SilkS) (width 0.12))
-    (fp_line (start -0.675 1.16) (end 0.735 1.16) (layer F.SilkS) (width 0.12))
-    (fp_line (start 0.675 -1.1) (end -0.175 -1.1) (layer F.Fab) (width 0.1))
-    (fp_line (start -0.675 -0.6) (end -0.675 1.1) (layer F.Fab) (width 0.1))
-    (fp_line (start 0.675 -1.1) (end 0.675 1.1) (layer F.Fab) (width 0.1))
-    (fp_line (start 0.675 1.1) (end -0.675 1.1) (layer F.Fab) (width 0.1))
-    (fp_line (start -0.175 -1.1) (end -0.675 -0.6) (layer F.Fab) (width 0.1))
-    (pad 1 smd rect (at -1.33 -0.65 90) (size 0.45 1.5) (layers F.Cu F.Paste F.Mask)
-      (net 144 "Net-(Q1-Pad1)"))
-    (pad 2 smd rect (at -1.33 0.65 90) (size 0.45 1.5) (layers F.Cu F.Paste F.Mask)
-      (net 145 "Net-(Q1-Pad2)"))
-    (pad 3 smd rect (at 1.33 0 90) (size 0.45 1.5) (layers F.Cu F.Paste F.Mask)
-      (net 103 GND))
-    (model ${KISYS3DMOD}/TO_SOT_Packages_SMD.3dshapes/SOT-323_SC-70.wrl
-      (at (xyz 0 0 0))
-      (scale (xyz 1 1 1))
-      (rotate (xyz 0 0 0))
-    )
-  )
   (module Resistors_SMD:R_0603_HandSoldering (layer F.Cu)
     (at 132.758 -24.638 180)
@@
       (effects (font (size 1 1) (thickness 0.15)))
     )
-    (fp_text value 500 (at 0 1.55) (layer F.Fab)
+    (fp_text value 40 (at 0 1.55) (layer F.Fab)
       (effects (font (size 1 1) (thickness 0.15)))
     )
@@
     (pad 1 np_thru_hole circle (at 0 0) (size 3 3) (drill 3) (layers *.Cu *.Mask))
   )
+  (module TO_SOT_Packages_SMD:SOT-23 (layer F.Cu)
+    (at 128.464 -21.53 180)
+    (descr "SOT-23, Standard")
+    (tags SOT-23)
+    (attr smd)
+    (fp_text reference Q1 (at 0 -2.5 180) (layer F.SilkS)
+      (effects (font (size 1 1) (thickness 0.15)))
+    )
+    (fp_text value Q_NPN_BCE (at 0 2.5 180) (layer F.Fab)
+      (effects (font (size 1 1) (thickness 0.15)))
+    )
+    (fp_text user %R (at 0 0 270) (layer F.Fab)
+      (effects (font (size 0.5 0.5) (thickness 0.075)))
+    )
+    (fp_line (start -0.7 -0.95) (end -0.7 1.5) (layer F.Fab) (width 0.1))
+    (fp_line (start -0.15 -1.52) (end 0.7 -1.52) (layer F.Fab) (width 0.1))
+    (fp_line (start -0.7 -0.95) (end -0.15 -1.52) (layer F.Fab) (width 0.1))
+    (fp_line (start 0.7 -1.52) (end 0.7 1.52) (layer F.Fab) (width 0.1))
+    (fp_line (start -0.7 1.52) (end 0.7 1.52) (layer F.Fab) (width 0.1))
+    (fp_line (start 0.76 1.58) (end 0.76 0.65) (layer F.SilkS) (width 0.12))
+    (fp_line (start 0.76 -1.58) (end 0.76 -0.65) (layer F.SilkS) (width 0.12))
+    (fp_line (start -1.7 -1.75) (end 1.7 -1.75) (layer F.CrtYd) (width 0.05))
+    (fp_line (start 1.7 -1.75) (end 1.7 1.75) (layer F.CrtYd) (width 0.05))
+    (fp_line (start 1.7 1.75) (end -1.7 1.75) (layer F.CrtYd) (width 0.05))
+    (fp_line (start -1.7 1.75) (end -1.7 -1.75) (layer F.CrtYd) (width 0.05))
+    (fp_line (start 0.76 -1.58) (end -1.4 -1.58) (layer F.SilkS) (width 0.12))
+    (fp_line (start 0.76 1.58) (end -0.7 1.58) (layer F.SilkS) (width 0.12))
+    (pad 1 smd rect (at -1 -0.95 180) (size 0.9 0.8) (layers F.Cu F.Paste F.Mask)
+      (net 144 "Net-(Q1-Pad1)"))
+    (pad 2 smd rect (at -1 0.95 180) (size 0.9 0.8) (layers F.Cu F.Paste F.Mask)
+      (net 145 "Net-(Q1-Pad2)"))
+    (pad 3 smd rect (at 1 0 180) (size 0.9 0.8) (layers F.Cu F.Paste F.Mask)
+      (net 103 GND))
+    (model ${KISYS3DMOD}/TO_SOT_Packages_SMD.3dshapes/SOT-23.wrl
+      (at (xyz 0 0 0))
+      (scale (xyz 1 1 1))
+      (rotate (xyz 0 0 0))
+    )
+  )
   (dimension 139.7 (width 0.3) (layer Eco1.User)
     (gr_text "139.700 mm" (at 124.126 62.268443 270) (layer Eco1.User)
@@
   (segment (start 111.252 226.06) (end 112.656 227.464) (width 0.254) (layer F.Cu) (net 101))
   (segment (start 112.656 227.464) (end 115.892 227.464) (width 0.254) (layer F.Cu) (net 101))
+  (segment (start 162.016 253.532) (end 162.016 253.782) (width 0.254) (layer F.Cu) (net 103))
+  (segment (start 162.016 253.782) (end 164.012 255.778) (width 0.254) (layer F.Cu) (net 103))
+  (segment (start 164.012 255.778) (end 164.084 255.778) (width 0.254) (layer F.Cu) (net 103))
+  (via (at 164.084 255.778) (size 1.10236) (drill 0.6096) (layers F.Cu B.Cu) (net 103))
+  (segment (start 162.016 259.032) (end 158.798 259.032) (width 0.254) (layer F.Cu) (net 103))
+  (segment (start 158.798 259.032) (end 158.75 259.08) (width 0.254) (layer F.Cu) (net 103))
+  (via (at 158.75 259.08) (size 1.10236) (drill 0.6096) (layers F.Cu B.Cu) (net 103))
+  (segment (start 162.016 253.532) (end 162.016 255.036) (width 0.254) (layer F.Cu) (net 103))
+  (segment (start 162.758 255.778) (end 163.068 255.778) (width 0.254) (layer F.Cu) (net 103))
+  (segment (start 151.08 244.87) (end 152.668 244.87) (width 0.254) (layer F.Cu) (net 103))
+  (via (at 153.67 245.872) (size 1.10236) (drill 0.6096) (layers F.Cu B.Cu) (net 103))
+  (segment (start 152.668 244.87) (end 153.67 245.872) (width 0.254) (layer F.Cu) (net 103))
+  (segment (start 125.984 -20.754) (end 125.984 -20.32) (width 0.254) (layer F.Cu) (net 103))
+  (via (at 125.984 -20.32) (size 1.10236) (drill 0.6096) (layers F.Cu B.Cu) (net 103))
+  (segment (start 127.464 -21.53) (end 126.76 -21.53) (width 0.254) (layer F.Cu) (net 103))
+  (segment (start 126.76 -21.53) (end 125.984 -20.754) (width 0.254) (layer F.Cu) (net 103))
   (segment (start 152.955 245.364) (end 154.178 245.364) (width 0.381) (layer F.Cu) (net 103))
-  (via (at 154.178 245.364) (size 1.10236) (drill 0.6096) (layers F.Cu B.Cu) (net 103))
   (segment (start 151.08 244.87) (end 152.461 244.87) (width 0.381) (layer F.Cu) (net 103))
   (segment (start 152.461 244.87) (end 152.955 245.364) (width 0.381) (layer F.Cu) (net 103))
@@
   (segment (start 162.016 253.532) (end 162.016 254.218) (width 0.381) (layer F.Cu) (net 103))
   (segment (start 162.016 254.218) (end 163.322 255.524) (width 0.381) (layer F.Cu) (net 103))
-  (via (at 163.322 255.524) (size 1.10236) (drill 0.6096) (layers F.Cu B.Cu) (net 103))
   (segment (start 135.89 243.2) (end 135.89 245.618) (width 0.381) (layer F.Cu) (net 103))
   (segment (start 135.89 245.618) (end 136.652 246.38) (width 0.381) (layer F.Cu) (net 103))
@@
   (segment (start 127.134 -21.53) (end 127.134 -19.17) (width 0.381) (layer F.Cu) (net 103))
   (segment (start 127.134 -19.17) (end 127.254 -19.05) (width 0.381) (layer F.Cu) (net 103))
-  (via (at 127.254 -19.05) (size 1.10236) (drill 0.6096) (layers F.Cu B.Cu) (net 103))
   (segment (start 164.338 -25.568) (end 163.634 -25.568) (width 0.254) (layer F.Cu) (net 136))
   (segment (start 163.634 -25.568) (end 163.441381 -25.375381) (width 0.254) (layer F.Cu) (net 136))
@@
     (polygon
       (pts
-        (xy 166.37 -26.67) (xy 124.46 -26.67) (xy 124.46 -8.89) (xy 166.37 -8.89)
+        (xy 166.37 -26.67) (xy 124.46 -26.67) (xy 124.46 -13.97) (xy 166.37 -13.97)
       )
     )
@@
     (polygon
       (pts
-        (xy 166.37 -26.67) (xy 76.2 -26.67) (xy 76.2 261.874) (xy 166.37 261.874)
+        (xy 166.37 -26.67) (xy 166.37 261.874) (xy 76.2 261.874) (xy 76.2 -26.67)
       )
     )
@@
     (polygon
       (pts
-        (xy 91.44 214.63) (xy 166.37 214.63) (xy 166.37 261.874) (xy 91.44 261.874)
+        (xy 166.37 214.63) (xy 91.44 214.63) (xy 91.44 261.874) (xy 166.37 261.874)
       )
     )
