File: Circuit/Backplane/Backplane.kicad_pcb (KiCad board)
At the start: 2 copper layers, 90.2 x 288.5 mm, 86 parts, among them CON1 peripheral_bridge, CON2 power_distributor, J1 USB_OTG, J2 power_source_mode, J3 general_power_source, J4 pneumatic, J5 pressure_sensor, J6 RS232_DVL, P1 imaging_sonar, P2 DVL, P3 computer1, P4 computer2, P5 ethernet_switch, P6 general, Q1 Q_NPN_BCE, U1 LM1117-3.3, U2 TUSB4041I, U3 TLV73311PDBVT, Y1 24MHz

Commit message: Rb 40 to 150
Parts:
- R22: value 40 -> 150
Changed lines of the file:
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@@
   (general
     (links 258)
-    (no_connects 67)
+    (no_connects 3)
     (area 76.124999 -26.745001 166.445001 261.949001)
     (thickness 1.6)
@@
       (effects (font (size 1 1) (thickness 0.15)))
     )
-    (fp_text value 40 (at 0 1.55) (layer F.Fab)
+    (fp_text value 150 (at 0 1.55) (layer F.Fab)
       (effects (font (size 1 1) (thickness 0.15)))
     )
@@
     (arrow2b (pts (xy 91.44 119.634) (xy 90.853579 118.507496)))
   )
+  (segment (start 162.758 255.778) (end 163.068 255.778) (width 0.254) (layer F.Cu) (net 0))
   (segment (start 156.579408 -14.478) (end 153.416 -14.478) (width 0.254) (layer F.Cu) (net 1))
   (segment (start 153.416 -14.478) (end 151.638 -16.256) (width 0.254) (layer F.Cu) (net 1))
@@
   (via (at 158.75 259.08) (size 1.10236) (drill 0.6096) (layers F.Cu B.Cu) (net 103))
   (segment (start 162.016 253.532) (end 162.016 255.036) (width 0.254) (layer F.Cu) (net 103))
-  (segment (start 162.758 255.778) (end 163.068 255.778) (width 0.254) (layer F.Cu) (net 103))
   (segment (start 151.08 244.87) (end 152.668 244.87) (width 0.254) (layer F.Cu) (net 103))
   (via (at 153.67 245.872) (size 1.10236) (drill 0.6096) (layers F.Cu B.Cu) (net 103))

Commit message: retracking
Parts:
- Q1: value Q_NPN_BCE -> BC817-40
Connections:
- D8 pad 1: Net-(D8-Pad1) -> +5V
- D8 pad 2: +5V -> Net-(D8-Pad2)
- Q1 pad 2: Net-(Q1-Pad2) -> GND
- Q1 pad 3: GND -> Net-(Q1-Pad3)
- R21 pad 1: Net-(Q1-Pad2) -> Net-(D8-Pad2)
- R21 pad 2: Net-(D8-Pad1) -> Net-(Q1-Pad3)
Routing:
- net +5V: track 516.8 -> 544.8 mm, vias 8 -> 9
- net Net-(D8-Pad1): track 8.97 -> 0.00 mm
- net Net-(Q1-Pad3): track 0.00 -> 7.37 mm
- net Net-(D8-Pad2): track 0.00 -> 6.63 mm
- net Net-(Q1-Pad2): track 5.49 -> 0.00 mm
- net GND: track 51.6 -> 46.9 mm, vias 16 -> 15
- removed copper zone on B.Cu, net GND
- removed copper zone on F.Cu, net GND
Changed lines of the file:
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@@
   (general
     (links 258)
-    (no_connects 3)
+    (no_connects 69)
     (area 76.124999 -26.745001 166.445001 261.949001)
     (thickness 1.6)
     (drawings 32)
-    (tracks 1505)
+    (tracks 1510)
     (zones 0)
     (modules 86)
@@
   (net 141 +1V1)
   (net 142 "Net-(U2-Pad47)")
-  (net 143 "Net-(D8-Pad1)")
-  (net 144 "Net-(Q1-Pad1)")
-  (net 145 "Net-(Q1-Pad2)")
+  (net 143 "Net-(Q1-Pad1)")
+  (net 144 "Net-(D8-Pad2)")
+  (net 145 "Net-(Q1-Pad3)")
   (net_class Default "This is the default net class."
     (clearance 0.2032)
@@
     (add_net "Net-(D6-Pad1)")
     (add_net "Net-(D7-Pad1)")
-    (add_net "Net-(D8-Pad1)")
+    (add_net "Net-(D8-Pad2)")
     (add_net "Net-(J1-Pad2)")
     (add_net "Net-(J1-Pad3)")
     (add_net "Net-(J1-Pad4)")
     (add_net "Net-(Q1-Pad1)")
-    (add_net "Net-(Q1-Pad2)")
+    (add_net "Net-(Q1-Pad3)")
     (add_net "Net-(R1-Pad1)")
     (add_net "Net-(R10-Pad1)")
@@
     (fp_line (start -0.8 -0.4) (end -0.8 0.4) (layer F.Fab) (width 0.1))
     (pad 1 smd rect (at -1.1 0 270) (size 1.2 0.9) (layers F.Cu F.Paste F.Mask)
-      (net 143 "Net-(D8-Pad1)"))
-    (pad 2 smd rect (at 1.1 0 270) (size 1.2 0.9) (layers F.Cu F.Paste F.Mask)
       (net 3 +5V))
+    (pad 2 smd rect (at 1.1 0 270) (size 1.2 0.9) (layers F.Cu F.Paste F.Mask)
+      (net 144 "Net-(D8-Pad2)"))
     (model ${KISYS3DMOD}/LEDs.3dshapes/LED_0603.wrl
       (at (xyz 0 0 0))
@@
     (fp_line (start 1.95 0.7) (end -1.96 0.7) (layer F.CrtYd) (width 0.05))
     (pad 1 smd rect (at -1.1 0 180) (size 1.2 0.9) (layers F.Cu F.Paste F.Mask)
-      (net 145 "Net-(Q1-Pad2)"))
+      (net 144 "Net-(D8-Pad2)"))
     (pad 2 smd rect (at 1.1 0 180) (size 1.2 0.9) (layers F.Cu F.Paste F.Mask)
-      (net 143 "Net-(D8-Pad1)"))
+      (net 145 "Net-(Q1-Pad3)"))
     (model ${KISYS3DMOD}/Resistors_SMD.3dshapes/R_0603.wrl
       (at (xyz 0 0 0))
@@
     (fp_line (start 1.95 0.7) (end -1.96 0.7) (layer F.CrtYd) (width 0.05))
     (pad 1 smd rect (at -1.1 0) (size 1.2 0.9) (layers F.Cu F.Paste F.Mask)
-      (net 144 "Net-(Q1-Pad1)"))
+      (net 143 "Net-(Q1-Pad1)"))
     (pad 2 smd rect (at 1.1 0) (size 1.2 0.9) (layers F.Cu F.Paste F.Mask)
       (net 141 +1V1))
@@
       (effects (font (size 1 1) (thickness 0.15)))
     )
-    (fp_text value Q_NPN_BCE (at 0 2.5 180) (layer F.Fab)
+    (fp_text value BC817-40 (at 0 2.5 180) (layer F.Fab)
       (effects (font (size 1 1) (thickness 0.15)))
     )
@@
     (fp_line (start 0.76 1.58) (end -0.7 1.58) (layer F.SilkS) (width 0.12))
     (pad 1 smd rect (at -1 -0.95 180) (size 0.9 0.8) (layers F.Cu F.Paste F.Mask)
-      (net 144 "Net-(Q1-Pad1)"))
+      (net 143 "Net-(Q1-Pad1)"))
     (pad 2 smd rect (at -1 0.95 180) (size 0.9 0.8) (layers F.Cu F.Paste F.Mask)
-      (net 145 "Net-(Q1-Pad2)"))
-    (pad 3 smd rect (at 1 0 180) (size 0.9 0.8) (layers F.Cu F.Paste F.Mask)
       (net 103 GND))
+    (pad 3 smd rect (at 1 0 180) (size 0.9 0.8) (layers F.Cu F.Paste F.Mask)
+      (net 145 "Net-(Q1-Pad3)"))
     (model ${KISYS3DMOD}/TO_SOT_Packages_SMD.3dshapes/SOT-23.wrl
       (at (xyz 0 0 0))
@@
   (segment (start 155.966 253.432) (end 155.966 252.028) (width 0.254) (layer F.Cu) (net 2))
   (segment (start 155.966 252.028) (end 155.398 251.46) (width 0.254) (layer F.Cu) (net 2))
+  (segment (start 140.655594 -21.322964) (end 153.429036 -21.322964) (width 0.254) (layer B.Cu) (net 3))
+  (segment (start 153.429036 -21.322964) (end 155.448 -19.304) (width 0.254) (layer B.Cu) (net 3))
+  (segment (start 140.462 -25.002) (end 140.462 -21.516558) (width 0.254) (layer F.Cu) (net 3))
+  (segment (start 140.462 -21.516558) (end 140.655594 -21.322964) (width 0.254) (layer F.Cu) (net 3))
+  (via (at 140.655594 -21.322964) (size 1.10236) (drill 0.6096) (layers F.Cu B.Cu) (net 3))
+  (segment (start 139.446 -25.314) (end 140.15 -25.314) (width 0.254) (layer F.Cu) (net 3))
+  (segment (start 140.15 -25.314) (end 140.462 -25.002) (width 0.254) (layer F.Cu) (net 3))
   (segment (start 137.16 98.298) (end 137.16 93.726) (width 0.254) (layer F.Cu) (net 3))
   (segment (start 137.16 93.726) (end 137.16 91.948) (width 0.254) (layer F.Cu) (net 3))
@@
   (segment (start 153.466733 233.670251) (end 154.500733 233.670251) (width 0.254) (layer F.Cu) (net 3))
   (segment (start 156.260733 235.430251) (end 156.260733 235.758251) (width 0.254) (layer F.Cu) (net 3))
+  (segment (start 132.224 -25.908) (end 138.148 -25.908) (width 0.254) (layer F.Cu) (net 3))
+  (segment (start 138.148 -25.908) (end 138.742 -25.314) (width 0.254) (layer F.Cu) (net 3))
+  (segment (start 138.742 -25.314) (end 139.446 -25.314) (width 0.254) (layer F.Cu) (net 3))
   (segment (start 122.428 256.032) (end 122.428 258.797) (width 0.254) (layer F.Cu) (net 4))
   (segment (start 122.428 258.797) (end 123.473 259.842) (width 0.254) (layer F.Cu) (net 4))
@@
   (via (at 153.67 245.872) (size 1.10236) (drill 0.6096) (layers F.Cu B.Cu) (net 103))
   (segment (start 152.668 244.87) (end 153.67 245.872) (width 0.254) (layer F.Cu) (net 103))
-  (segment (start 125.984 -20.754) (end 125.984 -20.32) (width 0.254) (layer F.Cu) (net 103))
-  (via (at 125.984 -20.32) (size 1.10236) (drill 0.6096) (layers F.Cu B.Cu) (net 103))
-  (segment (start 127.464 -21.53) (end 126.76 -21.53) (width 0.254) (layer F.Cu) (net 103))
-  (segment (start 126.76 -21.53) (end 125.984 -20.754) (width 0.254) (layer F.Cu) (net 103))
   (segment (start 152.955 245.364) (end 154.178 245.364) (width 0.381) (layer F.Cu) (net 103))
   (segment (start 151.08 244.87) (end 152.461 244.87) (width 0.381) (layer F.Cu) (net 103))
@@
   (segment (start 135.89 245.618) (end 136.652 246.38) (width 0.381) (layer F.Cu) (net 103))
   (via (at 136.652 246.38) (size 1.10236) (drill 0.6096) (layers F.Cu B.Cu) (net 103))
-  (segment (start 127.134 -21.53) (end 127.134 -19.17) (width 0.381) (layer F.Cu) (net 103))
-  (segment (start 127.134 -19.17) (end 127.254 -19.05) (width 0.381) (layer F.Cu) (net 103))
   (segment (start 164.338 -25.568) (end 163.634 -25.568) (width 0.254) (layer F.Cu) (net 136))
   (segment (start 163.634 -25.568) (end 163.441381 -25.375381) (width 0.254) (layer F.Cu) (net 136))
@@
   (segment (start 146.203733 233.350251) (end 148.132733 235.279251) (width 0.254) (layer F.Cu) (net 141))
   (segment (start 148.132733 235.279251) (end 148.132733 235.504251) (width 0.254) (layer F.Cu) (net 141))
-  (segment (start 132.224 -25.908) (end 138.148 -25.908) (width 0.254) (layer F.Cu) (net 143))
-  (segment (start 138.148 -25.908) (end 138.742 -25.314) (width 0.254) (layer F.Cu) (net 143))
-  (segment (start 138.742 -25.314) (end 139.446 -25.314) (width 0.254) (layer F.Cu) (net 143))
-  (segment (start 131.658 -24.638) (end 131.658 -25.342) (width 0.254) (layer F.Cu) (net 143))
-  (segment (start 131.658 -25.342) (end 132.224 -25.908) (width 0.254) (layer F.Cu) (net 143))
-  (segment (start 129.794 -20.88) (end 130.798 -20.88) (width 0.254) (layer F.Cu) (net 144))
-  (segment (start 130.798 -20.88) (end 131.658 -20.02) (width 0.254) (layer F.Cu) (net 144))
-  (segment (start 131.658 -20.02) (end 131.658 -19.246) (width 0.254) (layer F.Cu) (net 144))
-  (segment (start 131.658 -19.246) (end 131.658 -18.542) (width 0.254) (layer F.Cu) (net 144))
-  (segment (start 129.794 -22.18) (end 132.104 -22.18) (width 0.254) (layer F.Cu) (net 145))
-  (segment (start 132.104 -22.18) (end 133.858 -23.934) (width 0.254) (layer F.Cu) (net 145))
-  (segment (start 133.858 -23.934) (end 133.858 -24.638) (width 0.254) (layer F.Cu) (net 145))
-  (zone (net 103) (net_name GND) (layer F.Cu) (hatch edge 0.508)
-    (connect_pads yes (clearance 0.1524))
-    (min_thickness 0.254)
-    (fill yes (arc_segments 16) (thermal_gap 0.508) (thermal_bridge_width 0.508))
-    (polygon
-      (pts
-        (xy 166.37 -26.67) (xy 124.46 -26.67) (xy 124.46 -13.97) (xy 166.37 -13.97)
-      )
-    )
-  )
-  (zone (net 103) (net_name GND) (layer B.Cu) (hatch edge 0.508)
-    (connect_pads yes (clearance 0.1524))
-    (min_thickness 0.254)
-    (fill yes (arc_segments 16) (thermal_gap 0.508) (thermal_bridge_width 0.508))
-    (polygon
-      (pts
-        (xy 166.37 -26.67) (xy 166.37 261.874) (xy 76.2 261.874) (xy 76.2 -26.67)
-      )
-    )
-  )
-  (zone (net 103) (net_name GND) (layer F.Cu) (hatch edge 0.508)
-    (connect_pads yes (clearance 0.1524))
-    (min_thickness 0.254)
-    (fill yes (arc_segments 16) (thermal_gap 0.508) (thermal_bridge_width 0.508))
-    (polygon
-      (pts
-        (xy 166.37 214.63) (xy 91.44 214.63) (xy 91.44 261.874) (xy 166.37 261.874)
-      )
-    )
-  )
+  (segment (start 129.794 -20.88) (end 130.798 -20.88) (width 0.254) (layer F.Cu) (net 143))
+  (segment (start 130.798 -20.88) (end 131.658 -20.02) (width 0.254) (layer F.Cu) (net 143))
+  (segment (start 131.658 -20.02) (end 131.658 -19.246) (width 0.254) (layer F.Cu) (net 143))
+  (segment (start 131.658 -19.246) (end 131.658 -18.542) (width 0.254) (layer F.Cu) (net 143))
+  (segment (start 133.858 -24.638) (end 133.858 -23.934) (width 0.254) (layer F.Cu) (net 144))
+  (segment (start 133.858 -23.934) (end 134.678 -23.114) (width 0.254) (layer F.Cu) (net 144))
+  (segment (start 134.678 -23.114) (end 138.742 -23.114) (width 0.254) (layer F.Cu) (net 144))
+  (segment (start 138.742 -23.114) (end 139.446 -23.114) (width 0.254) (layer F.Cu) (net 144))
+  (segment (start 127.464 -21.53) (end 127.464 -22.184) (width 0.254) (layer F.Cu) (net 145))
+  (segment (start 127.464 -22.184) (end 129.918 -24.638) (width 0.254) (layer F.Cu) (net 145))
+  (segment (start 129.918 -24.638) (end 131.658 -24.638) (width 0.254) (layer F.Cu) (net 145))
+  (segment (start 131.658 -24.638) (end 131.658 -25.342) (width 0.254) (layer F.Cu) (net 145))
+  (segment (start 131.658 -25.342) (end 132.224 -25.908) (width 0.254) (layer F.Cu) (net 145))
 )

Commit message: TUSB
Parts:
- moved C5 57.2 mm to (105.1, 205.5), turned to 0 degrees
- moved C7 54.7 mm to (110.7, 205.5), turned to 180 degrees
- moved R10 50.4 mm to (99.8, 211.8), turned to 90 degrees
- moved Y1 48.1 mm to (108.2, 209.3), turned to 0 degrees
- moved C6 48.0 mm to (102.1, 211.8), turned to 90 degrees
- moved R9 42.4 mm to (118.6, 212.0), turned to 90 degrees
- moved C8 41.7 mm to (130.8, 215.2), turned to 90 degrees
- moved R7 41.2 mm to (108.3, 212.9), turned to 180 degrees
- moved C11 37.6 mm to (99.2, 241.0), turned to 180 degrees
- moved R13 37.1 mm to (138.0, 242.1), turned to 180 degrees
- moved R8 36.8 mm to (127.2, 250.5), turned to 270 degrees
- moved C21 36.4 mm to (122.1, 216.4), turned to 0 degrees
- moved C20 35.9 mm to (99.4, 238.5), turned to 180 degrees
- moved C9 35.7 mm to (138.1, 239.5), turned to 0 degrees
- moved C18 35.4 mm to (99.3, 233.7), turned to 180 degrees
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Routing:
- net +5V: track 544.8 -> 15.8 mm, vias 9 -> 0
- net +12V: track 429.2 -> 0.00 mm, vias 16 -> 0
- net +3V3: track 399.1 -> 45.1 mm, vias 14 -> 0
- net VPCIE: track 303.1 -> 0.00 mm, vias 10 -> 0
- net VBUS: track 320.8 -> 25.5 mm, vias 2 -> 0
- net +1V1: track 297.6 -> 7.75 mm, vias 10 -> 0
- net +BATT: track 246.4 -> 0.00 mm, vias 8 -> 0
- net GNDA: track 228.8 -> 0.00 mm, vias 11 -> 0
- net Net-(CON1-PadA7): track 178.1 -> 0.00 mm, vias 2 -> 0
- net Net-(CON1-PadA6): track 170.9 -> 0.00 mm, vias 2 -> 0
- net Net-(CON1-PadA4): track 166.8 -> 0.00 mm, vias 2 -> 0
- net Net-(CON1-PadB6): track 153.6 -> 0.00 mm
- net genPow: track 147.5 -> 0.00 mm, vias 4 -> 0
- net Net-(CON1-PadA13): track 112.6 -> 0.00 mm
- net Net-(CON1-PadA15): track 111.2 -> 0.00 mm
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
Commit message: extend power wire
Routing:
- net +12V: track 0.00 -> 444.6 mm, vias 0 -> 7
- net VBUS: track 25.5 -> 415.4 mm, vias 0 -> 8
- net +5V: track 15.8 -> 398.4 mm, vias 0 -> 18
- net +3V3: track 45.1 -> 334.1 mm, vias 0 -> 12
- net +1V1: track 7.75 -> 286.8 mm, vias 0 -> 10
- net VPCIE: track 0.00 -> 224.6 mm, vias 0 -> 10
- net +BATT: track 0.00 -> 220.9 mm, vias 0 -> 6
- net Net-(CON1-PadA7): track 0.00 -> 166.9 mm, vias 0 -> 6
- net Net-(CON1-PadA6): track 0.00 -> 166.0 mm, vias 0 -> 6
- net Net-(CON1-PadA4): track 0.00 -> 157.1 mm, vias 0 -> 6
- net genPow: track 0.00 -> 155.9 mm, vias 0 -> 4
- net Net-(CON1-PadB6): track 0.00 -> 136.2 mm, vias 0 -> 4
- net Net-(CON1-PadA13): track 0.00 -> 119.7 mm
- net Net-(CON1-PadA15): track 0.00 -> 118.5 mm
- net Net-(CON1-PadA17): track 0.00 -> 116.5 mm
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
Commit message: AddGround
Routing:
- net GNDA: track 90.8 -> 190.9 mm, vias 3 -> 7
- net GND: track 0.00 -> 26.6 mm, vias 0 -> 8
- added copper zone on B.Cu, net GND
- added copper zone on F.Cu, net GND
Changed lines of the file:
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@@
     (thickness 1.6)
     (drawings 32)
-    (tracks 1551)
+    (tracks 1596)
     (zones 0)
     (modules 86)
@@
   )
   (setup
-    (last_trace_width 0.3048)
+    (last_trace_width 0.254)
     (user_trace_width 0.2794)
     (user_trace_width 0.3048)
@@
   (segment (start 149.377529 67.0052) (end 146.05 70.332729) (width 0.762) (layer F.Cu) (net 48))
   (segment (start 160.782 67.0052) (end 158.267529 67.0052) (width 0.762) (layer F.Cu) (net 48))
+  (segment (start 142.24 36.576) (end 142.24 -0.762) (width 0.254) (layer F.Cu) (net 54))
+  (segment (start 142.24 -0.762) (end 140.716 -2.286) (width 0.254) (layer F.Cu) (net 54))
+  (segment (start 142.748 -15.996) (end 142.748 -16.85) (width 0.254) (layer F.Cu) (net 54))
+  (segment (start 140.716 -2.286) (end 140.716 -9.144) (width 0.254) (layer F.Cu) (net 54))
+  (segment (start 140.716 -9.144) (end 142.748 -11.176) (width 0.254) (layer F.Cu) (net 54))
+  (segment (start 142.748 -11.176) (end 142.748 -15.996) (width 0.254) (layer F.Cu) (net 54))
+  (segment (start 142.24 43.434) (end 142.24 36.576) (width 0.254) (layer B.Cu) (net 54))
+  (via (at 142.24 36.576) (size 1.10236) (drill 0.6096) (layers F.Cu B.Cu) (net 54))
+  (segment (start 142.24 72.136) (end 142.24 43.434) (width 0.254) (layer F.Cu) (net 54))
+  (via (at 142.24 43.434) (size 1.10236) (drill 0.6096) (layers F.Cu B.Cu) (net 54))
+  (segment (start 147.828 72.136) (end 142.24 72.136) (width 0.254) (layer B.Cu) (net 54))
+  (via (at 142.24 72.136) (size 1.10236) (drill 0.6096) (layers F.Cu B.Cu) (net 54))
+  (segment (start 151.892 72.136) (end 147.828 72.136) (width 0.254) (layer F.Cu) (net 54))
+  (via (at 147.828 72.136) (size 1.10236) (drill 0.6096) (layers F.Cu B.Cu) (net 54))
   (segment (start 103.886 108.966) (end 95.20347 108.966) (width 0.381) (layer B.Cu) (net 54))
   (segment (start 95.20347 108.966) (end 95.13997 108.9025) (width 0.381) (layer B.Cu) (net 54))
@@
   (segment (start 123.392 238.864) (end 123.392 248.88191) (width 0.254) (layer F.Cu) (net 101))
   (segment (start 123.392 248.88191) (end 123.881618 249.371528) (width 0.254) (layer F.Cu) (net 101))
+  (segment (start 129.464 -22.48) (end 131.19 -22.48) (width 0.254) (layer F.Cu) (net 103))
+  (segment (start 131.19 -22.48) (end 131.318 -22.352) (width 0.254) (layer F.Cu) (net 103))
+  (via (at 131.318 -22.352) (size 1.10236) (drill 0.6096) (layers F.Cu B.Cu) (net 103))
+  (segment (start 146.812 -16.85) (end 147.516 -16.85) (width 0.254) (layer F.Cu) (net 103))
+  (segment (start 147.516 -16.85) (end 148.624 -17.958) (width 0.254) (layer F.Cu) (net 103))
+  (segment (start 148.624 -17.958) (end 149.41 -17.958) (width 0.254) (layer F.Cu) (net 103))
+  (segment (start 149.41 -17.958) (end 150.114 -17.254) (width 0.254) (layer F.Cu) (net 103))
+  (segment (start 150.114 -17.254) (end 150.114 -17.104) (width 0.254) (layer F.Cu) (net 103))
+  (segment (start 146.492 96.52) (end 146.492 97.978) (width 0.254) (layer F.Cu) (net 103))
+  (segment (start 146.492 97.978) (end 147.32 98.806) (width 0.254) (layer F.Cu) (net 103))
+  (via (at 147.32 98.806) (size 1.10236) (drill 0.6096) (layers F.Cu B.Cu) (net 103))
+  (segment (start 83.058 108.204) (end 82.833 108.204) (width 0.254) (layer F.Cu) (net 103))
+  (segment (start 82.833 108.204) (end 80.801 110.236) (width 0.254) (layer F.Cu) (net 103))
+  (segment (start 80.801 110.236) (end 80.772 110.236) (width 0.254) (layer F.Cu) (net 103))
+  (via (at 80.772 110.236) (size 1.10236) (drill 0.6096) (layers F.Cu B.Cu) (net 103))
+  (segment (start 123.058 216.408) (end 123.058 217.038) (width 0.254) (layer F.Cu) (net 103))
+  (segment (start 123.058 217.038) (end 124.206 218.186) (width 0.254) (layer F.Cu) (net 103))
+  (via (at 124.206 218.186) (size 1.10236) (drill 0.6096) (layers F.Cu B.Cu) (net 103))
+  (segment (start 98.364 233.68) (end 98.364 234.63) (width 0.254) (layer F.Cu) (net 103))
+  (segment (start 98.364 234.63) (end 97.536 235.458) (width 0.254) (layer F.Cu) (net 103))
+  (via (at 97.536 235.458) (size 1.10236) (drill 0.6096) (layers F.Cu B.Cu) (net 103))
+  (segment (start 162.016 259.032) (end 159.56 259.032) (width 0.254) (layer F.Cu) (net 103))
+  (segment (start 159.56 259.032) (end 159.512 259.08) (width 0.254) (layer F.Cu) (net 103))
+  (via (at 159.512 259.08) (size 1.10236) (drill 0.6096) (layers F.Cu B.Cu) (net 103))
+  (segment (start 162.016 253.532) (end 164.298 253.532) (width 0.254) (layer F.Cu) (net 103))
+  (segment (start 164.298 253.532) (end 164.338 253.492) (width 0.254) (layer F.Cu) (net 103))
+  (via (at 164.338 253.492) (size 1.10236) (drill 0.6096) (layers F.Cu B.Cu) (net 103))
+  (segment (start 109.728 205.486) (end 109.503 205.486) (width 0.3048) (layer F.Cu) (net 103))
+  (segment (start 117.982 195.052) (end 116.352 195.052) (width 0.3048) (layer F.Cu) (net 103))
+  (segment (start 116.352 195.052) (end 113.792 197.612) (width 0.3048) (layer F.Cu) (net 103))
+  (via (at 113.792 197.612) (size 1.10236) (drill 0.6096) (layers F.Cu B.Cu) (net 103))
   (segment (start 162.814 -20.98801) (end 162.814 -20.828) (width 0.254) (layer F.Cu) (net 136))
   (segment (start 162.814 -20.828) (end 164.338 -19.304) (width 0.254) (layer F.Cu) (net 136))
@@
   (segment (start 129.918 -24.638) (end 127.464 -22.184) (width 0.254) (layer F.Cu) (net 145))
   (segment (start 127.464 -22.184) (end 127.464 -21.53) (width 0.254) (layer F.Cu) (net 145))
+  (zone (net 103) (net_name GND) (layer F.Cu) (hatch edge 0.508)
+    (connect_pads yes (clearance 0.1524))
+    (min_thickness 0.254)
+    (fill yes (arc_segments 16) (thermal_gap 0.508) (thermal_bridge_width 0.508))
+    (polygon
+      (pts
+        (xy 166.37 -26.67) (xy 166.37 -13.97) (xy 124.46 -13.97) (xy 124.46 -26.67)
+      )
+    )
+  )
+  (zone (net 103) (net_name GND) (layer B.Cu) (hatch edge 0.508)
+    (connect_pads yes (clearance 0.1524))
+    (min_thickness 0.254)
+    (fill yes (arc_segments 16) (thermal_gap 0.508) (thermal_bridge_width 0.508))
+    (polygon
+      (pts
+        (xy 166.37 -26.67) (xy 166.37 261.874) (xy 76.2 261.874) (xy 76.2 -26.67)
+      )
+    )
+  )
+  (zone (net 103) (net_name GND) (layer F.Cu) (hatch edge 0.508)
+    (connect_pads yes (clearance 0.1524))
+    (min_thickness 0.254)
+    (fill yes (arc_segments 16) (thermal_gap 0.508) (thermal_bridge_width 0.508))
+    (polygon
+      (pts
+        (xy 76.2 261.874) (xy 166.37 261.874) (xy 166.37 212.09) (xy 121.92 212.09) (xy 121.92 204.47)
+        (xy 76.2 204.47)
+      )
+    )
+  )
 )
