File: Circuit/peripheral-bridge-v3/peripheral-birdge-v3.kicad_pcb (KiCad board)
At the start: 2 copper layers, 60 x 59.3 mm, 79 parts, among them CON1 Conn-Edge-PCIE-x1, J1 To DVL, J2 Pressure Sensor, J3 Solenoid, J4 USB_OTG, J5 DSP_Reset, P1 Solenoid Power, Q1 BSS138, U1 FT2232H, U2 93LC56BT-I/OT, U3 ADM3251E, U4 ADC101S021, U5 ACPL-247-500E, U6 ACPL-247-500E, U7 LM1117-33, Y1 12MHz

Commit message: GND pin of ADC of peripheral bridge not connected to GND
Connections:
- C22 pad 2: Net-(C22-Pad2) -> GND
- C23 pad 1: Net-(C22-Pad2) -> GND
- J2 pad 3: Net-(C22-Pad2) -> GND
- U4 pad 2: Net-(C22-Pad2) -> GND
Routing:
- net GND: track 232.1 -> 247.1 mm
- net Net-(C22-Pad2): track 15.0 -> 0.00 mm
