File: Circuit/PWM_Isolator/PWM_Isolator.sch (KiCad schematic (older format))
At the start: 12 parts, among them P1 GND_IN_1, P10 NC, P2 GND_IN_2, P3 Pololu PWM + Power rail, P4 PWM_OUT_1, P5 PWM_OUT_2, P6 Motor_Pwr1, P7 Motor_Pwr2, P8 Motor PWR, P9 Motor PWR, U1 Si8660BA-B-IS1, U2 Si8660BA-B-IS1

Commit message: updated pins and sockets of PWM_Isolator
Parts:
- removed P1: GND_IN_1, Socket_Strips:Socket_Strip_Straight_2x06, symbol CONN_02X06
- removed P10: NC, Socket_Strips:Socket_Strip_Straight_1x07, symbol CONN_01X07
- removed P2: GND_IN_2, Socket_Strips:Socket_Strip_Straight_2x06, symbol CONN_02X06
- removed P3: Pololu PWM + Power rail, Socket_Strips:Socket_Strip_Straight_1x13, symbol CONN_01X13
- removed P4: PWM_OUT_1, Pin_Headers:Pin_Header_Straight_1x06, symbol CONN_01X06
- removed P5: PWM_OUT_2, Pin_Headers:Pin_Header_Straight_1x06, symbol CONN_01X06
- removed P6: Motor_Pwr1, Pin_Headers:Pin_Header_Straight_2x06, symbol CONN_02X06
- removed P7: Motor_Pwr2, Pin_Headers:Pin_Header_Straight_2x06, symbol CONN_02X06
- removed P8, P9: Motor PWR, Pin_Headers:Pin_Header_Straight_1x01, symbol CONN_01X01
- added P1: GND_IN_1, Socket_Strips:Socket_Strip_Straight_2x06_Pitch2.54mm, symbol Conn_02x06_Odd_Even
- added P10: NC, Socket_Strips:Socket_Strip_Straight_1x07_Pitch2.54mm, symbol Conn_01x07
- added P2: GND_IN_2, Socket_Strips:Socket_Strip_Straight_2x06_Pitch2.54mm, symbol Conn_02x06_Odd_Even
- added P3: Pololu PWM + Power rail, Socket_Strips:Socket_Strip_Straight_1x13_Pitch2.54mm, symbol Conn_01x13
- added P4: PWM_OUT_1, Pin_Headers:Pin_Header_Straight_1x06_Pitch2.54mm, symbol Conn_01x06
- added P5: PWM_OUT_2, Pin_Headers:Pin_Header_Straight_1x06_Pitch2.54mm, symbol Conn_01x06
- added P6: Motor_Pwr1, Pin_Headers:Pin_Header_Straight_2x06_Pitch2.54mm, symbol Conn_02x06_Odd_Even
- added P7: Motor_Pwr2, Pin_Headers:Pin_Header_Straight_2x06_Pitch2.54mm, symbol Conn_02x06_Odd_Even
- added P8, P9: Motor PWR, Pin_Headers:Pin_Header_Straight_1x01_Pitch2.54mm, symbol Conn_01x01
