File: Circuit/Peripheral_bridge/Comm_Bridge.sch (KiCad schematic (older format))
At the start: 95 parts, among them P1 USB_B, P2 CONN_01X03, P3 Solenoid, P4 XT60, P5 CONN_01X03, P6 CONN_01X03, U1 FT4232H, U10 ADM3251E, U11 ADM3251E, U2 93LC56BT-I/OT, U3 74HC595_CUST, U4 LM1117-XX, U5 ADC101S021, U6 NLSX4373, U7 NLSX4373, U8 ACPL-247-500E, U9 ACPL-247-500E, Y1 12MHz

Commit message: removed ignored files of Peripheral_bridge
Parts:
- removed P3: Solenoid, Zeabus:Pin_Header_Straight_2x04, symbol CONN_02X04
- added P3: Solenoid, Zeabus:Pin_Header_Straight_2x04, symbol Conn_02x04_Odd_Even
- P2, P5, P6: symbol CONN_01X03 -> Conn_01x03
Changed lines of the file:
@@
 LIBS:ftdi
 LIBS:zeabus
+LIBS:Comm_Bridge-cache
 EELAYER 25 0
 EELAYER END
@@
 $EndComp
 $Comp
-L CONN_01X03 P6
+L Conn_01x03 P6
 U 1 1 5648C117
 P 11050 5750
@@
 $EndComp
 $Comp
-L CONN_01X03 P5
+L Conn_01x03 P5
 U 1 1 564BB4DC
 P 11050 4200
@@
 	5200 1100 5850 1100
 $Comp
-L CONN_01X03 P2
+L Conn_01x03 P2
 U 1 1 58CBB843
 P 5700 750
@@
 Text Notes 10350 1900 0    60   ~ 12
 Solenoid Power\n
-$Comp
-L CONN_02X04 P3
-U 1 1 58CE0E11
-P 10100 1150
-F 0 "P3" H 10100 1450 50  0000 C CNN
-F 1 "Solenoid" H 10100 1400 50  0000 C CNB
-F 2 "Zeabus:Pin_Header_Straight_2x04" H 10100 -50 50  0001 C CNN
-F 3 "" H 10100 -50 50  0000 C CNN
-	1    10100 1150
-	1    0    0    -1
-$EndComp
 $Comp
 L +12V #PWR058
@@
 	1    0    0    -1
 $EndComp
+$Comp
+L Conn_02x04_Odd_Even P3
+U 1 1 5B211298
+P 10050 1100
+F 0 "P3" H 10100 1300 50  0000 C CNN
+F 1 "Solenoid" H 10100 800 50  0000 C CNN
+F 2 "Zeabus:Pin_Header_Straight_2x04" H 10050 1100 50  0001 C CNN
+F 3 "" H 10050 1100 50  0001 C CNN
+	1    10050 1100
+	1    0    0    -1
+$EndComp
