File: Circuit/Switch_board/Switch_board.sch (KiCad schematic (older format))
At the start: 27 parts, among them J1 switch_mode, J2 switch_connector, P1 power_in, Q1 2N7002, Q2 2N7002, Q3 2N7002, Q4 2N7002, U1 DRV5023

Commit message: added reverse voltage protection and reduced start-up voltage of Switch_board
Parts:
- added D?: BZX585-C12, Diodes_SMD:D_SOD-523, symbol D_Zener
- added Q?: RSC002P03, TO_SOT_Packages_SMD:SOT-23_Handsoldering, symbol Q_PMOS_GSD
- added R?: 100, Resistors_SMD:R_0603_HandSoldering, symbol R
- added R?: 10k, Resistors_SMD:R_0603_HandSoldering, symbol R
Connections:
- wire segments 65 -> 71
Other:
- moved on the sheet: P1
Changed lines of the file:
@@
 L XT30 P1
 U 1 1 5A826541
-P 2000 4250
-F 0 "P1" H 2000 4400 50  0000 C CNN
-F 1 "power_in" H 2000 4100 50  0000 C CNN
-F 2 "zeabus:XT30" H 2000 4250 60  0001 C CNN
-F 3 "" H 2000 4250 60  0000 C CNN
-	1    2000 4250
+P 1200 4250
+F 0 "P1" H 1200 4400 50  0000 C CNN
+F 1 "power_in" H 1200 4100 50  0000 C CNN
+F 2 "zeabus:XT30" H 1200 4250 60  0001 C CNN
+F 3 "" H 1200 4250 60  0000 C CNN
+	1    1200 4250
 	-1   0    0    -1
 $EndComp
@@
 L GND #PWR3
 U 1 1 5A826918
-P 2300 4350
-F 0 "#PWR3" H 2300 4100 50  0001 C CNN
-F 1 "GND" H 2300 4200 50  0000 C CNN
-F 2 "" H 2300 4350 50  0001 C CNN
-F 3 "" H 2300 4350 50  0001 C CNN
-	1    2300 4350
+P 1500 4350
+F 0 "#PWR3" H 1500 4100 50  0001 C CNN
+F 1 "GND" H 1500 4200 50  0000 C CNN
+F 2 "" H 1500 4350 50  0001 C CNN
+F 3 "" H 1500 4350 50  0001 C CNN
+	1    1500 4350
 	1    0    0    -1
 $EndComp
@@
 L VCC #PWR6
 U 1 1 5A89DB47
-P 3050 3900
-F 0 "#PWR6" H 3050 3750 50  0001 C CNN
-F 1 "VCC" H 3050 4050 50  0000 C CNN
-F 2 "" H 3050 3900 50  0001 C CNN
-F 3 "" H 3050 3900 50  0001 C CNN
-	1    3050 3900
+P 2550 3900
+F 0 "#PWR6" H 2550 3750 50  0001 C CNN
+F 1 "VCC" H 2550 4050 50  0000 C CNN
+F 2 "" H 2550 3900 50  0001 C CNN
+F 3 "" H 2550 3900 50  0001 C CNN
+	1    2550 3900
 	1    0    0    -1
 $EndComp
@@
 L PWR_FLAG #FLG2
 U 1 1 5A8DF01C
-P 2700 3250
-F 0 "#FLG2" H 2700 3325 50  0001 C CNN
-F 1 "PWR_FLAG" H 2700 3400 50  0000 C CNN
-F 2 "" H 2700 3250 50  0001 C CNN
-F 3 "" H 2700 3250 50  0001 C CNN
-	1    2700 3250
+P 1950 3150
+F 0 "#FLG2" H 1950 3225 50  0001 C CNN
+F 1 "PWR_FLAG" H 1950 3300 50  0000 C CNN
+F 2 "" H 1950 3150 50  0001 C CNN
+F 3 "" H 1950 3150 50  0001 C CNN
+	1    1950 3150
 	1    0    0    -1
 $EndComp
@@
 L PWR_FLAG #FLG1
 U 1 1 5A8DF1C6
-P 2300 3400
-F 0 "#FLG1" H 2300 3475 50  0001 C CNN
-F 1 "PWR_FLAG" H 2300 3550 50  0000 C CNN
-F 2 "" H 2300 3400 50  0001 C CNN
-F 3 "" H 2300 3400 50  0001 C CNN
-	1    2300 3400
+P 1550 3300
+F 0 "#FLG1" H 1550 3375 50  0001 C CNN
+F 1 "PWR_FLAG" H 1550 3450 50  0000 C CNN
+F 2 "" H 1550 3300 50  0001 C CNN
+F 3 "" H 1550 3300 50  0001 C CNN
+	1    1550 3300
 	-1   0    0    1
 $EndComp
@@
 L VCC #PWR2
 U 1 1 5A8E00E8
-P 2300 3250
-F 0 "#PWR2" H 2300 3100 50  0001 C CNN
-F 1 "VCC" H 2300 3400 50  0000 C CNN
-F 2 "" H 2300 3250 50  0001 C CNN
-F 3 "" H 2300 3250 50  0001 C CNN
-	1    2300 3250
+P 1550 3150
+F 0 "#PWR2" H 1550 3000 50  0001 C CNN
+F 1 "VCC" H 1550 3300 50  0000 C CNN
+F 2 "" H 1550 3150 50  0001 C CNN
+F 3 "" H 1550 3150 50  0001 C CNN
+	1    1550 3150
 	1    0    0    -1
 $EndComp
@@
 L GND #PWR5
 U 1 1 5A8E04F5
-P 2700 3400
-F 0 "#PWR5" H 2700 3150 50  0001 C CNN
-F 1 "GND" H 2700 3250 50  0000 C CNN
-F 2 "" H 2700 3400 50  0001 C CNN
-F 3 "" H 2700 3400 50  0001 C CNN
-	1    2700 3400
+P 1950 3300
+F 0 "#PWR5" H 1950 3050 50  0001 C CNN
+F 1 "GND" H 1950 3150 50  0000 C CNN
+F 2 "" H 1950 3300 50  0001 C CNN
+F 3 "" H 1950 3300 50  0001 C CNN
+	1    1950 3300
 	1    0    0    -1
 $EndComp
@@
 +switch
 Wire Wire Line
-	3050 3900 3050 4300
-Wire Wire Line
 	3700 4650 3700 4750
 Wire Wire Line
-	3050 4600 3050 4700
-Wire Wire Line
-	3050 4700 3700 4700
-Connection ~ 3700 4700
-Connection ~ 3050 4200
-Wire Wire Line
-	2200 4300 2300 4300
+	3050 4600 3050 4750
+Wire Wire Line
+	1400 4300 1500 4300
 Wire Wire Line
 	4400 4050 4400 4350
@@
 	8350 3950 8550 3950
 Wire Wire Line
-	2300 4300 2300 4350
+	1500 4300 1500 4350
 Wire Wire Line
 	4400 3650 4400 3750
 Wire Wire Line
 	6300 3400 6250 3400
-Wire Wire Line
-	2200 4200 3200 4200
 Wire Wire Line
 	5850 3850 5850 3950
@@
 	7350 2700 7350 3050
 Wire Wire Line
-	2300 3250 2300 3400
-Wire Wire Line
-	2700 3250 2700 3400
+	1550 3150 1550 3300
+Wire Wire Line
+	1950 3150 1950 3300
 Wire Wire Line
 	1550 2050 1550 2150
@@
 Wire Wire Line
 	8350 3950 8350 4100
+$Comp
+L Q_PMOS_GSD Q?
+U 1 1 5B46388D
+P 1900 4300
+F 0 "Q?" V 2100 4350 50  0000 L CNN
+F 1 "RSC002P03" V 2100 4250 50  0000 R CNN
+F 2 "TO_SOT_Packages_SMD:SOT-23_Handsoldering" H 2100 4400 50  0001 L CNN
+F 3 "" H 1900 4300 50  0001 C CNN
+	1    1900 4300
+	0    -1   -1   0
+$EndComp
+$Comp
+L R R?
+U 1 1 5B4649A0
+P 2800 4200
+F 0 "R?" V 2880 4200 50  0000 C CNN
+F 1 "100" V 2800 4200 50  0000 C CNN
+F 2 "Resistors_SMD:R_0603_HandSoldering" V 2730 4200 50  0001 C CNN
+F 3 "" H 2800 4200 50  0001 C CNN
+	1    2800 4200
+	0    1    1    0
+$EndComp
+Wire Wire Line
+	3050 4300 3050 4200
+Connection ~ 3050 4200
+Wire Wire Line
+	2550 3900 2550 4600
+Connection ~ 2550 4200
+Wire Wire Line
+	2550 4600 2400 4600
+Wire Wire Line
+	1900 4500 1900 4750
+$Comp
+L R R?
+U 1 1 5B4652C3
+P 1900 4900
+F 0 "R?" V 1980 4900 50  0000 C CNN
+F 1 "10k" V 1900 4900 50  0000 C CNN
+F 2 "Resistors_SMD:R_0603_HandSoldering" V 1830 4900 50  0001 C CNN
+F 3 "" H 1900 4900 50  0001 C CNN
+	1    1900 4900
+	1    0    0    -1
+$EndComp
+$Comp
+L GND #PWR?
+U 1 1 5B465687
+P 1900 5200
+F 0 "#PWR?" H 1900 4950 50  0001 C CNN
+F 1 "GND" H 1900 5050 50  0000 C CNN
+F 2 "" H 1900 5200 50  0001 C CNN
+F 3 "" H 1900 5200 50  0001 C CNN
+	1    1900 5200
+	1    0    0    -1
+$EndComp
+Wire Wire Line
+	1900 5200 1900 5050
+Wire Wire Line
+	2100 4600 1900 4600
+Connection ~ 1900 4600
+Wire Wire Line
+	1700 4200 1400 4200
+Wire Wire Line
+	2100 4200 2650 4200
+Wire Wire Line
+	2950 4200 3200 4200
+$Comp
+L GND #PWR?
+U 1 1 5B467A51
+P 3050 4750
+F 0 "#PWR?" H 3050 4500 50  0001 C CNN
+F 1 "GND" H 3050 4600 50  0000 C CNN
+F 2 "" H 3050 4750 50  0001 C CNN
+F 3 "" H 3050 4750 50  0001 C CNN
+	1    3050 4750
+	1    0    0    -1
+$EndComp
+$Comp
+L D_Zener D?
+U 1 1 5B468894
+P 2250 4600
+F 0 "D?" H 2250 4700 50  0000 C CNN
+F 1 "BZX585-C12" H 2250 4500 50  0000 C CNN
+F 2 "Diodes_SMD:D_SOD-523" H 2250 4600 50  0001 C CNN
+F 3 "" H 2250 4600 50  0001 C CNN
+	1    2250 4600
+	-1   0    0    1
+$EndComp
 $EndSCHEMATC

Commit message: changed 12v zener diode to BZT52c12s on Switch_board
Parts:
- D1, D?: value BZX585-C12 -> BZT52C12S; footprint Diodes_SMD:D_SOD-523 -> Diodes_SMD:D_SOD-323_HandSoldering
Changed lines of the file:
@@
 P 7850 3300
 F 0 "D1" H 7850 3400 50  0000 C CNN
-F 1 "BZX585-C12" H 7850 3200 50  0000 C CNN
-F 2 "Diodes_SMD:D_SOD-523" H 7850 3300 50  0001 C CNN
+F 1 "BZT52C12S" H 7850 3200 50  0000 C CNN
+F 2 "Diodes_SMD:D_SOD-323_HandSoldering" H 7850 3300 50  0001 C CNN
 F 3 "" H 7850 3300 50  0001 C CNN
 	1    7850 3300
@@
 P 2250 4600
 F 0 "D?" H 2250 4700 50  0000 C CNN
-F 1 "BZX585-C12" H 2250 4500 50  0000 C CNN
-F 2 "Diodes_SMD:D_SOD-523" H 2250 4600 50  0001 C CNN
+F 1 "BZT52C12S" H 2250 4500 50  0000 C CNN
+F 2 "Diodes_SMD:D_SOD-323_HandSoldering" H 2250 4600 50  0001 C CNN
 F 3 "" H 2250 4600 50  0001 C CNN
 	1    2250 4600

Commit message: Switch_board Rev1.1 was routed
Parts:
- gave numbers to parts that had none: 4
Changed lines of the file:
@@
 Sheet 1 1
 Title "Switch_board"
-Date "2018-02-21"
-Rev "1.0.0"
-Comp "Zeabus"
+Date "2018-07-12"
+Rev "1.1.0"
+Comp "Zeabus2018"
 Comment1 ""
 Comment2 ""
@@
 $EndComp
 $Comp
-L GND #PWR8
+L GND #PWR10
 U 1 1 5A826833
 P 3700 4750
-F 0 "#PWR8" H 3700 4500 50  0001 C CNN
+F 0 "#PWR10" H 3700 4500 50  0001 C CNN
 F 1 "GND" H 3700 4600 50  0000 C CNN
 F 2 "" H 3700 4750 50  0001 C CNN
@@
 $EndComp
 $Comp
-L GND #PWR3
+L GND #PWR1
 U 1 1 5A826918
 P 1500 4350
-F 0 "#PWR3" H 1500 4100 50  0001 C CNN
+F 0 "#PWR1" H 1500 4100 50  0001 C CNN
 F 1 "GND" H 1500 4200 50  0000 C CNN
 F 2 "" H 1500 4350 50  0001 C CNN
@@
 $EndComp
 $Comp
-L GND #PWR20
+L GND #PWR22
 U 1 1 5A829801
 P 8350 4100
-F 0 "#PWR20" H 8350 3850 50  0001 C CNN
+F 0 "#PWR22" H 8350 3850 50  0001 C CNN
 F 1 "GND" H 8350 3950 50  0000 C CNN
 F 2 "" H 8350 4100 50  0001 C CNN
@@
 $EndComp
 $Comp
-L GND #PWR14
+L GND #PWR16
 U 1 1 5A829CAE
 P 5850 3950
-F 0 "#PWR14" H 5850 3700 50  0001 C CNN
+F 0 "#PWR16" H 5850 3700 50  0001 C CNN
 F 1 "GND" H 5850 3800 50  0000 C CNN
 F 2 "" H 5850 3950 50  0001 C CNN
@@
 $EndComp
 $Comp
-L GND #PWR11
+L GND #PWR13
 U 1 1 5A883892
 P 4400 4750
-F 0 "#PWR11" H 4400 4500 50  0001 C CNN
+F 0 "#PWR13" H 4400 4500 50  0001 C CNN
 F 1 "GND" H 4400 4600 50  0000 C CNN
 F 2 "" H 4400 4750 50  0001 C CNN
@@
 $EndComp
 $Comp
-L GND #PWR16
+L GND #PWR18
 U 1 1 5A88921C
 P 6600 3700
-F 0 "#PWR16" H 6600 3450 50  0001 C CNN
+F 0 "#PWR18" H 6600 3450 50  0001 C CNN
 F 1 "GND" H 6600 3550 50  0000 C CNN
 F 2 "" H 6600 3700 50  0001 C CNN
@@
 $EndComp
 $Comp
-L VCC #PWR6
+L VCC #PWR7
 U 1 1 5A89DB47
 P 2550 3900
-F 0 "#PWR6" H 2550 3750 50  0001 C CNN
+F 0 "#PWR7" H 2550 3750 50  0001 C CNN
 F 1 "VCC" H 2550 4050 50  0000 C CNN
 F 2 "" H 2550 3900 50  0001 C CNN
@@
 $EndComp
 $Comp
-L GND #PWR19
+L GND #PWR21
 U 1 1 5A89F539
 P 7850 3550
-F 0 "#PWR19" H 7850 3300 50  0001 C CNN
+F 0 "#PWR21" H 7850 3300 50  0001 C CNN
 F 1 "GND" H 7850 3400 50  0000 C CNN
 F 2 "" H 7850 3550 50  0001 C CNN
@@
 $EndComp
 $Comp
-L GND #PWR17
+L GND #PWR19
 U 1 1 5A8DDCE5
 P 6600 4850
-F 0 "#PWR17" H 6600 4600 50  0001 C CNN
+F 0 "#PWR19" H 6600 4600 50  0001 C CNN
 F 1 "GND" H 6600 4700 50  0000 C CNN
 F 2 "" H 6600 4850 50  0001 C CNN
@@
 $EndComp
 $Comp
-L GND #PWR18
+L GND #PWR20
 U 1 1 5A8DDCF1
 P 7350 4600
-F 0 "#PWR18" H 7350 4350 50  0001 C CNN
+F 0 "#PWR20" H 7350 4350 50  0001 C CNN
 F 1 "GND" H 7350 4450 50  0000 C CNN
 F 2 "" H 7350 4600 50  0001 C CNN
@@
 $EndComp
 $Comp
-L VCC #PWR15
+L VCC #PWR17
 U 1 1 5A8DFBDA
 P 6600 2600
-F 0 "#PWR15" H 6600 2450 50  0001 C CNN
+F 0 "#PWR17" H 6600 2450 50  0001 C CNN
 F 1 "VCC" H 6600 2750 50  0000 C CNN
 F 2 "" H 6600 2600 50  0001 C CNN
@@
 $EndComp
 $Comp
-L VCC #PWR10
+L VCC #PWR12
 U 1 1 5A89E7B6
 P 4400 3650
-F 0 "#PWR10" H 4400 3500 50  0001 C CNN
+F 0 "#PWR12" H 4400 3500 50  0001 C CNN
 F 1 "VCC" H 4400 3800 50  0000 C CNN
 F 2 "" H 4400 3650 50  0001 C CNN
@@
 $EndComp
 $Comp
-L VCC #PWR2
+L VCC #PWR3
 U 1 1 5A8E00E8
 P 1550 3150
-F 0 "#PWR2" H 1550 3000 50  0001 C CNN
+F 0 "#PWR3" H 1550 3000 50  0001 C CNN
 F 1 "VCC" H 1550 3300 50  0000 C CNN
 F 2 "" H 1550 3150 50  0001 C CNN
@@
 $EndComp
 $Comp
-L VCC #PWR1
+L VCC #PWR2
 U 1 1 5A908EA5
 P 1550 2050
-F 0 "#PWR1" H 1550 1900 50  0001 C CNN
+F 0 "#PWR2" H 1550 1900 50  0001 C CNN
 F 1 "VCC" H 1550 2200 50  0000 C CNN
 F 2 "" H 1550 2050 50  0001 C CNN
@@
 $EndComp
 $Comp
-L GND #PWR4
+L GND #PWR6
 U 1 1 5A90AC6B
 P 2350 2250
-F 0 "#PWR4" H 2350 2000 50  0001 C CNN
+F 0 "#PWR6" H 2350 2000 50  0001 C CNN
 F 1 "GND" H 2350 2100 50  0000 C CNN
 F 2 "" H 2350 2250 50  0001 C CNN
@@
 $EndComp
 $Comp
-L GND #PWR9
+L GND #PWR11
 U 1 1 5A90FC02
 P 4100 2950
-F 0 "#PWR9" H 4100 2700 50  0001 C CNN
+F 0 "#PWR11" H 4100 2700 50  0001 C CNN
 F 1 "GND" H 4100 2800 50  0000 C CNN
 F 2 "" H 4100 2950 50  0001 C CNN
@@
 $EndComp
 $Comp
-L VCC #PWR7
+L VCC #PWR9
 U 1 1 5A919C90
 P 3250 2050
-F 0 "#PWR7" H 3250 1900 50  0001 C CNN
+F 0 "#PWR9" H 3250 1900 50  0001 C CNN
 F 1 "VCC" H 3250 2200 50  0000 C CNN
 F 2 "" H 3250 2050 50  0001 C CNN
@@
 $EndComp
 $Comp
-L GND #PWR13
+L GND #PWR15
 U 1 1 5A932A61
 P 5850 2950
-F 0 "#PWR13" H 5850 2700 50  0001 C CNN
+F 0 "#PWR15" H 5850 2700 50  0001 C CNN
 F 1 "GND" H 5850 2800 50  0000 C CNN
 F 2 "" H 5850 2950 50  0001 C CNN
@@
 $EndComp
 $Comp
-L VCC #PWR12
+L VCC #PWR14
 U 1 1 5A932A73
 P 5000 2050
-F 0 "#PWR12" H 5000 1900 50  0001 C CNN
+F 0 "#PWR14" H 5000 1900 50  0001 C CNN
 F 1 "VCC" H 5000 2200 50  0000 C CNN
 F 2 "" H 5000 2050 50  0001 C CNN
@@
 	8350 3950 8350 4100
 $Comp
-L Q_PMOS_GSD Q?
+L Q_PMOS_GSD Q5
 U 1 1 5B46388D
 P 1900 4300
-F 0 "Q?" V 2100 4350 50  0000 L CNN
+F 0 "Q5" V 2100 4350 50  0000 L CNN
 F 1 "RSC002P03" V 2100 4250 50  0000 R CNN
 F 2 "TO_SOT_Packages_SMD:SOT-23_Handsoldering" H 2100 4400 50  0001 L CNN
@@
 $EndComp
 $Comp
-L R R?
+L R R14
 U 1 1 5B4649A0
 P 2800 4200
-F 0 "R?" V 2880 4200 50  0000 C CNN
+F 0 "R14" V 2880 4200 50  0000 C CNN
 F 1 "100" V 2800 4200 50  0000 C CNN
 F 2 "Resistors_SMD:R_0603_HandSoldering" V 2730 4200 50  0001 C CNN
@@
 	1900 4500 1900 4750
 $Comp
-L R R?
+L R R13
 U 1 1 5B4652C3
 P 1900 4900
-F 0 "R?" V 1980 4900 50  0000 C CNN
+F 0 "R13" V 1980 4900 50  0000 C CNN
 F 1 "10k" V 1900 4900 50  0000 C CNN
 F 2 "Resistors_SMD:R_0603_HandSoldering" V 1830 4900 50  0001 C CNN
@@
 $EndComp
 $Comp
-L GND #PWR?
+L GND #PWR4
 U 1 1 5B465687
 P 1900 5200
-F 0 "#PWR?" H 1900 4950 50  0001 C CNN
+F 0 "#PWR4" H 1900 4950 50  0001 C CNN
 F 1 "GND" H 1900 5050 50  0000 C CNN
 F 2 "" H 1900 5200 50  0001 C CNN
@@
 	2950 4200 3200 4200
 $Comp
-L GND #PWR?
+L GND #PWR8
 U 1 1 5B467A51
 P 3050 4750
-F 0 "#PWR?" H 3050 4500 50  0001 C CNN
+F 0 "#PWR8" H 3050 4500 50  0001 C CNN
 F 1 "GND" H 3050 4600 50  0000 C CNN
 F 2 "" H 3050 4750 50  0001 C CNN
@@
 $EndComp
 $Comp
-L D_Zener D?
+L D_Zener D6
 U 1 1 5B468894
 P 2250 4600
-F 0 "D?" H 2250 4700 50  0000 C CNN
+F 0 "D6" H 2250 4700 50  0000 C CNN
 F 1 "BZT52C12S" H 2250 4500 50  0000 C CNN
 F 2 "Diodes_SMD:D_SOD-323_HandSoldering" H 2250 4600 50  0001 C CNN
