File: Circuit/Switch_board/Switch_board.sch (KiCad schematic (older format))
At the start: 31 parts, among them J1 switch_mode, J2 switch_connector, P1 power_in, Q1 2N7002, Q2 2N7002, Q3 2N7002, Q4 2N7002, Q5 RSC002P03, U1 DRV5023

Commit message: changed DRV5023 apprance and labels on switch_board
Connections:
- net labels added: switch+
- net labels removed: +switch
Changed lines of the file:
@@
 LIBS:valves
 LIBS:zeabus
-LIBS:Switch_board-cache
 EELAYER 25 0
 EELAYER END
@@
 	1    0    0    -1
 $EndComp
-Text GLabel 4900 4750 2    60   Input ~ 0
+Text GLabel 4900 4750 2    60   Output ~ 0
 hall_sensor_out
 Text GLabel 3350 2650 0    60   Input ~ 0
 hall_sensor_out
-Text GLabel 8500 3050 2    60   Input ~ 0
-+switch
+Text GLabel 8500 3050 2    60   Output ~ 0
+switch+
 Wire Wire Line
 	3700 4650 3700 4750
@@
 $EndComp
 Text GLabel 5100 2650 0    60   Input ~ 0
-+switch
+switch+
 Wire Wire Line
 	5550 2650 5500 2650
