File: Circuit/Peripheral-bridge-v3/peripheral-birdge-v3.sch (KiCad schematic (older format))
At the start: 76 parts, among them CON1 Conn-Edge-PCIE-x1, J1 To DVL, J2 Pressure Sensor, J3 Solenoid, J4 USB_OTG, J5 DSP_Reset, P1 Solenoid Power, Q1 BSS138, U1 FT2232H, U2 93LC56BT-I/OT, U3 ADM3251E, U4 ADC101S021, U5 ACPL-247-500E, U6 ACPL-247-500E, U7 LM1117-33, Y1 12MHz

Commit message: added SEL_+5V_SRC to peripheral_bridge_v3
Parts:
- added J?: SEL_+5V_SRC, symbol Conn_01x03_Selection_Source
Connections:
- net labels added: +5V, +5_PCIE, +5_USB
- net labels removed: +5Vin
- wire segments 302 -> 310
Other:
- moved on the sheet: C22, C23, J2, L4, R1, R2, U4

Commit message: added SEL_DATA_SRC to peripheral_bridge_v3
Parts:
- added C?: 0.1uF, Capacitors_SMD:C_0603, symbol C_Small
- added J?: SEL_DATA_SRC, symbol Conn_01x03_Selection_Source
- added R?: 50, Resistors_SMD:R_0603, symbol R
- added R?: 100, Resistors_SMD:R_0603, symbol R
- added U?: FSUSB30, Housings_SSOP:MSOP-10_3x3mm_Pitch0.5mm, symbol FSUSB30
Connections:
- net labels added: DM_CTRL, DM_PCIE, DM_USB, DP_CTRL, DP_PCIE, DP_USB
- net labels removed: D+, D-
- wire segments 310 -> 333
Other:
- moved on the sheet: F1

Commit message: changed +5V flags to +5V_CTRL and VBUS to +5V
Connections:
- net labels added: +5_CTRL
- net labels removed: VBUS

Commit message: added power rail leds to peripheral_bridge_v3
Parts:
- added D? (x5): LED_Small, symbol LED_Small
- added R? (x4): 1k, Resistors_SMD:R_0603, symbol R
- added R?: 150, Resistors_SMD:R_0603, symbol R
Connections:
- wire segments 333 -> 362

Commit message: added label on power rail leds in peripheral_bridge-v3
Parts:
- D?: value LED_Small -> +12V_LED
- D?: value LED_Small -> +5V_USB_LED
- D?: value LED_Small -> +5V_PCIE_LED
- D?: value LED_Small -> +5V_CTRL_LED
- D?: value LED_Small -> +3V3_LED
Changed lines of the file:
@@
 P -700 850
 F 0 "D?" H -750 975 50  0000 L CNN
-F 1 "LED_Small" H -875 750 50  0000 L CNN
+F 1 "+12V_LED" H -875 750 50  0000 L CNN
 F 2 "" V -700 850 50  0001 C CNN
 F 3 "" V -700 850 50  0001 C CNN
@@
 P -700 1450
 F 0 "D?" H -750 1575 50  0000 L CNN
-F 1 "LED_Small" H -875 1350 50  0000 L CNN
+F 1 "+5V_USB_LED" H -1000 1350 50  0000 L CNN
 F 2 "" V -700 1450 50  0001 C CNN
 F 3 "" V -700 1450 50  0001 C CNN
@@
 P -700 1950
 F 0 "D?" H -750 2075 50  0000 L CNN
-F 1 "LED_Small" H -875 1850 50  0000 L CNN
+F 1 "+5V_PCIE_LED" H -1000 1850 50  0000 L CNN
 F 2 "" V -700 1950 50  0001 C CNN
 F 3 "" V -700 1950 50  0001 C CNN
@@
 P -700 2450
 F 0 "D?" H -750 2575 50  0000 L CNN
-F 1 "LED_Small" H -875 2350 50  0000 L CNN
+F 1 "+5V_CTRL_LED" H -1000 2350 50  0000 L CNN
 F 2 "" V -700 2450 50  0001 C CNN
 F 3 "" V -700 2450 50  0001 C CNN
@@
 P -700 2950
 F 0 "D?" H -750 3075 50  0000 L CNN
-F 1 "LED_Small" H -875 2850 50  0000 L CNN
+F 1 "+3V3_LED" H -875 2850 50  0000 L CNN
 F 2 "" V -700 2950 50  0001 C CNN
 F 3 "" V -700 2950 50  0001 C CNN

Commit message: added main switch of GPIO switch on peripheral_bridge-v3
Parts:
- added Q?: BSS138, TO_SOT_Packages_SMD:SOT-23, symbol BSS138
- added R?: 1k, Resistors_SMD:R_0603, symbol R
- added R?: 1M, Resistors_SMD:R_0603, symbol R
Connections:
- net labels added: GPIO_SW, PRESSURE_VOLTAGE, RS232_GND, RS232_Rx, RS232_Tx, SOL_CTRL
- net labels removed: Analog_In, Rx, Tx
- wire segments 362 -> 390
- no-connect marks 9 -> 28
Other:
- moved on the sheet: C?, D3, D4, D5, D6, D7, D8, D9, J3, J5, P1, R12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
